Commit message: modified worms xacro (WIP)

File: catkin_ws/src/worms_description/urdf/worms_old.urdf (robot description, URDF)
Before this commit: robot worms, 26 links, 25 joints
Joints:
- joint j_thigh_lf: origin xyz=0 0 0 rpy= 0 3.14159 3.14159 -> xyz=0 0 0 rpy=3.14159 0  0
- joint j_thigh_lm: origin xyz=0 0 0 rpy= 0 3.14159 3.14159 -> xyz=0 0 0 rpy=3.14159 0  0
- joint j_thigh_lr: origin xyz=0 0 0 rpy= 0 3.14159 3.14159 -> xyz=0 0 0 rpy=3.14159 0  0
- joint j_thigh_rf: origin xyz=0 0 0 rpy= 0 3.14159 3.14159 -> xyz=0 0 0 rpy=3.14159 0  0
- joint j_thigh_rm: origin xyz=0 0 0 rpy= 0 3.14159 3.14159 -> xyz=0 0 0 rpy=3.14159 0  0
- joint j_thigh_rr: origin xyz=0 0 0 rpy= 0 3.14159 3.14159 -> xyz=0 0 0 rpy=3.14159 0  0
- joint j_worms_attachment: origin (none) -> xyz=0 0 0 rpy=0 0 0

File: catkin_ws/src/worms_description/urdf/worms_urdf.xacro (robot description, xacro)
@@ -21,8 +21,8 @@
           <geometry>
             <!--box size="0.102 0.109 0.106" /-->
-            <mesh filename="package://worms_description/meshes/body.STL"  scale="1 1 1"/>
+            <mesh filename="package://worms_description/meshes/Pallet.stl"  scale="1 1 1"/>
           </geometry>
-          <material name="Grey">
-            <color rgba="0.20 0.20 0.20 1.0"/>
+          <material name="Red">
+            <color rgba="0.2 0.2 0.2 1.0"/>
           </material>
         </visual>
@@ -35,5 +35,5 @@
       </link>
       <gazebo reference="MP_BODY">
-        <material>Gazebo/Grey</material>
+        <material>Gazebo/Red</material>
       </gazebo>
     <xacro:leg_l xyz="0.1248 -0.06164  0.001116"  rpy="0 4.7123 0.7853981633974483" suffix="rf"/>
