Commit message: added centered/rotated meshes for worms, reproduced worms.urdf with changes in xacro

File: catkin_ws/src/worms_description/urdf/worms_old2.urdf (robot description, URDF)
Before this commit: robot worms, 26 links, 25 joints
Links:
- link MP_BODY: geometry collision mesh filename=package://worms_description/meshes/Pallet.stl scale=1 1 1; visual mesh filename=package://worms_description/meshes/Pallet.stl scale=1 1 1
- link c1_lf: geometry collision mesh filename=package://worms_description/meshes/connect_coll.STL scale=1 1 1; visual mesh filename=package://worms_description/meshes/connect.STL scale=1 1 1
- link c1_lm: geometry collision mesh filename=package://worms_description/meshes/connect_coll.STL scale=1 1 1; visual mesh filename=package://worms_description/meshes/connect.STL scale=1 1 1
- link c1_lr: geometry collision mesh filename=package://worms_description/meshes/connect_coll.STL scale=1 1 1; visual mesh filename=package://worms_description/meshes/connect.STL scale=1 1 1
- link c1_rf: geometry collision mesh filename=package://worms_description/meshes/connect_coll.STL scale=1 1 1; visual mesh filename=package://worms_description/meshes/connect.STL scale=1 1 1
- link c1_rm: geometry collision mesh filename=package://worms_description/meshes/connect_coll.STL scale=1 1 1; visual mesh filename=package://worms_description/meshes/connect.STL scale=1 1 1
- link c1_rr: geometry collision mesh filename=package://worms_description/meshes/connect_coll.STL scale=1 1 1; visual mesh filename=package://worms_description/meshes/connect.STL scale=1 1 1
- link c2_lf: geometry collision mesh filename=package://worms_description/meshes/connect_coll.STL scale=1 1 1; visual mesh filename=package://worms_description/meshes/connect.STL scale=1 1 1
- link c2_lm: geometry collision mesh filename=package://worms_description/meshes/connect_coll.STL scale=1 1 1; visual mesh filename=package://worms_description/meshes/connect.STL scale=1 1 1
- link c2_lr: geometry collision mesh filename=package://worms_description/meshes/connect_coll.STL scale=1 1 1; visual mesh filename=package://worms_description/meshes/connect.STL scale=1 1 1
- link c2_rf: geometry collision mesh filename=package://worms_description/meshes/connect_coll.STL scale=1 1 1; visual mesh filename=package://worms_description/meshes/connect.STL scale=1 1 1
- link c2_rm: geometry collision mesh filename=package://worms_description/meshes/connect_coll.STL scale=1 1 1; visual mesh filename=package://worms_description/meshes/connect.STL scale=1 1 1
- link c2_rr: geometry collision mesh filename=package://worms_description/meshes/connect_coll.STL scale=1 1 1; visual mesh filename=package://worms_description/meshes/connect.STL scale=1 1 1
- link thigh_lf: geometry collision mesh filename=package://worms_description/meshes/thigh_l_coll.STL scale=1 1 1; visual mesh filename=package://worms_description/meshes/thigh_l.STL scale=1 1 1
- link thigh_lm: geometry collision mesh filename=package://worms_description/meshes/thigh_l_coll.STL scale=1 1 1; visual mesh filename=package://worms_description/meshes/thigh_l.STL scale=1 1 1
- link thigh_lr: geometry collision mesh filename=package://worms_description/meshes/thigh_l_coll.STL scale=1 1 1; visual mesh filename=package://worms_description/meshes/thigh_l.STL scale=1 1 1
- link thigh_rf: geometry collision mesh filename=package://worms_description/meshes/thigh_l_coll.STL scale=1 1 1; visual mesh filename=package://worms_description/meshes/thigh_l.STL scale=1 1 1
- link thigh_rm: geometry collision mesh filename=package://worms_description/meshes/thigh_l_coll.STL scale=1 1 1; visual mesh filename=package://worms_description/meshes/thigh_l.STL scale=1 1 1
- link thigh_rr: geometry collision mesh filename=package://worms_description/meshes/thigh_l_coll.STL scale=1 1 1; visual mesh filename=package://worms_description/meshes/thigh_l.STL scale=1 1 1
- link tibia_lf: geometry collision mesh filename=package://worms_description/meshes/tibia_l_coll.STL scale=1 1 1; visual mesh filename=package://worms_description/meshes/tibia_l.STL scale=1 1 1
- link tibia_lm: geometry collision mesh filename=package://worms_description/meshes/tibia_l_coll.STL scale=1 1 1; visual mesh filename=package://worms_description/meshes/tibia_l.STL scale=1 1 1
- link tibia_lr: geometry collision mesh filename=package://worms_description/meshes/tibia_l_coll.STL scale=1 1 1; visual mesh filename=package://worms_description/meshes/tibia_l.STL scale=1 1 1
- link tibia_rf: geometry collision mesh filename=package://worms_description/meshes/tibia_l_coll.STL scale=1 1 1; visual mesh filename=package://worms_description/meshes/tibia_l.STL scale=1 1 1
- link tibia_rm: geometry collision mesh filename=package://worms_description/meshes/tibia_l_coll.STL scale=1 1 1; visual mesh filename=package://worms_description/meshes/tibia_l.STL scale=1 1 1
- link tibia_rr: geometry collision mesh filename=package://worms_description/meshes/tibia_l_coll.STL scale=1 1 1; visual mesh filename=package://worms_description/meshes/tibia_l.STL scale=1 1 1

File: catkin_ws/src/worms_description/urdf/worms_urdf.xacro (robot description, xacro)
@@ -22,5 +22,5 @@
           <geometry>
             <!--box size="0.102 0.109 0.106" /-->
-            <mesh filename="package://worms_description/meshes/Pallet.stl"  scale="1 1 1"/>
+            <mesh filename="package://worms_description/meshes/pallet.stl"  scale="1 1 1"/>
           </geometry>
           <material name="Red">
@@ -31,5 +31,5 @@
           <origin xyz="0 0 0" rpy="0 0 0" />
           <geometry>
-            <mesh filename="package://worms_description/meshes/Pallet.stl"  scale="1 1 1"/>
+            <mesh filename="package://worms_description/meshes/pallet_coll.stl"  scale="1 1 1"/>
           </geometry>
         </collision>
@@ -56,14 +56,14 @@
       <geometry>
         <!--box size="0.045 0.022 0.0325" /-->
-        <mesh filename="package://worms_description/meshes/connect.STL"  scale="1 1 1"/>
-      </geometry>
-      <material name="Grey">
-        <color rgba="0.20 0.20 0.20 1.0"/>
-      </material>
-    </visual>
-    <collision>
-      <origin xyz="0 -${connect_offset} 0" rpy="0 0 0"  />
-      <geometry>
-        <mesh filename="package://worms_description/meshes/connect_coll.STL"  scale="1 1 1"/>
+        <mesh filename="package://worms_description/meshes/UIB.STL"  scale="1 1 1"/>
+      </geometry>
+      <material name="Grey">
+        <color rgba="0.20 0.20 0.20 1.0"/>
+      </material>
+    </visual>
+    <collision>
+      <origin xyz="0 -${connect_offset} 0" rpy="0 0 0"  />
+      <geometry>
+        <mesh filename="package://worms_description/meshes/UIB.STL"  scale="1 1 1"/>
       </geometry>
     </collision>
@@ -79,14 +79,14 @@
       <geometry>
         <!--box size="0.045 0.022 0.0325" /-->
-        <mesh filename="package://worms_description/meshes/connect.STL"  scale="1 1 1"/>
-      </geometry>
-      <material name="Grey">
-        <color rgba="0.20 0.20 0.20 1.0"/>
-      </material>
-    </visual>
-    <collision>
-      <origin xyz="0 -${connect_offset} 0" rpy="0 0 0"  />
-      <geometry>
-        <mesh filename="package://worms_description/meshes/connect_coll.STL"  scale="1 1 1"/>
+        <mesh filename="package://worms_description/meshes/end_effector.STL"  scale="1 1 1"/>
+      </geometry>
+      <material name="Grey">
+        <color rgba="0.20 0.20 0.20 1.0"/>
+      </material>
+    </visual>
+    <collision>
+      <origin xyz="0 -${connect_offset} 0" rpy="0 0 0"  />
+      <geometry>
+        <mesh filename="package://worms_description/meshes/end_effector.STL"  scale="1 1 1"/>
       </geometry>
     </collision>
@@ -102,14 +102,14 @@
       <geometry>
         <!--box size="0.045 0.022 0.0325" /-->
-        <mesh filename="package://worms_description/meshes/thigh_l.STL"  scale="1 1 1"/>
-      </geometry>
-      <material name="Grey">
-        <color rgba="0.20 0.20 0.20 1.0"/>
-      </material>
-    </visual>
-    <collision>
-      <origin xyz="0 0 0" rpy="0 0 0"  />
-      <geometry>
-        <mesh filename="package://worms_description/meshes/thigh_l_coll.STL"  scale="1 1 1"/>
+        <mesh filename="package://worms_description/meshes/thigh.STL"  scale="1 1 1"/>
+      </geometry>
+      <material name="Grey">
+        <color rgba="0.20 0.20 0.20 1.0"/>
+      </material>
+    </visual>
+    <collision>
+      <origin xyz="0 0 0" rpy="0 0 0"  />
+      <geometry>
+        <mesh filename="package://worms_description/meshes/thigh.STL"  scale="1 1 1"/>
       </geometry>
     </collision>
@@ -125,14 +125,14 @@
       <geometry>
         <!--box size="0.045 0.022 0.0325" /-->
-        <mesh filename="package://worms_description/meshes/tibia_l.STL"  scale="1 1 1"/>
-      </geometry>
-      <material name="Grey">
-        <color rgba="0.20 0.20 0.20 1.0"/>
-      </material>
-    </visual>
-    <collision>
-      <origin xyz="0 0 0" rpy="0 0 0"  />
-      <geometry>
-        <mesh filename="package://worms_description/meshes/tibia_l_coll.STL"  scale="1 1 1"/>
+        <mesh filename="package://worms_description/meshes/shin.STL"  scale="1 1 1"/>
+      </geometry>
+      <material name="Grey">
+        <color rgba="0.20 0.20 0.20 1.0"/>
+      </material>
+    </visual>
+    <collision>
+      <origin xyz="0 0 0" rpy="0 0 0"  />
+      <geometry>
+        <mesh filename="package://worms_description/meshes/shin.STL"  scale="1 1 1"/>
       </geometry>
     </collision>
