Commit message: updated urdf weights

File: catkin_ws/src/worms_description/urdf/worms_urdf.xacro (robot description, xacro)
@@ -22,5 +22,6 @@
           <origin xyz="0 0 0" rpy="0 0 1.57" />
           <!-- <mass value="0.97559947"/> -->
-          <mass value="0.01"/>
+          <!--mass value="0.01"/> -->
+	  <mass value="6.0" />
           <inertia ixx="3.1081800"  ixy="-0.25460189"  ixz="2.0318174" iyy="6.3787776" iyz="0.16417863" izz="5.3316425" />
         </inertial>
@@ -59,5 +60,6 @@
     <inertial>
       <origin xyz="0 -${uib_length/2} 0" rpy="0 0 0"  />
-      <mass value="0.024357719"/>
+      <!--mass value="0.024357719"/> -->
+      <mass value="0.5"/>
      <inertia ixx="0.0051411124"  ixy="-0.00057530255"  ixz="-0.000024729049" iyy="0.0081915737" iyz="-0.000019223094" izz="0.0011379812" />
     </inertial>
@@ -81,5 +83,6 @@
     <inertial>
       <origin xyz="0 -${ee_length/2} 0" rpy="0 0 0"  />
-      <mass value="0.024357719"/>
+      <!--mass value="0.024357719"/> -->
+      <mass value = "0.5"/>
      <inertia ixx="0.0051411124"  ixy="-0.00057530255"  ixz="-0.000024729049" iyy="0.0081915737" iyz="-0.000019223094" izz="0.0011379812" />
     </inertial>
@@ -103,5 +106,6 @@
     <inertial>
       <origin xyz="0 -${coxa_length/2 + motor_diameter/2} 0" rpy="0 0 0"  />
-      <mass value="0.024357719"/>
+      <!--mass value="0.024357719"/> -->
+      <mass value="3.67"/>
      <inertia ixx="0.0051411124"  ixy="-0.00057530255"  ixz="-0.000024729049" iyy="0.0081915737" iyz="-0.000019223094" izz="0.0011379812" />
     </inertial>
@@ -125,5 +129,6 @@
     <inertial>
       <origin xyz="0 -${thigh_length/2 + motor_diameter/2} 0" rpy="0 0 0"  />
-      <mass value="0.024357719"/>
+      <!--mass value="0.024357719"/> -->
+      <mass value="3.67"/>
      <inertia ixx="0.0051411124"  ixy="-0.00057530255"  ixz="-0.000024729049" iyy="0.0081915737" iyz="-0.000019223094" izz="0.0011379812" />
     </inertial>
@@ -147,5 +152,6 @@
     <inertial>
       <origin xyz="0 -${shin_length/2 + motor_diameter/2} 0" rpy="0 0 0"  />
-      <mass value="0.024357719"/>
+      <!-- mass value="0.024357719"/> -->
+      <mass value="3.67"/>
      <inertia ixx="0.0051411124"  ixy="-0.00057530255"  ixz="-0.000024729049" iyy="0.0081915737" iyz="-0.000019223094" izz="0.0011379812" />
     </inertial>

Commit message: renamed updated mesh folder, updated component masses and dims in xacro

File: catkin_ws/src/worms_description/urdf/worms_urdf.xacro (robot description, xacro)
@@ -6,8 +6,8 @@
 <xacro:property name="uib_length" value="0.08" />
 <xacro:property name="ee_length" value="0.055" />
-<xacro:property name="coxa_length" value="0.05" />
-<xacro:property name="motor_diameter" value="0.05" />
-<xacro:property name="thigh_length" value="0.35" />
-<xacro:property name="shin_length" value="0.475" />
+<xacro:property name="coxa_length" value="0.15" />
+<xacro:property name="motor_diameter" value="0.098" />
+<xacro:property name="thigh_length" value="0.27" />
+<xacro:property name="shin_length" value="0.45" />
 <!--  Masses of WORMS-1 components (in kg)-->
 <!--  Source: https://docs.google.com/spreadsheets/d/1z4cjFRy08wv40s6Jl9g9mymmIja3-cVj/edit#gid=1875184855-->
@@ -25,4 +25,5 @@
 <!-- TODO: Update component masses and inertias -->
 <!-- TODO: Add second ee, uib, and shoe -->
+<!-- TODO: Check link length specs -->
 <xacro:macro name="worms" params="parent *origin">
       <joint name="j_worms_attachment" type="fixed">
@@ -121,5 +122,5 @@
       <origin xyz="0 -${coxa_length/2 + motor_diameter/2} 0" rpy="0 0 0"  />
       <geometry>
-        <mesh filename="package://worms_description/meshes/motor_coxa.stl"  scale="1 1 1"/>
+        <mesh filename="package://worms_description/meshes/updated_parts/motor_coxa.stl"  scale="1 1 1"/>
       </geometry>
       <material name="Grey">
@@ -130,5 +131,5 @@
       <origin xyz="0 -${coxa_length/2 + motor_diameter/2} 0" rpy="0 0 0"  />
       <geometry>
-        <mesh filename="package://worms_description/meshes/motor_coxa.stl"  scale="1 1 1"/>
+        <mesh filename="package://worms_description/meshes/updated_parts/motor_coxa.stl"  scale="1 1 1"/>
       </geometry>
     </collision>
@@ -143,5 +144,5 @@
       <origin xyz="0 -${thigh_length/2 + motor_diameter/2} 0" rpy="0 0 0"  />
       <geometry>
-        <mesh filename="package://worms_description/meshes/motor_thigh.stl"  scale="1 1 1"/>
+        <mesh filename="package://worms_description/meshes/updated_parts/motor_thigh.stl"  scale="1 1 1"/>
       </geometry>
       <material name="Grey">
@@ -152,5 +153,5 @@
       <origin xyz="0 -${thigh_length/2 + motor_diameter/2} 0" rpy="0 0 0"  />
       <geometry>
-        <mesh filename="package://worms_description/meshes/motor_thigh.stl"  scale="1 1 1"/>
+        <mesh filename="package://worms_description/meshes/updated_parts/motor_thigh.stl"  scale="1 1 1"/>
       </geometry>
     </collision>
@@ -165,5 +166,5 @@
       <origin xyz="0 -${shin_length/2 + motor_diameter/2} 0" rpy="0 0 0"  />
       <geometry>
-        <mesh filename="package://worms_description/meshes/motor_shin.stl"  scale="1 1 1"/>
+        <mesh filename="package://worms_description/meshes/updated_parts/motor_shin.stl"  scale="1 1 1"/>
       </geometry>
       <material name="Grey">
@@ -174,5 +175,5 @@
       <origin xyz="0 -${shin_length/2 + motor_diameter/2} 0" rpy="0 0 0"  />
       <geometry>
-        <mesh filename="package://worms_description/meshes/motor_shin.stl"  scale="1 1 1"/>
+        <mesh filename="package://worms_description/meshes/updated_parts/motor_shin.stl"  scale="1 1 1"/>
       </geometry>
     </collision>

Commit message: updated worms_urdf.xacro

File: catkin_ws/src/worms_description/urdf/worms_urdf.xacro (robot description, xacro)
@@ -49,5 +49,5 @@
         </visual>
         <collision>
-          <origin xyz="0 0 ${initial_z_offset}" rpy="0 0 0" />
+          <origin xyz="0 0 ${initial_z_offset}" rpy="0 0 1.57" />
           <geometry>
             <mesh filename="package://worms_description/meshes/pallet_coll.STL"  scale="1 1 1"/>
@@ -73,5 +73,5 @@
       <origin xyz="0 -${uib_length/2} 0" rpy="0 0 0"  />
       <mass value="${m_uib}"/>
-      <inertia ixx="0.0051411124"  ixy="-0.00057530255"  ixz="-0.000024729049" iyy="0.0081915737" iyz="-0.000019223094" izz="0.0011379812" />
+      <inertia ixx="0.0004167"  ixy="0.0"  ixz="0.0" iyy="0.0007417" iyz="0.0" izz="0.0007417" />
     </inertial>
     <visual>
@@ -95,5 +95,5 @@
       <origin xyz="0 -${ee_length/2} 0" rpy="0 0 0"  />
       <mass value = "${m_ee + m_motor}"/>
-      <inertia ixx="0.0051411124"  ixy="-0.00057530255"  ixz="-0.000024729049" iyy="0.0081915737" iyz="-0.000019223094" izz="0.0011379812" />
+      <inertia ixx="0.0004167"  ixy="0.0"  ixz="0.0" iyy="0.0007417" iyz="0.0" izz="0.0007417" />
     </inertial>
     <visual>
@@ -117,5 +117,5 @@
       <origin xyz="0 -${coxa_length/2 + motor_diameter/2} 0" rpy="0 0 0"  />
       <mass value="${m_coxa + m_motor}"/>
-     <inertia ixx="0.0051411124"  ixy="-0.00057530255"  ixz="-0.000024729049" iyy="0.0081915737" iyz="-0.000019223094" izz="0.0011379812" />
+      <inertia ixx="0.0004167"  ixy="0.0"  ixz="0.0" iyy="0.0007417" iyz="0.0" izz="0.0007417" />
     </inertial>
     <visual>
@@ -139,5 +139,5 @@
       <origin xyz="0 -${thigh_length/2 + motor_diameter/2} 0" rpy="0 0 0"  />
       <mass value="${m_thigh + m_motor}"/>
-     <inertia ixx="0.0051411124"  ixy="-0.00057530255"  ixz="-0.000024729049" iyy="0.0081915737" iyz="-0.000019223094" izz="0.0011379812" />
+      <inertia ixx="0.0004167"  ixy="0.0"  ixz="0.0" iyy="0.0007417" iyz="0.0" izz="0.0007417" />
     </inertial>
     <visual>
@@ -161,5 +161,5 @@
       <origin xyz="0 -${shin_length/2 + motor_diameter/2} 0" rpy="0 0 0"  />
       <mass value="${m_shin + m_motor}"/>
-      <inertia ixx="0.0051411124"  ixy="-0.00057530255"  ixz="-0.000024729049" iyy="0.0081915737" iyz="-0.000019223094" izz="0.0011379812" />
+      <inertia ixx="0.0004167"  ixy="0.0"  ixz="0.0" iyy="0.0007417" iyz="0.0" izz="0.0007417" />
     </inertial>
     <visual>

Commit message: latest experiments with walking

File: catkin_ws/src/worms_description/urdf/worms_urdf.xacro (robot description, xacro)
@@ -21,4 +21,5 @@
 <xacro:property name="m_pallet" value="7" />
 <xacro:property name="m_motor" value="0.85" />
+<xacro:property name="m_hip_structure" value="0.41" />
 <xacro:property name="m_coxa" value="0.5" />
 <xacro:property name="m_thigh" value="2" />
@@ -239,5 +240,5 @@
   <link name="hip_structure_${suffix}">
     <inertial>
-      <origin xyz="0 -${hip_structure_length + uib_ee_gap_length} 0" rpy="0 0 0"  />
+      <origin xyz="0 -${(hip_structure_length + uib_ee_gap_length)/2} 0" rpy="0 0 0"  />
       <mass value="${m_uib}"/>
       <inertia ixx="0.001999"  ixy="0.000001"  ixz="0.000001" iyy="0.001386" iyz="0.000035" izz="0.002027" />
@@ -261,5 +262,5 @@
   <link name="coxa_${suffix}">
     <inertial>
-      <origin xyz="0 0 0" rpy="0 0 0"  />
+      <origin xyz="0 -${coxa_length/2} 0" rpy="0 0 0"  />
       <mass value="${m_coxa + m_motor}"/>
       <inertia ixx="0.003441"  ixy="0.000110"  ixz="-0.000001" iyy="0.000974" iyz="-0.000027" izz="0.003627" />
@@ -283,5 +284,5 @@
   <link name="thigh_${suffix}">
     <inertial>
-      <origin xyz="0 0 0" rpy="0 0 0"  />
+      <origin xyz="0 -${thigh_length/2} 0" rpy="0 0 0"  />
       <mass value="${m_thigh + m_motor}"/>
       <inertia ixx="0.012495"  ixy="0.000134"  ixz="0.000071" iyy="0.003683" iyz="0.004692" izz="0.009695" />
@@ -305,5 +306,5 @@
   <link name="shin_${suffix}">
     <inertial>
-      <origin xyz="0 0 0" rpy="0 0 0"  />
+      <origin xyz="0 -${shin_length/2} 0" rpy="0 0 0"  />
       <mass value="${m_shin + m_motor}"/>
       <inertia ixx="0.097990"  ixy="0.0"  ixz="0.0" iyy="0.004706" iyz="0.0" izz="0.097765" />
