Commit message: removed 'phantomx' from worms description files

File: catkin_ws/src/worms_description/urdf/worms.urdf (robot description, URDF)
Before this commit: robot PhantomX, 26 links, 25 joints
Links:
- link MP_BODY: geometry collision mesh filename=package://worms_description/meshes/body_coll.STL scale=1 1 1; visual mesh filename=package://worms_description/meshes/Pallet.stl scale=1 1 1
- link c1_lf: geometry collision mesh filename=package://worms_description/meshes/connect_coll.STL scale=1 1 1; visual mesh filename=package://worms_description/meshes/connect.STL scale=1 1 1
- link c1_lm: geometry collision mesh filename=package://worms_description/meshes/connect_coll.STL scale=1 1 1; visual mesh filename=package://worms_description/meshes/connect.STL scale=1 1 1
- link c1_lr: geometry collision mesh filename=package://worms_description/meshes/connect_coll.STL scale=1 1 1; visual mesh filename=package://worms_description/meshes/connect.STL scale=1 1 1
- link c1_rf: geometry collision mesh filename=package://worms_description/meshes/connect_coll.STL scale=1 1 1; visual mesh filename=package://worms_description/meshes/connect.STL scale=1 1 1
- link c1_rm: geometry collision mesh filename=package://worms_description/meshes/connect_coll.STL scale=1 1 1; visual mesh filename=package://worms_description/meshes/connect.STL scale=1 1 1
- link c1_rr: geometry collision mesh filename=package://worms_description/meshes/connect_coll.STL scale=1 1 1; visual mesh filename=package://worms_description/meshes/connect.STL scale=1 1 1
- link c2_lf: geometry collision mesh filename=package://worms_description/meshes/connect_coll.STL scale=1 1 1; visual mesh filename=package://worms_description/meshes/connect.STL scale=1 1 1
- link c2_lm: geometry collision mesh filename=package://worms_description/meshes/connect_coll.STL scale=1 1 1; visual mesh filename=package://worms_description/meshes/connect.STL scale=1 1 1
- link c2_lr: geometry collision mesh filename=package://worms_description/meshes/connect_coll.STL scale=1 1 1; visual mesh filename=package://worms_description/meshes/connect.STL scale=1 1 1
- link c2_rf: geometry collision mesh filename=package://worms_description/meshes/connect_coll.STL scale=1 1 1; visual mesh filename=package://worms_description/meshes/connect.STL scale=1 1 1
- link c2_rm: geometry collision mesh filename=package://worms_description/meshes/connect_coll.STL scale=1 1 1; visual mesh filename=package://worms_description/meshes/connect.STL scale=1 1 1
- link c2_rr: geometry collision mesh filename=package://worms_description/meshes/connect_coll.STL scale=1 1 1; visual mesh filename=package://worms_description/meshes/connect.STL scale=1 1 1
- link thigh_lf: geometry collision mesh filename=package://worms_description/meshes/thigh_l_coll.STL scale=1 1 1; visual mesh filename=package://worms_description/meshes/thigh_l.STL scale=1 1 1
- link thigh_lm: geometry collision mesh filename=package://worms_description/meshes/thigh_l_coll.STL scale=1 1 1; visual mesh filename=package://worms_description/meshes/thigh_l.STL scale=1 1 1
- link thigh_lr: geometry collision mesh filename=package://worms_description/meshes/thigh_l_coll.STL scale=1 1 1; visual mesh filename=package://worms_description/meshes/thigh_l.STL scale=1 1 1
- link thigh_rf: geometry collision mesh filename=package://worms_description/meshes/thigh_l_coll.STL scale=1 1 1; visual mesh filename=package://worms_description/meshes/thigh_l.STL scale=1 1 1
- link thigh_rm: geometry collision mesh filename=package://worms_description/meshes/thigh_l_coll.STL scale=1 1 1; visual mesh filename=package://worms_description/meshes/thigh_l.STL scale=1 1 1
- link thigh_rr: geometry collision mesh filename=package://worms_description/meshes/thigh_l_coll.STL scale=1 1 1; visual mesh filename=package://worms_description/meshes/thigh_l.STL scale=1 1 1
- link tibia_lf: geometry collision mesh filename=package://worms_description/meshes/tibia_l_coll.STL scale=1 1 1; visual mesh filename=package://worms_description/meshes/tibia_l.STL scale=1 1 1
- link tibia_lm: geometry collision mesh filename=package://worms_description/meshes/tibia_l_coll.STL scale=1 1 1; visual mesh filename=package://worms_description/meshes/tibia_l.STL scale=1 1 1
- link tibia_lr: geometry collision mesh filename=package://worms_description/meshes/tibia_l_coll.STL scale=1 1 1; visual mesh filename=package://worms_description/meshes/tibia_l.STL scale=1 1 1
- link tibia_rf: geometry collision mesh filename=package://worms_description/meshes/tibia_l_coll.STL scale=1 1 1; visual mesh filename=package://worms_description/meshes/tibia_l.STL scale=1 1 1
- link tibia_rm: geometry collision mesh filename=package://worms_description/meshes/tibia_l_coll.STL scale=1 1 1; visual mesh filename=package://worms_description/meshes/tibia_l.STL scale=1 1 1
- link tibia_rr: geometry collision mesh filename=package://worms_description/meshes/tibia_l_coll.STL scale=1 1 1; visual mesh filename=package://worms_description/meshes/tibia_l.STL scale=1 1 1
Joints:
- removed joint j_phantomx_attachment
- added joint j_worms_attachment: type fixed, parent base_link, child MP_BODY, origin xyz=0 0 0 rpy=0 0 0

File: catkin_ws/src/worms_description/urdf/worms_urdf.xacro (robot description, xacro)
@@ -4,6 +4,6 @@
 <xacro:property name="thigh_offset_y" value="-0.0645" />
 <xacro:property name="thigh_offset_z" value="-0.0145" />
-<xacro:macro name="phantomx" params="parent *origin">
-      <joint name="j_phantomx_attachment" type="fixed">
+<xacro:macro name="worms" params="parent *origin">
+      <joint name="j_worms_attachment" type="fixed">
         <parent link="${parent}"/>
         <child link="MP_BODY"/>
@@ -21,5 +21,5 @@
           <geometry>
             <!--box size="0.102 0.109 0.106" /-->
-            <mesh filename="package://phantomx_description/meshes/body.STL"  scale="1 1 1"/>
+            <mesh filename="package://worms_description/meshes/body.STL"  scale="1 1 1"/>
           </geometry>
           <material name="Grey">
@@ -30,5 +30,5 @@
           <origin xyz="0 0 0" rpy="0 0 0" />
           <geometry>
-            <mesh filename="package://phantomx_description/meshes/body_coll.STL"  scale="1 1 1"/>
+            <mesh filename="package://worms_description/meshes/body_coll.STL"  scale="1 1 1"/>
           </geometry>
         </collision>
@@ -55,14 +55,14 @@
       <geometry>
         <!--box size="0.045 0.022 0.0325" /-->
-        <mesh filename="package://phantomx_description/meshes/connect.STL"  scale="1 1 1"/>
-      </geometry>
-      <material name="Grey">
-        <color rgba="0.20 0.20 0.20 1.0"/>
-      </material>
-    </visual>
-    <collision>
-      <origin xyz="0 -${connect_offset} 0" rpy="0 0 0"  />
-      <geometry>
-        <mesh filename="package://phantomx_description/meshes/connect_coll.STL"  scale="1 1 1"/>
+        <mesh filename="package://worms_description/meshes/connect.STL"  scale="1 1 1"/>
+      </geometry>
+      <material name="Grey">
+        <color rgba="0.20 0.20 0.20 1.0"/>
+      </material>
+    </visual>
+    <collision>
+      <origin xyz="0 -${connect_offset} 0" rpy="0 0 0"  />
+      <geometry>
+        <mesh filename="package://worms_description/meshes/connect_coll.STL"  scale="1 1 1"/>
       </geometry>
     </collision>
@@ -78,14 +78,14 @@
       <geometry>
         <!--box size="0.045 0.022 0.0325" /-->
-        <mesh filename="package://phantomx_description/meshes/connect.STL"  scale="1 1 1"/>
-      </geometry>
-      <material name="Grey">
-        <color rgba="0.20 0.20 0.20 1.0"/>
-      </material>
-    </visual>
-    <collision>
-      <origin xyz="0 -${connect_offset} 0" rpy="0 0 0"  />
-      <geometry>
-        <mesh filename="package://phantomx_description/meshes/connect_coll.STL"  scale="1 1 1"/>
+        <mesh filename="package://worms_description/meshes/connect.STL"  scale="1 1 1"/>
+      </geometry>
+      <material name="Grey">
+        <color rgba="0.20 0.20 0.20 1.0"/>
+      </material>
+    </visual>
+    <collision>
+      <origin xyz="0 -${connect_offset} 0" rpy="0 0 0"  />
+      <geometry>
+        <mesh filename="package://worms_description/meshes/connect_coll.STL"  scale="1 1 1"/>
       </geometry>
     </collision>
@@ -101,14 +101,14 @@
       <geometry>
         <!--box size="0.045 0.022 0.0325" /-->
-        <mesh filename="package://phantomx_description/meshes/thigh_l.STL"  scale="1 1 1"/>
-      </geometry>
-      <material name="Grey">
-        <color rgba="0.20 0.20 0.20 1.0"/>
-      </material>
-    </visual>
-    <collision>
-      <origin xyz="0 0 0" rpy="0 0 0"  />
-      <geometry>
-        <mesh filename="package://phantomx_description/meshes/thigh_l_coll.STL"  scale="1 1 1"/>
+        <mesh filename="package://worms_description/meshes/thigh_l.STL"  scale="1 1 1"/>
+      </geometry>
+      <material name="Grey">
+        <color rgba="0.20 0.20 0.20 1.0"/>
+      </material>
+    </visual>
+    <collision>
+      <origin xyz="0 0 0" rpy="0 0 0"  />
+      <geometry>
+        <mesh filename="package://worms_description/meshes/thigh_l_coll.STL"  scale="1 1 1"/>
       </geometry>
     </collision>
@@ -124,14 +124,14 @@
       <geometry>
         <!--box size="0.045 0.022 0.0325" /-->
-        <mesh filename="package://phantomx_description/meshes/tibia_l.STL"  scale="1 1 1"/>
-      </geometry>
-      <material name="Grey">
-        <color rgba="0.20 0.20 0.20 1.0"/>
-      </material>
-    </visual>
-    <collision>
-      <origin xyz="0 0 0" rpy="0 0 0"  />
-      <geometry>
-        <mesh filename="package://phantomx_description/meshes/tibia_l_coll.STL"  scale="1 1 1"/>
+        <mesh filename="package://worms_description/meshes/tibia_l.STL"  scale="1 1 1"/>
+      </geometry>
+      <material name="Grey">
+        <color rgba="0.20 0.20 0.20 1.0"/>
+      </material>
+    </visual>
+    <collision>
+      <origin xyz="0 0 0" rpy="0 0 0"  />
+      <geometry>
+        <mesh filename="package://worms_description/meshes/tibia_l_coll.STL"  scale="1 1 1"/>
       </geometry>
     </collision>

Commit message: added reset_sim node to worms_gazebo, updated worms_urdf.xacro

File: catkin_ws/src/worms_description/urdf/worms.urdf (robot description, URDF)
Before this commit: robot worms, 26 links, 25 joints
Links:
- link MP_BODY: mass 0.97559947 -> 0.01; geometry collision mesh filename=package://worms_description/meshes/Pallet.stl scale=1 1 1; visual mesh filename=package://worms_description/meshes/Pallet.stl scale=1 1 1
Joints:
- joint j_c1_lf: origin xyz=0.1248 0.06164  0.001116 rpy=0 4.7123 2.356194490192345 -> xyz=0.1248 0.3175 0.001116 rpy=0 4.7123 2.356194490192345
- joint j_c1_lm: origin xyz=0 0.1034  0.001116 rpy=0 4.7123 3.14159 -> xyz=0 0.3175  0.001116 rpy=0 4.7123 3.14159
- joint j_c1_lr: origin xyz=-0.1248 0.06164  0.001116 rpy=0 4.7123 3.9269908169872414 -> xyz=-0.1248 0.3175  0.001116 rpy=0 4.7123 3.9269908169872414
- joint j_c1_rf: origin xyz=0.1248 -0.06164  0.001116 rpy=0 4.7123 0.7853981633974483 -> xyz=0.1248 -0.3175 0.001116 rpy=0 4.7123 0.7853981633974483
- joint j_c1_rm: origin xyz=0 -0.1034  0.001116 rpy=0 4.7123 0 -> xyz=0 -0.3175  0.001116 rpy=0 4.7123 0
- joint j_c1_rr: origin xyz=-0.1248 -0.06164  0.001116 rpy=0 4.7123 -0.7853981633974483 -> xyz=-0.1248 -0.3175  0.001116 rpy=0 4.7123 -0.7853981633974483

File: catkin_ws/src/worms_description/urdf/worms_urdf.xacro (robot description, xacro)
@@ -13,5 +13,6 @@
         <inertial>
           <origin xyz="0 0 0" />
-          <mass value="0.97559947"/>
+          <!-- <mass value="0.97559947"/> -->
+          <mass value="0.01"/>
           <inertia ixx="3.1081800"  ixy="-0.25460189"  ixz="2.0318174" iyy="6.3787776" iyz="0.16417863" izz="5.3316425" />
         </inertial>
@@ -30,5 +31,5 @@
           <origin xyz="0 0 0" rpy="0 0 0" />
           <geometry>
-            <mesh filename="package://worms_description/meshes/body_coll.STL"  scale="1 1 1"/>
+            <mesh filename="package://worms_description/meshes/Pallet.stl"  scale="1 1 1"/>
           </geometry>
         </collision>
@@ -37,10 +38,10 @@
         <material>Gazebo/Red</material>
       </gazebo>
-    <xacro:leg_l xyz="0.1248 -0.06164  0.001116"  rpy="0 4.7123 0.7853981633974483" suffix="rf"/>
-    <xacro:leg_l xyz="0 -0.1034  0.001116"  rpy="0 4.7123 0" suffix="rm"/>
-    <xacro:leg_l xyz="-0.1248 -0.06164  0.001116"  rpy="0 4.7123 -0.7853981633974483" suffix="rr"/>
-    <xacro:leg_l xyz="0.1248 0.06164  0.001116"  rpy="0 4.7123 2.356194490192345" suffix="lf"/>
-    <xacro:leg_l xyz="0 0.1034  0.001116"  rpy="0 4.7123 3.14159" suffix="lm"/>
-    <xacro:leg_l xyz="-0.1248 0.06164  0.001116"  rpy="0 4.7123 3.9269908169872414" suffix="lr"/>
+    <xacro:leg_l xyz="0.1248 -0.3175 0.001116"  rpy="0 4.7123 0.7853981633974483" suffix="rf"/>
+    <xacro:leg_l xyz="0 -0.3175  0.001116"  rpy="0 4.7123 0" suffix="rm"/>
+    <xacro:leg_l xyz="-0.1248 -0.3175  0.001116"  rpy="0 4.7123 -0.7853981633974483" suffix="rr"/>
+    <xacro:leg_l xyz="0.1248 0.3175 0.001116"  rpy="0 4.7123 2.356194490192345" suffix="lf"/>
+    <xacro:leg_l xyz="0 0.3175  0.001116"  rpy="0 4.7123 3.14159" suffix="lm"/>
+    <xacro:leg_l xyz="-0.1248 0.3175  0.001116"  rpy="0 4.7123 3.9269908169872414" suffix="lr"/>
 </xacro:macro>
  <xacro:macro name="leg_l" params="xyz rpy suffix">
