Commit message: updated worms urdf and xacro

File: catkin_ws/src/worms_description/urdf/worms.urdf (robot description, URDF)
Before this commit: robot worms, 26 links, 25 joints
Links:
- removed link c1_lf
- removed link c1_lm
- removed link c1_lr
- removed link c1_rf
- removed link c1_rm
- removed link c1_rr
- removed link c2_lf
- removed link c2_lm
- removed link c2_lr
- removed link c2_rf
- removed link c2_rm
- removed link c2_rr
- removed link thigh_lf
- removed link thigh_lm
- removed link thigh_lr
- removed link thigh_rf
- removed link thigh_rm
- removed link thigh_rr
- removed link tibia_lf
- removed link tibia_lm
- removed link tibia_lr
- removed link tibia_rf
- removed link tibia_rm
- removed link tibia_rr
- added link ee_lf, mass 0.024357719; collision mesh filename=package://worms_description/meshes/end_effector.STL scale=1 1 1; visual mesh filename=package://worms_description/meshes/end_effector.STL scale=1 1 1
- added link ee_lm, mass 0.024357719; collision mesh filename=package://worms_description/meshes/end_effector.STL scale=1 1 1; visual mesh filename=package://worms_description/meshes/end_effector.STL scale=1 1 1
- added link ee_lr, mass 0.024357719; collision mesh filename=package://worms_description/meshes/end_effector.STL scale=1 1 1; visual mesh filename=package://worms_description/meshes/end_effector.STL scale=1 1 1
- added link ee_rf, mass 0.024357719; collision mesh filename=package://worms_description/meshes/end_effector.STL scale=1 1 1; visual mesh filename=package://worms_description/meshes/end_effector.STL scale=1 1 1
- added link ee_rm, mass 0.024357719; collision mesh filename=package://worms_description/meshes/end_effector.STL scale=1 1 1; visual mesh filename=package://worms_description/meshes/end_effector.STL scale=1 1 1
- added link ee_rr, mass 0.024357719; collision mesh filename=package://worms_description/meshes/end_effector.STL scale=1 1 1; visual mesh filename=package://worms_description/meshes/end_effector.STL scale=1 1 1
- added link uib_lf, mass 0.024357719; collision mesh filename=package://worms_description/meshes/UIB.STL scale=1 1 1; visual mesh filename=package://worms_description/meshes/UIB.STL scale=1 1 1
- added link uib_lm, mass 0.024357719; collision mesh filename=package://worms_description/meshes/UIB.STL scale=1 1 1; visual mesh filename=package://worms_description/meshes/UIB.STL scale=1 1 1
- added link uib_lr, mass 0.024357719; collision mesh filename=package://worms_description/meshes/UIB.STL scale=1 1 1; visual mesh filename=package://worms_description/meshes/UIB.STL scale=1 1 1
- added link uib_rf, mass 0.024357719; collision mesh filename=package://worms_description/meshes/UIB.STL scale=1 1 1; visual mesh filename=package://worms_description/meshes/UIB.STL scale=1 1 1
- added link uib_rm, mass 0.024357719; collision mesh filename=package://worms_description/meshes/UIB.STL scale=1 1 1; visual mesh filename=package://worms_description/meshes/UIB.STL scale=1 1 1
- added link uib_rr, mass 0.024357719; collision mesh filename=package://worms_description/meshes/UIB.STL scale=1 1 1; visual mesh filename=package://worms_description/meshes/UIB.STL scale=1 1 1
Joints:
- removed joint j_c1_lf
- removed joint j_c1_lm
- removed joint j_c1_lr
- removed joint j_c1_rf
- removed joint j_c1_rm
- removed joint j_c1_rr
- removed joint j_c2_lf
- removed joint j_c2_lm
- removed joint j_c2_lr
- removed joint j_c2_rf
- removed joint j_c2_rm
- removed joint j_c2_rr
- removed joint j_thigh_lf
- removed joint j_thigh_lm
- removed joint j_thigh_lr
- removed joint j_thigh_rf
- removed joint j_thigh_rm
- removed joint j_thigh_rr
- removed joint j_tibia_lf
- removed joint j_tibia_lm
- removed joint j_tibia_lr
- removed joint j_tibia_rf
- removed joint j_tibia_rm
- removed joint j_tibia_rr
- added joint j_ee_lf: type fixed, parent uib_lf, child ee_lf, origin xyz=0.4330 0.2500 0.0000 rpy=0 0 2.09, axis 1 0 0, limit lower=-2.6179939 upper=2.6179939 effort=2.8 velocity=5.6548668
- added joint j_ee_lm: type fixed, parent uib_lm, child ee_lm, origin xyz=0.0000 0.5000 0.0000 rpy=0 0 3.14, axis 1 0 0, limit lower=-2.6179939 upper=2.6179939 effort=2.8 velocity=5.6548668
- added joint j_ee_lr: type fixed, parent uib_lr, child ee_lr, origin xyz=-0.4330 0.2500 0.0000 rpy=0 0 4.180000000000001, axis 1 0 0, limit lower=-2.6179939 upper=2.6179939 effort=2.8 velocity=5.6548668
- added joint j_ee_rf: type fixed, parent uib_rf, child ee_rf, origin xyz=0.4330 -0.2500 0.0000 rpy=0 0 1.05, axis 1 0 0, limit lower=-2.6179939 upper=2.6179939 effort=2.8 velocity=5.6548668
- added joint j_ee_rm: type fixed, parent uib_rm, child ee_rm, origin xyz=0.0000 -0.5000 0.0000 rpy=0 0 0.0, axis 1 0 0, limit lower=-2.6179939 upper=2.6179939 effort=2.8 velocity=5.6548668
- added joint j_ee_rr: type fixed, parent uib_rr, child ee_rr, origin xyz=-0.4330 -0.2500 0.0000 rpy=0 0 -1.0400000000000003, axis 1 0 0, limit lower=-2.6179939 upper=2.6179939 effort=2.8 velocity=5.6548668
- added joint j_uib_lf: type fixed, parent MP_BODY, child uib_lf, origin xyz=0.4330 0.2500 0.0000 rpy=0 0 2.09, axis 1 0 0, limit lower=-2.6179939 upper=2.6179939 effort=2.8 velocity=5.6548668
- added joint j_uib_lm: type fixed, parent MP_BODY, child uib_lm, origin xyz=0.0000 0.5000 0.0000 rpy=0 0 3.14, axis 1 0 0, limit lower=-2.6179939 upper=2.6179939 effort=2.8 velocity=5.6548668
- added joint j_uib_lr: type fixed, parent MP_BODY, child uib_lr, origin xyz=-0.4330 0.2500 0.0000 rpy=0 0 4.180000000000001, axis 1 0 0, limit lower=-2.6179939 upper=2.6179939 effort=2.8 velocity=5.6548668
- added joint j_uib_rf: type fixed, parent MP_BODY, child uib_rf, origin xyz=0.4330 -0.2500 0.0000 rpy=0 0 1.05, axis 1 0 0, limit lower=-2.6179939 upper=2.6179939 effort=2.8 velocity=5.6548668
- added joint j_uib_rm: type fixed, parent MP_BODY, child uib_rm, origin xyz=0.0000 -0.5000 0.0000 rpy=0 0 0.0, axis 1 0 0, limit lower=-2.6179939 upper=2.6179939 effort=2.8 velocity=5.6548668
- added joint j_uib_rr: type fixed, parent MP_BODY, child uib_rr, origin xyz=-0.4330 -0.2500 0.0000 rpy=0 0 -1.0400000000000003, axis 1 0 0, limit lower=-2.6179939 upper=2.6179939 effort=2.8 velocity=5.6548668

File: catkin_ws/src/worms_description/urdf/worms_urdf.xacro (robot description, xacro)
@@ -1,5 +1,6 @@
 <?xml version="1.0" ?>
 <robot xmlns:xacro="http://www.ros.org/wiki/xacro">
-<xacro:property name="connect_offset" value="0.02633" />
+<xacro:property name="uib_connect_offset" value="0.04" />
+<xacro:property name="ee_connect_offset" value="0.0275" />
 <xacro:property name="thigh_offset_y" value="-0.0645" />
 <xacro:property name="thigh_offset_z" value="-0.0145" />
@@ -12,5 +13,5 @@
       <link name="MP_BODY">
         <inertial>
-          <origin xyz="0 0 0" />
+          <origin xyz="0 0 0" rpy="0 0 1.57" />
           <!-- <mass value="0.97559947"/> -->
           <mass value="0.01"/>
@@ -19,8 +20,8 @@
         <visual>
           <!--origin xyz="-0.0235 0 -0.03525" rpy="0 0 0" /-->
-          <origin xyz="0 0 0" rpy="0 0 0" />
+          <origin xyz="0 0 0" rpy="0 0 1.57" />
           <geometry>
             <!--box size="0.102 0.109 0.106" /-->
-            <mesh filename="package://worms_description/meshes/pallet.stl"  scale="1 1 1"/>
+            <mesh filename="package://worms_description/meshes/pallet.STL"  scale="1 1 1"/>
           </geometry>
           <material name="Red">
@@ -31,5 +32,5 @@
           <origin xyz="0 0 0" rpy="0 0 0" />
           <geometry>
-            <mesh filename="package://worms_description/meshes/pallet_coll.stl"  scale="1 1 1"/>
+            <mesh filename="package://worms_description/meshes/pallet_coll.STL"  scale="1 1 1"/>
           </geometry>
         </collision>
@@ -38,20 +39,20 @@
         <material>Gazebo/Red</material>
       </gazebo>
-    <xacro:leg_l xyz="0.1248 -0.3175 0.001116"  rpy="0 4.7123 0.7853981633974483" suffix="rf"/>
-    <xacro:leg_l xyz="0 -0.3175  0.001116"  rpy="0 4.7123 0" suffix="rm"/>
-    <xacro:leg_l xyz="-0.1248 -0.3175  0.001116"  rpy="0 4.7123 -0.7853981633974483" suffix="rr"/>
-    <xacro:leg_l xyz="0.1248 0.3175 0.001116"  rpy="0 4.7123 2.356194490192345" suffix="lf"/>
-    <xacro:leg_l xyz="0 0.3175  0.001116"  rpy="0 4.7123 3.14159" suffix="lm"/>
-    <xacro:leg_l xyz="-0.1248 0.3175  0.001116"  rpy="0 4.7123 3.9269908169872414" suffix="lr"/>
+    <xacro:leg_l xyz="0.4330 -0.2500 0.0000"  rpy="0 0 ${-0.52 + 1.57}" suffix="rf"/>
+    <xacro:leg_l xyz="0.0000 -0.5000 0.0000"  rpy="0 0 ${-1.57 + 1.57}" suffix="rm"/>
+    <xacro:leg_l xyz="-0.4330 -0.2500 0.0000"  rpy="0 0 ${-1.57 -1.04 + 1.57}" suffix="rr"/>
+    <xacro:leg_l xyz="0.4330 0.2500 0.0000"  rpy="0 0 ${0.52 + 1.57}" suffix="lf"/>
+    <xacro:leg_l xyz="0.0000 0.5000 0.0000"  rpy="0 0 ${1.57 + 1.57}" suffix="lm"/>
+    <xacro:leg_l xyz="-0.4330 0.2500 0.0000"  rpy="0 0 ${1.57 + 1.04 + 1.57}" suffix="lr"/>
 </xacro:macro>
  <xacro:macro name="leg_l" params="xyz rpy suffix">
-  <link name="c1_${suffix}">
-    <inertial>
-      <origin xyz="0 -${connect_offset} 0" rpy="0 0 0"  />
-      <mass value="0.024357719"/>
-     <inertia ixx="0.0051411124"  ixy="-0.00057530255"  ixz="-0.000024729049" iyy="0.0081915737" iyz="-0.000019223094" izz="0.0011379812" />
-    </inertial>
-    <visual>
-      <origin xyz="0 -0.0252 0" rpy="0 0 0"  />
+  <link name="uib_${suffix}">
+    <inertial>
+      <origin xyz="${uib_connect_offset} 0 0" rpy="0 0 0"  />
+      <mass value="0.024357719"/>
+     <inertia ixx="0.0051411124"  ixy="-0.00057530255"  ixz="-0.000024729049" iyy="0.0081915737" iyz="-0.000019223094" izz="0.0011379812" />
+    </inertial>
+    <visual>
+      <origin xyz="2 0 0" rpy="0 0 0"  />
       <geometry>
         <!--box size="0.045 0.022 0.0325" /-->
@@ -63,5 +64,5 @@
     </visual>
     <collision>
-      <origin xyz="0 -${connect_offset} 0" rpy="0 0 0"  />
+      <origin xyz="${uib_connect_offset} 0 0" rpy="0 0 0"  />
       <geometry>
         <mesh filename="package://worms_description/meshes/UIB.STL"  scale="1 1 1"/>
@@ -69,7 +70,7 @@
     </collision>
   </link>
-  <link name="c2_${suffix}">
-    <inertial>
-      <origin xyz="0 -${connect_offset} 0" rpy="0 0 0"  />
+  <link name="ee_${suffix}">
+    <inertial>
+      <origin xyz="${ee_connect_offset} 0 0" rpy="0 0 0"  />
       <mass value="0.024357719"/>
      <inertia ixx="0.0051411124"  ixy="-0.00057530255"  ixz="-0.000024729049" iyy="0.0081915737" iyz="-0.000019223094" izz="0.0011379812" />
@@ -86,7 +87,29 @@
     </visual>
     <collision>
+      <origin xyz="${ee_connect_offset} 0 0" rpy="0 0 0"  />
+      <geometry>
+        <mesh filename="package://worms_description/meshes/end_effector.STL"  scale="1 1 1"/>
+      </geometry>
+    </collision>
+  </link>
+  <!-- <link name="coxa_${suffix}">
+    <inertial>
       <origin xyz="0 -${connect_offset} 0" rpy="0 0 0"  />
-      <geometry>
-        <mesh filename="package://worms_description/meshes/end_effector.STL"  scale="1 1 1"/>
+      <mass value="0.024357719"/>
+     <inertia ixx="0.0051411124"  ixy="-0.00057530255"  ixz="-0.000024729049" iyy="0.0081915737" iyz="-0.000019223094" izz="0.0011379812" />
+    </inertial>
+    <visual>
+      <origin xyz="0 -0.0252 0" rpy="0 0 0"  />
+      <geometry>
+        <mesh filename="package://worms_description/meshes/coxa.STL"  scale="1 1 1"/>
+      </geometry>
+      <material name="Grey">
+        <color rgba="0.20 0.20 0.20 1.0"/>
+      </material>
+    </visual>
+    <collision>
+      <origin xyz="0 -${connect_offset} 0" rpy="0 0 0"  />
+      <geometry>
+        <mesh filename="package://worms_description/meshes/coxa.STL"  scale="1 1 1"/>
       </geometry>
     </collision>
@@ -101,5 +124,4 @@
       <origin xyz="0 0 0" rpy="0 0 0"  />
       <geometry>
-        <!--box size="0.045 0.022 0.0325" /-->
         <mesh filename="package://worms_description/meshes/thigh.STL"  scale="1 1 1"/>
       </geometry>
@@ -115,14 +137,13 @@
     </collision>
   </link>
-  <link name="tibia_${suffix}">
-    <inertial>
-      <origin xyz="0 0 0" rpy="0 0 0"  />
-      <mass value="0.024357719"/>
-     <inertia ixx="0.0051411124"  ixy="-0.00057530255"  ixz="-0.000024729049" iyy="0.0081915737" iyz="-0.000019223094" izz="0.0011379812" />
-    </inertial>
-    <visual>
-      <origin xyz="0 0 0" rpy="0 0 0"  />
-      <geometry>
-        <!--box size="0.045 0.022 0.0325" /-->
+  <link name="shin_${suffix}">
+    <inertial>
+      <origin xyz="0 0 0" rpy="0 0 0"  />
+      <mass value="0.024357719"/>
+     <inertia ixx="0.0051411124"  ixy="-0.00057530255"  ixz="-0.000024729049" iyy="0.0081915737" iyz="-0.000019223094" izz="0.0011379812" />
+    </inertial>
+    <visual>
+      <origin xyz="0 0 0" rpy="0 0 0"  />
+      <geometry>
         <mesh filename="package://worms_description/meshes/shin.STL"  scale="1 1 1"/>
       </geometry>
@@ -137,19 +158,29 @@
       </geometry>
     </collision>
-  </link>
-  <joint name="j_c1_${suffix}" type="revolute">
+  </link> -->
+  <!-- Joint definitions -->
+  <joint name="j_uib_${suffix}" type="fixed">
     <parent link="MP_BODY"/>
-    <child link="c1_${suffix}"/>
+    <child link="uib_${suffix}"/>
     <origin xyz="${xyz}" rpy="${rpy}" />
     <axis xyz="1 0 0" />
     <limit effort="2.8" velocity="5.6548668" lower="-2.6179939" upper="2.6179939" />
   </joint>
-  <joint name="j_c2_${suffix}" type="fixed">
-    <parent link="c1_${suffix}"/>
-    <child link="c2_${suffix}"/>
-    <origin xyz="0 -0.054 0" rpy="0 1.5704 3.14159" />
+  <joint name="j_ee_${suffix}" type="fixed">
+    <parent link="uib_${suffix}"/>
+    <child link="ee_${suffix}"/>
+    <origin xyz="${xyz}" rpy="${rpy}" />
+    <axis xyz="1 0 0" />
+    <limit effort="2.8" velocity="5.6548668" lower="-2.6179939" upper="2.6179939" />
+  </joint>
+  <!-- <joint name="j_coxa_${suffix}" type="revolute">
+    <parent link="ee_${suffix}"/>
+    <child link="coxa_${suffix}"/>
+    <origin xyz="${xyz}" rpy="${rpy}" />
+    <axis xyz="1 0 0" />
+    <limit effort="2.8" velocity="5.6548668" lower="-2.6179939" upper="2.6179939" />
   </joint>
   <joint name="j_thigh_${suffix}" type="revolute">
-    <parent link="c2_${suffix}"/>
+    <parent link="coxa_${suffix}"/>
     <child link="thigh_${suffix}"/>
     <origin xyz="0 0 0" rpy=" 0 3.14159 3.14159" />
@@ -157,17 +188,18 @@
     <limit effort="2.8" velocity="5.6548668" lower="-2.6179939" upper="2.6179939" />
   </joint>
-  <joint name="j_tibia_${suffix}" type="revolute">
+  <joint name="j_shin_${suffix}" type="revolute">
     <parent link="thigh_${suffix}"/>
-    <child link="tibia_${suffix}"/>
+    <child link="shin_${suffix}"/>
     <origin xyz="0 ${thigh_offset_y} ${thigh_offset_z}" rpy="-1.5707 0 3.14159" />
     <axis xyz="1 0 0" />
     <limit effort="2.8" velocity="5.6548668" lower="-2.6179939" upper="2.6179939" />
-  </joint>
-   <transmission name="t_c1_${suffix}">
+  </joint> -->
+  <!-- Joint transmission definitions -->
+   <!-- <transmission name="t_coxa_${suffix}">
     <type>transmission_interface/SimpleTransmission</type>
-    <joint name="j_c1_${suffix}">
+    <joint name="j_coxa_${suffix}">
       <hardwareInterface>EffortJointInterface</hardwareInterface>
     </joint>
-    <actuator name="m_c1_${suffix}">
+    <actuator name="m_coxa_${suffix}">
       <hardwareInterface>EffortJointInterface</hardwareInterface>
       <mechanicalReduction>1</mechanicalReduction>
@@ -184,18 +216,22 @@
     </actuator>
   </transmission>
-   <transmission name="t_tibia_${suffix}">
+   <transmission name="t_shin_${suffix}">
     <type>transmission_interface/SimpleTransmission</type>
-    <joint name="j_tibia_${suffix}">
+    <joint name="j_shin_${suffix}">
       <hardwareInterface>EffortJointInterface</hardwareInterface>
     </joint>
-    <actuator name="m_tibia_${suffix}">
+    <actuator name="m_shin_${suffix}">
       <hardwareInterface>EffortJointInterface</hardwareInterface>
       <mechanicalReduction>1</mechanicalReduction>
     </actuator>
-  </transmission>
-  <gazebo reference="c1_${suffix}">
-    <material>Gazebo/Grey</material>
-  </gazebo>
-  <gazebo reference="c2_${suffix}">
+  </transmission> -->
+<!-- Gazebo material definitions -->
+  <gazebo reference="uib_${suffix}">
+    <material>Gazebo/Grey</material>
+  </gazebo>
+  <gazebo reference="ee_${suffix}">
+    <material>Gazebo/Grey</material>
+  </gazebo>
+  <gazebo reference="coxa_${suffix}">
     <material>Gazebo/Grey</material>
   </gazebo>
@@ -203,5 +239,5 @@
     <material>Gazebo/Grey</material>
   </gazebo>
-  <gazebo reference="tibia_${suffix}">
+  <gazebo reference="shin_${suffix}">
     <material>Gazebo/Grey</material>
   </gazebo>
