Commit message: updated worms urdf and xacro (uib, ee, coxa)

File: catkin_ws/src/worms_description/urdf/worms.urdf (robot description, URDF)
Before this commit: robot worms, 14 links, 13 joints
Links:
- added link coxa_lf, mass 0.024357719; collision mesh filename=package://worms_description/meshes/coxa.STL scale=1 1 1; visual mesh filename=package://worms_description/meshes/coxa.STL scale=1 1 1
- added link coxa_lm, mass 0.024357719; collision mesh filename=package://worms_description/meshes/coxa.STL scale=1 1 1; visual mesh filename=package://worms_description/meshes/coxa.STL scale=1 1 1
- added link coxa_lr, mass 0.024357719; collision mesh filename=package://worms_description/meshes/coxa.STL scale=1 1 1; visual mesh filename=package://worms_description/meshes/coxa.STL scale=1 1 1
- added link coxa_rf, mass 0.024357719; collision mesh filename=package://worms_description/meshes/coxa.STL scale=1 1 1; visual mesh filename=package://worms_description/meshes/coxa.STL scale=1 1 1
- added link coxa_rm, mass 0.024357719; collision mesh filename=package://worms_description/meshes/coxa.STL scale=1 1 1; visual mesh filename=package://worms_description/meshes/coxa.STL scale=1 1 1
- added link coxa_rr, mass 0.024357719; collision mesh filename=package://worms_description/meshes/coxa.STL scale=1 1 1; visual mesh filename=package://worms_description/meshes/coxa.STL scale=1 1 1
Joints:
- added joint j_coxa_lf: type revolute, parent ee_lf, child coxa_lf, origin xyz=0 -0.10500000000000001 0 rpy=0 0 0, axis 1 0 0, limit lower=-2.6179939 upper=2.6179939 effort=2.8 velocity=5.6548668
- added joint j_coxa_lm: type revolute, parent ee_lm, child coxa_lm, origin xyz=0 -0.10500000000000001 0 rpy=0 0 0, axis 1 0 0, limit lower=-2.6179939 upper=2.6179939 effort=2.8 velocity=5.6548668
- added joint j_coxa_lr: type revolute, parent ee_lr, child coxa_lr, origin xyz=0 -0.10500000000000001 0 rpy=0 0 0, axis 1 0 0, limit lower=-2.6179939 upper=2.6179939 effort=2.8 velocity=5.6548668
- added joint j_coxa_rf: type revolute, parent ee_rf, child coxa_rf, origin xyz=0 -0.10500000000000001 0 rpy=0 0 0, axis 1 0 0, limit lower=-2.6179939 upper=2.6179939 effort=2.8 velocity=5.6548668
- added joint j_coxa_rm: type revolute, parent ee_rm, child coxa_rm, origin xyz=0 -0.10500000000000001 0 rpy=0 0 0, axis 1 0 0, limit lower=-2.6179939 upper=2.6179939 effort=2.8 velocity=5.6548668
- added joint j_coxa_rr: type revolute, parent ee_rr, child coxa_rr, origin xyz=0 -0.10500000000000001 0 rpy=0 0 0, axis 1 0 0, limit lower=-2.6179939 upper=2.6179939 effort=2.8 velocity=5.6548668
- joint j_ee_lf: origin xyz=0.4330 0.2500 0.0000 rpy=0 0 2.09 -> xyz=0 -0.08 0 rpy=0 0 0
- joint j_ee_lm: origin xyz=0.0000 0.5000 0.0000 rpy=0 0 3.14 -> xyz=0 -0.08 0 rpy=0 0 0
- joint j_ee_lr: origin xyz=-0.4330 0.2500 0.0000 rpy=0 0 4.180000000000001 -> xyz=0 -0.08 0 rpy=0 0 0
- joint j_ee_rf: origin xyz=0.4330 -0.2500 0.0000 rpy=0 0 1.05 -> xyz=0 -0.08 0 rpy=0 0 0
- joint j_ee_rm: origin xyz=0.0000 -0.5000 0.0000 rpy=0 0 0.0 -> xyz=0 -0.08 0 rpy=0 0 0
- joint j_ee_rr: origin xyz=-0.4330 -0.2500 0.0000 rpy=0 0 -1.0400000000000003 -> xyz=0 -0.08 0 rpy=0 0 0

File: catkin_ws/src/worms_description/urdf/worms_urdf.xacro (robot description, xacro)
@@ -1,8 +1,11 @@
 <?xml version="1.0" ?>
 <robot xmlns:xacro="http://www.ros.org/wiki/xacro">
-<xacro:property name="uib_connect_offset" value="0.04" />
-<xacro:property name="ee_connect_offset" value="0.0275" />
+<xacro:property name="uib_length" value="0.08" />
+<xacro:property name="ee_length" value="0.055" />
+<xacro:property name="coxa_length" value="0.05" />
+<xacro:property name="motor_diameter" value="0.05" />
 <xacro:property name="thigh_offset_y" value="-0.0645" />
 <xacro:property name="thigh_offset_z" value="-0.0145" />
+<!-- TODO: Update component masses and inertias -->
 <xacro:macro name="worms" params="parent *origin">
       <joint name="j_worms_attachment" type="fixed">
@@ -19,5 +22,4 @@
         </inertial>
         <visual>
-          <!--origin xyz="-0.0235 0 -0.03525" rpy="0 0 0" /-->
           <origin xyz="0 0 0" rpy="0 0 1.57" />
           <geometry>
@@ -39,4 +41,6 @@
         <material>Gazebo/Red</material>
       </gazebo>
+<!-- RPY are set to offset the UIB (first component in leg from the pallet) by 90 degrees then by the angle to match the hexagon -->
+<!-- TODO: Replace xyz with calculations based on hexagon diameter -->
     <xacro:leg_l xyz="0.4330 -0.2500 0.0000"  rpy="0 0 ${-0.52 + 1.57}" suffix="rf"/>
     <xacro:leg_l xyz="0.0000 -0.5000 0.0000"  rpy="0 0 ${-1.57 + 1.57}" suffix="rm"/>
@@ -49,12 +53,11 @@
   <link name="uib_${suffix}">
     <inertial>
-      <origin xyz="${uib_connect_offset} 0 0" rpy="0 0 0"  />
-      <mass value="0.024357719"/>
-     <inertia ixx="0.0051411124"  ixy="-0.00057530255"  ixz="-0.000024729049" iyy="0.0081915737" iyz="-0.000019223094" izz="0.0011379812" />
-    </inertial>
-    <visual>
-      <origin xyz="2 0 0" rpy="0 0 0"  />
-      <geometry>
-        <!--box size="0.045 0.022 0.0325" /-->
+      <origin xyz="0 -${uib_length/2} 0" rpy="0 0 0"  />
+      <mass value="0.024357719"/>
+     <inertia ixx="0.0051411124"  ixy="-0.00057530255"  ixz="-0.000024729049" iyy="0.0081915737" iyz="-0.000019223094" izz="0.0011379812" />
+    </inertial>
+    <visual>
+      <origin xyz="0 -${uib_length/2} 0" rpy="0 0 0"  />
+      <geometry>
         <mesh filename="package://worms_description/meshes/UIB.STL"  scale="1 1 1"/>
       </geometry>
@@ -64,5 +67,5 @@
     </visual>
     <collision>
-      <origin xyz="${uib_connect_offset} 0 0" rpy="0 0 0"  />
+      <origin xyz="0 -${uib_length/2} 0" rpy="0 0 0"  />
       <geometry>
         <mesh filename="package://worms_description/meshes/UIB.STL"  scale="1 1 1"/>
@@ -72,12 +75,11 @@
   <link name="ee_${suffix}">
     <inertial>
-      <origin xyz="${ee_connect_offset} 0 0" rpy="0 0 0"  />
-      <mass value="0.024357719"/>
-     <inertia ixx="0.0051411124"  ixy="-0.00057530255"  ixz="-0.000024729049" iyy="0.0081915737" iyz="-0.000019223094" izz="0.0011379812" />
-    </inertial>
-    <visual>
-      <origin xyz="0 -0.0252 0" rpy="0 0 0"  />
-      <geometry>
-        <!--box size="0.045 0.022 0.0325" /-->
+      <origin xyz="0 -${ee_length/2} 0" rpy="0 0 0"  />
+      <mass value="0.024357719"/>
+     <inertia ixx="0.0051411124"  ixy="-0.00057530255"  ixz="-0.000024729049" iyy="0.0081915737" iyz="-0.000019223094" izz="0.0011379812" />
+    </inertial>
+    <visual>
+      <origin xyz="0 -${ee_length/2} 0" rpy="0 0 0"  />
+      <geometry>
         <mesh filename="package://worms_description/meshes/end_effector.STL"  scale="1 1 1"/>
       </geometry>
@@ -87,5 +89,5 @@
     </visual>
     <collision>
-      <origin xyz="${ee_connect_offset} 0 0" rpy="0 0 0"  />
+      <origin xyz="0 -${ee_length/2} 0" rpy="0 0 0"  />
       <geometry>
         <mesh filename="package://worms_description/meshes/end_effector.STL"  scale="1 1 1"/>
@@ -93,12 +95,12 @@
     </collision>
   </link>
-  <!-- <link name="coxa_${suffix}">
-    <inertial>
-      <origin xyz="0 -${connect_offset} 0" rpy="0 0 0"  />
-      <mass value="0.024357719"/>
-     <inertia ixx="0.0051411124"  ixy="-0.00057530255"  ixz="-0.000024729049" iyy="0.0081915737" iyz="-0.000019223094" izz="0.0011379812" />
-    </inertial>
-    <visual>
-      <origin xyz="0 -0.0252 0" rpy="0 0 0"  />
+  <link name="coxa_${suffix}">
+    <inertial>
+      <origin xyz="0 -${coxa_length/2} 0" rpy="0 0 0"  />
+      <mass value="0.024357719"/>
+     <inertia ixx="0.0051411124"  ixy="-0.00057530255"  ixz="-0.000024729049" iyy="0.0081915737" iyz="-0.000019223094" izz="0.0011379812" />
+    </inertial>
+    <visual>
+      <origin xyz="0 -${coxa_length/2} 0" rpy="0 0 0"  />
       <geometry>
         <mesh filename="package://worms_description/meshes/coxa.STL"  scale="1 1 1"/>
@@ -109,5 +111,5 @@
     </visual>
     <collision>
-      <origin xyz="0 -${connect_offset} 0" rpy="0 0 0"  />
+      <origin xyz="0 -${coxa_length/2} 0" rpy="0 0 0"  />
       <geometry>
         <mesh filename="package://worms_description/meshes/coxa.STL"  scale="1 1 1"/>
@@ -115,5 +117,5 @@
     </collision>
   </link>
-  <link name="thigh_${suffix}">
+  <!-- <link name="thigh_${suffix}">
     <inertial>
       <origin xyz="0 0 0" rpy="0 0 0"  />
@@ -170,16 +172,16 @@
     <parent link="uib_${suffix}"/>
     <child link="ee_${suffix}"/>
-    <origin xyz="${xyz}" rpy="${rpy}" />
+    <origin xyz="0 -${uib_length} 0" rpy="0 0 0" />
     <axis xyz="1 0 0" />
     <limit effort="2.8" velocity="5.6548668" lower="-2.6179939" upper="2.6179939" />
   </joint>
-  <!-- <joint name="j_coxa_${suffix}" type="revolute">
+  <joint name="j_coxa_${suffix}" type="revolute">
     <parent link="ee_${suffix}"/>
     <child link="coxa_${suffix}"/>
-    <origin xyz="${xyz}" rpy="${rpy}" />
+    <origin xyz="0 -${ee_length + motor_diameter} 0" rpy="0 0 0" />
     <axis xyz="1 0 0" />
     <limit effort="2.8" velocity="5.6548668" lower="-2.6179939" upper="2.6179939" />
   </joint>
-  <joint name="j_thigh_${suffix}" type="revolute">
+<!--   <joint name="j_thigh_${suffix}" type="revolute">
     <parent link="coxa_${suffix}"/>
     <child link="thigh_${suffix}"/>
@@ -187,6 +189,6 @@
     <axis xyz="1 0 0" />
     <limit effort="2.8" velocity="5.6548668" lower="-2.6179939" upper="2.6179939" />
-  </joint>
-  <joint name="j_shin_${suffix}" type="revolute">
+  </joint> -->
+  <!-- <joint name="j_shin_${suffix}" type="revolute">
     <parent link="thigh_${suffix}"/>
     <child link="shin_${suffix}"/>

Commit message: minimal hexapod complete (coxa, thigh, shin)

File: catkin_ws/src/worms_description/urdf/worms.urdf (robot description, URDF)
Before this commit: robot worms, 20 links, 19 joints
Links:
- added link shin_lf, mass 0.024357719; collision mesh filename=package://worms_description/meshes/shin.STL scale=1 1 1; visual mesh filename=package://worms_description/meshes/shin.STL scale=1 1 1
- added link shin_lm, mass 0.024357719; collision mesh filename=package://worms_description/meshes/shin.STL scale=1 1 1; visual mesh filename=package://worms_description/meshes/shin.STL scale=1 1 1
- added link shin_lr, mass 0.024357719; collision mesh filename=package://worms_description/meshes/shin.STL scale=1 1 1; visual mesh filename=package://worms_description/meshes/shin.STL scale=1 1 1
- added link shin_rf, mass 0.024357719; collision mesh filename=package://worms_description/meshes/shin.STL scale=1 1 1; visual mesh filename=package://worms_description/meshes/shin.STL scale=1 1 1
- added link shin_rm, mass 0.024357719; collision mesh filename=package://worms_description/meshes/shin.STL scale=1 1 1; visual mesh filename=package://worms_description/meshes/shin.STL scale=1 1 1
- added link shin_rr, mass 0.024357719; collision mesh filename=package://worms_description/meshes/shin.STL scale=1 1 1; visual mesh filename=package://worms_description/meshes/shin.STL scale=1 1 1
- added link thigh_lf, mass 0.024357719; collision mesh filename=package://worms_description/meshes/thigh.STL scale=1 1 1; visual mesh filename=package://worms_description/meshes/thigh.STL scale=1 1 1
- added link thigh_lm, mass 0.024357719; collision mesh filename=package://worms_description/meshes/thigh.STL scale=1 1 1; visual mesh filename=package://worms_description/meshes/thigh.STL scale=1 1 1
- added link thigh_lr, mass 0.024357719; collision mesh filename=package://worms_description/meshes/thigh.STL scale=1 1 1; visual mesh filename=package://worms_description/meshes/thigh.STL scale=1 1 1
- added link thigh_rf, mass 0.024357719; collision mesh filename=package://worms_description/meshes/thigh.STL scale=1 1 1; visual mesh filename=package://worms_description/meshes/thigh.STL scale=1 1 1
- added link thigh_rm, mass 0.024357719; collision mesh filename=package://worms_description/meshes/thigh.STL scale=1 1 1; visual mesh filename=package://worms_description/meshes/thigh.STL scale=1 1 1
- added link thigh_rr, mass 0.024357719; collision mesh filename=package://worms_description/meshes/thigh.STL scale=1 1 1; visual mesh filename=package://worms_description/meshes/thigh.STL scale=1 1 1
Joints:
- added joint j_shin_lf: type revolute, parent thigh_lf, child shin_lf, origin xyz=0 -0.39999999999999997 0 rpy=0.785398 0 0, axis 1 0 0, limit lower=-2.6179939 upper=2.6179939 effort=2.8 velocity=5.6548668
- added joint j_shin_lm: type revolute, parent thigh_lm, child shin_lm, origin xyz=0 -0.39999999999999997 0 rpy=0.785398 0 0, axis 1 0 0, limit lower=-2.6179939 upper=2.6179939 effort=2.8 velocity=5.6548668
- added joint j_shin_lr: type revolute, parent thigh_lr, child shin_lr, origin xyz=0 -0.39999999999999997 0 rpy=0.785398 0 0, axis 1 0 0, limit lower=-2.6179939 upper=2.6179939 effort=2.8 velocity=5.6548668
- added joint j_shin_rf: type revolute, parent thigh_rf, child shin_rf, origin xyz=0 -0.39999999999999997 0 rpy=0.785398 0 0, axis 1 0 0, limit lower=-2.6179939 upper=2.6179939 effort=2.8 velocity=5.6548668
- added joint j_shin_rm: type revolute, parent thigh_rm, child shin_rm, origin xyz=0 -0.39999999999999997 0 rpy=0.785398 0 0, axis 1 0 0, limit lower=-2.6179939 upper=2.6179939 effort=2.8 velocity=5.6548668
- added joint j_shin_rr: type revolute, parent thigh_rr, child shin_rr, origin xyz=0 -0.39999999999999997 0 rpy=0.785398 0 0, axis 1 0 0, limit lower=-2.6179939 upper=2.6179939 effort=2.8 velocity=5.6548668
- added joint j_thigh_lf: type revolute, parent coxa_lf, child thigh_lf, origin xyz=0 -0.1 0 rpy=0 0 0, axis 1 0 0, limit lower=-2.6179939 upper=2.6179939 effort=2.8 velocity=5.6548668
- added joint j_thigh_lm: type revolute, parent coxa_lm, child thigh_lm, origin xyz=0 -0.1 0 rpy=0 0 0, axis 1 0 0, limit lower=-2.6179939 upper=2.6179939 effort=2.8 velocity=5.6548668
- added joint j_thigh_lr: type revolute, parent coxa_lr, child thigh_lr, origin xyz=0 -0.1 0 rpy=0 0 0, axis 1 0 0, limit lower=-2.6179939 upper=2.6179939 effort=2.8 velocity=5.6548668
- added joint j_thigh_rf: type revolute, parent coxa_rf, child thigh_rf, origin xyz=0 -0.1 0 rpy=0 0 0, axis 1 0 0, limit lower=-2.6179939 upper=2.6179939 effort=2.8 velocity=5.6548668
- added joint j_thigh_rm: type revolute, parent coxa_rm, child thigh_rm, origin xyz=0 -0.1 0 rpy=0 0 0, axis 1 0 0, limit lower=-2.6179939 upper=2.6179939 effort=2.8 velocity=5.6548668
- added joint j_thigh_rr: type revolute, parent coxa_rr, child thigh_rr, origin xyz=0 -0.1 0 rpy=0 0 0, axis 1 0 0, limit lower=-2.6179939 upper=2.6179939 effort=2.8 velocity=5.6548668
- joint j_coxa_lf: origin xyz=0 -0.10500000000000001 0 rpy=0 0 0 -> xyz=0 -0.10500000000000001 0 rpy=0.785398 0 0
- joint j_coxa_lm: origin xyz=0 -0.10500000000000001 0 rpy=0 0 0 -> xyz=0 -0.10500000000000001 0 rpy=0.785398 0 0
- joint j_coxa_lr: origin xyz=0 -0.10500000000000001 0 rpy=0 0 0 -> xyz=0 -0.10500000000000001 0 rpy=0.785398 0 0
- joint j_coxa_rf: origin xyz=0 -0.10500000000000001 0 rpy=0 0 0 -> xyz=0 -0.10500000000000001 0 rpy=0.785398 0 0
- joint j_coxa_rm: origin xyz=0 -0.10500000000000001 0 rpy=0 0 0 -> xyz=0 -0.10500000000000001 0 rpy=0.785398 0 0
- joint j_coxa_rr: origin xyz=0 -0.10500000000000001 0 rpy=0 0 0 -> xyz=0 -0.10500000000000001 0 rpy=0.785398 0 0

File: catkin_ws/src/worms_description/urdf/worms_urdf.xacro (robot description, xacro)
@@ -1,11 +1,15 @@
 <?xml version="1.0" ?>
 <robot xmlns:xacro="http://www.ros.org/wiki/xacro">
+<!-- Basic dimensions of WORMS-1 components -->
 <xacro:property name="uib_length" value="0.08" />
 <xacro:property name="ee_length" value="0.055" />
 <xacro:property name="coxa_length" value="0.05" />
 <xacro:property name="motor_diameter" value="0.05" />
-<xacro:property name="thigh_offset_y" value="-0.0645" />
-<xacro:property name="thigh_offset_z" value="-0.0145" />
+<xacro:property name="thigh_length" value="0.35" />
+<xacro:property name="shin_length" value="0.475" />
+<!-- <xacro:property name="thigh_offset_y" value="-0.0645" />
+<xacro:property name="thigh_offset_z" value="-0.0145" /> -->
 <!-- TODO: Update component masses and inertias -->
+<!-- TODO: Merge motor mesh into individual link meshes (coxa, thigh, shin) -->
 <xacro:macro name="worms" params="parent *origin">
       <joint name="j_worms_attachment" type="fixed">
@@ -117,12 +121,12 @@
     </collision>
   </link>
-  <!-- <link name="thigh_${suffix}">
-    <inertial>
-      <origin xyz="0 0 0" rpy="0 0 0"  />
-      <mass value="0.024357719"/>
-     <inertia ixx="0.0051411124"  ixy="-0.00057530255"  ixz="-0.000024729049" iyy="0.0081915737" iyz="-0.000019223094" izz="0.0011379812" />
-    </inertial>
-    <visual>
-      <origin xyz="0 0 0" rpy="0 0 0"  />
+  <link name="thigh_${suffix}">
+    <inertial>
+      <origin xyz="0 -${thigh_length/2} 0" rpy="0 0 0"  />
+      <mass value="0.024357719"/>
+     <inertia ixx="0.0051411124"  ixy="-0.00057530255"  ixz="-0.000024729049" iyy="0.0081915737" iyz="-0.000019223094" izz="0.0011379812" />
+    </inertial>
+    <visual>
+      <origin xyz="0 -${thigh_length/2} 0" rpy="0 0 0"  />
       <geometry>
         <mesh filename="package://worms_description/meshes/thigh.STL"  scale="1 1 1"/>
@@ -133,5 +137,5 @@
     </visual>
     <collision>
-      <origin xyz="0 0 0" rpy="0 0 0"  />
+      <origin xyz="0 -${thigh_length/2} 0" rpy="0 0 0"  />
       <geometry>
         <mesh filename="package://worms_description/meshes/thigh.STL"  scale="1 1 1"/>
@@ -141,10 +145,10 @@
   <link name="shin_${suffix}">
     <inertial>
-      <origin xyz="0 0 0" rpy="0 0 0"  />
-      <mass value="0.024357719"/>
-     <inertia ixx="0.0051411124"  ixy="-0.00057530255"  ixz="-0.000024729049" iyy="0.0081915737" iyz="-0.000019223094" izz="0.0011379812" />
-    </inertial>
-    <visual>
-      <origin xyz="0 0 0" rpy="0 0 0"  />
+      <origin xyz="0 -${shin_length/2} 0" rpy="0 0 0"  />
+      <mass value="0.024357719"/>
+     <inertia ixx="0.0051411124"  ixy="-0.00057530255"  ixz="-0.000024729049" iyy="0.0081915737" iyz="-0.000019223094" izz="0.0011379812" />
+    </inertial>
+    <visual>
+      <origin xyz="0 -${shin_length/2} 0" rpy="0 0 0"  />
       <geometry>
         <mesh filename="package://worms_description/meshes/shin.STL"  scale="1 1 1"/>
@@ -155,10 +159,10 @@
     </visual>
     <collision>
-      <origin xyz="0 0 0" rpy="0 0 0"  />
+      <origin xyz="0 -${shin_length/2} 0" rpy="0 0 0"  />
       <geometry>
         <mesh filename="package://worms_description/meshes/shin.STL"  scale="1 1 1"/>
       </geometry>
     </collision>
-  </link> -->
+  </link>
   <!-- Joint definitions -->
   <joint name="j_uib_${suffix}" type="fixed">
@@ -179,24 +183,24 @@
     <parent link="ee_${suffix}"/>
     <child link="coxa_${suffix}"/>
-    <origin xyz="0 -${ee_length + motor_diameter} 0" rpy="0 0 0" />
-    <axis xyz="1 0 0" />
-    <limit effort="2.8" velocity="5.6548668" lower="-2.6179939" upper="2.6179939" />
-  </joint>
-<!--   <joint name="j_thigh_${suffix}" type="revolute">
+    <origin xyz="0 -${ee_length + motor_diameter} 0" rpy="0.785398 0 0" />
+    <axis xyz="1 0 0" />
+    <limit effort="2.8" velocity="5.6548668" lower="-2.6179939" upper="2.6179939" />
+  </joint>
+  <joint name="j_thigh_${suffix}" type="revolute">
     <parent link="coxa_${suffix}"/>
     <child link="thigh_${suffix}"/>
-    <origin xyz="0 0 0" rpy=" 0 3.14159 3.14159" />
-    <axis xyz="1 0 0" />
-    <limit effort="2.8" velocity="5.6548668" lower="-2.6179939" upper="2.6179939" />
-  </joint> -->
-  <!-- <joint name="j_shin_${suffix}" type="revolute">
+    <origin xyz="0 -${coxa_length + motor_diameter} 0" rpy="0 0 0" />
+    <axis xyz="1 0 0" />
+    <limit effort="2.8" velocity="5.6548668" lower="-2.6179939" upper="2.6179939" />
+  </joint>
+  <joint name="j_shin_${suffix}" type="revolute">
     <parent link="thigh_${suffix}"/>
     <child link="shin_${suffix}"/>
-    <origin xyz="0 ${thigh_offset_y} ${thigh_offset_z}" rpy="-1.5707 0 3.14159" />
-    <axis xyz="1 0 0" />
-    <limit effort="2.8" velocity="5.6548668" lower="-2.6179939" upper="2.6179939" />
-  </joint> -->
+    <origin xyz="0 -${thigh_length + motor_diameter} 0" rpy="0.785398 0 0" />
+    <axis xyz="1 0 0" />
+    <limit effort="2.8" velocity="5.6548668" lower="-2.6179939" upper="2.6179939" />
+  </joint>
   <!-- Joint transmission definitions -->
-   <!-- <transmission name="t_coxa_${suffix}">
+   <transmission name="t_coxa_${suffix}">
     <type>transmission_interface/SimpleTransmission</type>
     <joint name="j_coxa_${suffix}">
@@ -227,5 +231,5 @@
       <mechanicalReduction>1</mechanicalReduction>
     </actuator>
-  </transmission> -->
+  </transmission>
 <!-- Gazebo material definitions -->
   <gazebo reference="uib_${suffix}">
