Commit message: fixed joints, added link meshes with motors

File: catkin_ws/src/worms_description/urdf/worms.urdf (robot description, URDF)
Before this commit: robot worms, 32 links, 31 joints
Links:
- link coxa_lf: geometry collision mesh filename=package://worms_description/meshes/motor_coxa.stl scale=1 1 1; visual mesh filename=package://worms_description/meshes/motor_coxa.stl scale=1 1 1
- link coxa_lm: geometry collision mesh filename=package://worms_description/meshes/motor_coxa.stl scale=1 1 1; visual mesh filename=package://worms_description/meshes/motor_coxa.stl scale=1 1 1
- link coxa_lr: geometry collision mesh filename=package://worms_description/meshes/motor_coxa.stl scale=1 1 1; visual mesh filename=package://worms_description/meshes/motor_coxa.stl scale=1 1 1
- link coxa_rf: geometry collision mesh filename=package://worms_description/meshes/motor_coxa.stl scale=1 1 1; visual mesh filename=package://worms_description/meshes/motor_coxa.stl scale=1 1 1
- link coxa_rm: geometry collision mesh filename=package://worms_description/meshes/motor_coxa.stl scale=1 1 1; visual mesh filename=package://worms_description/meshes/motor_coxa.stl scale=1 1 1
- link coxa_rr: geometry collision mesh filename=package://worms_description/meshes/motor_coxa.stl scale=1 1 1; visual mesh filename=package://worms_description/meshes/motor_coxa.stl scale=1 1 1
- link shin_lf: geometry collision mesh filename=package://worms_description/meshes/motor_shin.stl scale=1 1 1; visual mesh filename=package://worms_description/meshes/motor_shin.stl scale=1 1 1
- link shin_lm: geometry collision mesh filename=package://worms_description/meshes/motor_shin.stl scale=1 1 1; visual mesh filename=package://worms_description/meshes/motor_shin.stl scale=1 1 1
- link shin_lr: geometry collision mesh filename=package://worms_description/meshes/motor_shin.stl scale=1 1 1; visual mesh filename=package://worms_description/meshes/motor_shin.stl scale=1 1 1
- link shin_rf: geometry collision mesh filename=package://worms_description/meshes/motor_shin.stl scale=1 1 1; visual mesh filename=package://worms_description/meshes/motor_shin.stl scale=1 1 1
- link shin_rm: geometry collision mesh filename=package://worms_description/meshes/motor_shin.stl scale=1 1 1; visual mesh filename=package://worms_description/meshes/motor_shin.stl scale=1 1 1
- link shin_rr: geometry collision mesh filename=package://worms_description/meshes/motor_shin.stl scale=1 1 1; visual mesh filename=package://worms_description/meshes/motor_shin.stl scale=1 1 1
- link thigh_lf: geometry collision mesh filename=package://worms_description/meshes/motor_thigh.stl scale=1 1 1; visual mesh filename=package://worms_description/meshes/motor_thigh.stl scale=1 1 1
- link thigh_lm: geometry collision mesh filename=package://worms_description/meshes/motor_thigh.stl scale=1 1 1; visual mesh filename=package://worms_description/meshes/motor_thigh.stl scale=1 1 1
- link thigh_lr: geometry collision mesh filename=package://worms_description/meshes/motor_thigh.stl scale=1 1 1; visual mesh filename=package://worms_description/meshes/motor_thigh.stl scale=1 1 1
- link thigh_rf: geometry collision mesh filename=package://worms_description/meshes/motor_thigh.stl scale=1 1 1; visual mesh filename=package://worms_description/meshes/motor_thigh.stl scale=1 1 1
- link thigh_rm: geometry collision mesh filename=package://worms_description/meshes/motor_thigh.stl scale=1 1 1; visual mesh filename=package://worms_description/meshes/motor_thigh.stl scale=1 1 1
- link thigh_rr: geometry collision mesh filename=package://worms_description/meshes/motor_thigh.stl scale=1 1 1; visual mesh filename=package://worms_description/meshes/motor_thigh.stl scale=1 1 1
Joints:
- joint j_coxa_lf: axis 1 0 0 -> 0 0 1; origin xyz=0 -0.10500000000000001 0 rpy=0.785398 0 0 -> xyz=0 -0.08 0 rpy=0 0 0
- joint j_coxa_lm: axis 1 0 0 -> 0 0 1; origin xyz=0 -0.10500000000000001 0 rpy=0.785398 0 0 -> xyz=0 -0.08 0 rpy=0 0 0
- joint j_coxa_lr: axis 1 0 0 -> 0 0 1; origin xyz=0 -0.10500000000000001 0 rpy=0.785398 0 0 -> xyz=0 -0.08 0 rpy=0 0 0
- joint j_coxa_rf: axis 1 0 0 -> 0 0 1; origin xyz=0 -0.10500000000000001 0 rpy=0.785398 0 0 -> xyz=0 -0.08 0 rpy=0 0 0
- joint j_coxa_rm: axis 1 0 0 -> 0 0 1; origin xyz=0 -0.10500000000000001 0 rpy=0.785398 0 0 -> xyz=0 -0.08 0 rpy=0 0 0
- joint j_coxa_rr: axis 1 0 0 -> 0 0 1; origin xyz=0 -0.10500000000000001 0 rpy=0.785398 0 0 -> xyz=0 -0.08 0 rpy=0 0 0
- joint j_shin_lf: origin xyz=0 -0.39999999999999997 0 rpy=0.785398 0 0 -> xyz=0 -0.39999999999999997 0 rpy=0.785 0 0
- joint j_shin_lm: origin xyz=0 -0.39999999999999997 0 rpy=0.785398 0 0 -> xyz=0 -0.39999999999999997 0 rpy=0.785 0 0
- joint j_shin_lr: origin xyz=0 -0.39999999999999997 0 rpy=0.785398 0 0 -> xyz=0 -0.39999999999999997 0 rpy=0.785 0 0
- joint j_shin_rf: origin xyz=0 -0.39999999999999997 0 rpy=0.785398 0 0 -> xyz=0 -0.39999999999999997 0 rpy=0.785 0 0
- joint j_shin_rm: origin xyz=0 -0.39999999999999997 0 rpy=0.785398 0 0 -> xyz=0 -0.39999999999999997 0 rpy=0.785 0 0
- joint j_shin_rr: origin xyz=0 -0.39999999999999997 0 rpy=0.785398 0 0 -> xyz=0 -0.39999999999999997 0 rpy=0.785 0 0
- joint j_thigh_lf: origin xyz=0 -0.1 0 rpy=0 0 0 -> xyz=0 -0.1 0 rpy=0.785 0 0
- joint j_thigh_lm: origin xyz=0 -0.1 0 rpy=0 0 0 -> xyz=0 -0.1 0 rpy=0.785 0 0
- joint j_thigh_lr: origin xyz=0 -0.1 0 rpy=0 0 0 -> xyz=0 -0.1 0 rpy=0.785 0 0
- joint j_thigh_rf: origin xyz=0 -0.1 0 rpy=0 0 0 -> xyz=0 -0.1 0 rpy=0.785 0 0
- joint j_thigh_rm: origin xyz=0 -0.1 0 rpy=0 0 0 -> xyz=0 -0.1 0 rpy=0.785 0 0
- joint j_thigh_rr: origin xyz=0 -0.1 0 rpy=0 0 0 -> xyz=0 -0.1 0 rpy=0.785 0 0

File: catkin_ws/src/worms_description/urdf/worms_urdf.xacro (robot description, xacro)
@@ -11,5 +11,5 @@
 <xacro:property name="thigh_offset_z" value="-0.0145" /> -->
 <!-- TODO: Update component masses and inertias -->
-<!-- TODO: Merge motor mesh into individual link meshes (coxa, thigh, shin) -->
+<!-- TODO: Add second ee, uib, and shoe -->
 <xacro:macro name="worms" params="parent *origin">
       <joint name="j_worms_attachment" type="fixed">
@@ -101,21 +101,21 @@
   <link name="coxa_${suffix}">
     <inertial>
-      <origin xyz="0 -${coxa_length/2} 0" rpy="0 0 0"  />
-      <mass value="0.024357719"/>
-     <inertia ixx="0.0051411124"  ixy="-0.00057530255"  ixz="-0.000024729049" iyy="0.0081915737" iyz="-0.000019223094" izz="0.0011379812" />
-    </inertial>
-    <visual>
-      <origin xyz="0 -${coxa_length/2} 0" rpy="0 0 0"  />
-      <geometry>
-        <mesh filename="package://worms_description/meshes/coxa.STL"  scale="1 1 1"/>
-      </geometry>
-      <material name="Grey">
-        <color rgba="0.20 0.20 0.20 1.0"/>
-      </material>
-    </visual>
-    <collision>
-      <origin xyz="0 -${coxa_length/2} 0" rpy="0 0 0"  />
-      <geometry>
-        <mesh filename="package://worms_description/meshes/coxa.STL"  scale="1 1 1"/>
+      <origin xyz="0 -${coxa_length/2 + motor_diameter/2} 0" rpy="0 0 0"  />
+      <mass value="0.024357719"/>
+     <inertia ixx="0.0051411124"  ixy="-0.00057530255"  ixz="-0.000024729049" iyy="0.0081915737" iyz="-0.000019223094" izz="0.0011379812" />
+    </inertial>
+    <visual>
+      <origin xyz="0 -${coxa_length/2 + motor_diameter/2} 0" rpy="0 0 0"  />
+      <geometry>
+        <mesh filename="package://worms_description/meshes/motor_coxa.stl"  scale="1 1 1"/>
+      </geometry>
+      <material name="Grey">
+        <color rgba="0.20 0.20 0.20 1.0"/>
+      </material>
+    </visual>
+    <collision>
+      <origin xyz="0 -${coxa_length/2 + motor_diameter/2} 0" rpy="0 0 0"  />
+      <geometry>
+        <mesh filename="package://worms_description/meshes/motor_coxa.stl"  scale="1 1 1"/>
       </geometry>
     </collision>
@@ -123,21 +123,21 @@
   <link name="thigh_${suffix}">
     <inertial>
-      <origin xyz="0 -${thigh_length/2} 0" rpy="0 0 0"  />
-      <mass value="0.024357719"/>
-     <inertia ixx="0.0051411124"  ixy="-0.00057530255"  ixz="-0.000024729049" iyy="0.0081915737" iyz="-0.000019223094" izz="0.0011379812" />
-    </inertial>
-    <visual>
-      <origin xyz="0 -${thigh_length/2} 0" rpy="0 0 0"  />
-      <geometry>
-        <mesh filename="package://worms_description/meshes/thigh.STL"  scale="1 1 1"/>
-      </geometry>
-      <material name="Grey">
-        <color rgba="0.20 0.20 0.20 1.0"/>
-      </material>
-    </visual>
-    <collision>
-      <origin xyz="0 -${thigh_length/2} 0" rpy="0 0 0"  />
-      <geometry>
-        <mesh filename="package://worms_description/meshes/thigh.STL"  scale="1 1 1"/>
+      <origin xyz="0 -${thigh_length/2 + motor_diameter/2} 0" rpy="0 0 0"  />
+      <mass value="0.024357719"/>
+     <inertia ixx="0.0051411124"  ixy="-0.00057530255"  ixz="-0.000024729049" iyy="0.0081915737" iyz="-0.000019223094" izz="0.0011379812" />
+    </inertial>
+    <visual>
+      <origin xyz="0 -${thigh_length/2 + motor_diameter/2} 0" rpy="0 0 0"  />
+      <geometry>
+        <mesh filename="package://worms_description/meshes/motor_thigh.stl"  scale="1 1 1"/>
+      </geometry>
+      <material name="Grey">
+        <color rgba="0.20 0.20 0.20 1.0"/>
+      </material>
+    </visual>
+    <collision>
+      <origin xyz="0 -${thigh_length/2 + motor_diameter/2} 0" rpy="0 0 0"  />
+      <geometry>
+        <mesh filename="package://worms_description/meshes/motor_thigh.stl"  scale="1 1 1"/>
       </geometry>
     </collision>
@@ -145,21 +145,21 @@
   <link name="shin_${suffix}">
     <inertial>
-      <origin xyz="0 -${shin_length/2} 0" rpy="0 0 0"  />
-      <mass value="0.024357719"/>
-     <inertia ixx="0.0051411124"  ixy="-0.00057530255"  ixz="-0.000024729049" iyy="0.0081915737" iyz="-0.000019223094" izz="0.0011379812" />
-    </inertial>
-    <visual>
-      <origin xyz="0 -${shin_length/2} 0" rpy="0 0 0"  />
-      <geometry>
-        <mesh filename="package://worms_description/meshes/shin.STL"  scale="1 1 1"/>
-      </geometry>
-      <material name="Grey">
-        <color rgba="0.20 0.20 0.20 1.0"/>
-      </material>
-    </visual>
-    <collision>
-      <origin xyz="0 -${shin_length/2} 0" rpy="0 0 0"  />
-      <geometry>
-        <mesh filename="package://worms_description/meshes/shin.STL"  scale="1 1 1"/>
+      <origin xyz="0 -${shin_length/2 + motor_diameter/2} 0" rpy="0 0 0"  />
+      <mass value="0.024357719"/>
+     <inertia ixx="0.0051411124"  ixy="-0.00057530255"  ixz="-0.000024729049" iyy="0.0081915737" iyz="-0.000019223094" izz="0.0011379812" />
+    </inertial>
+    <visual>
+      <origin xyz="0 -${shin_length/2 + motor_diameter/2} 0" rpy="0 0 0"  />
+      <geometry>
+        <mesh filename="package://worms_description/meshes/motor_shin.stl"  scale="1 1 1"/>
+      </geometry>
+      <material name="Grey">
+        <color rgba="0.20 0.20 0.20 1.0"/>
+      </material>
+    </visual>
+    <collision>
+      <origin xyz="0 -${shin_length/2 + motor_diameter/2} 0" rpy="0 0 0"  />
+      <geometry>
+        <mesh filename="package://worms_description/meshes/motor_shin.stl"  scale="1 1 1"/>
       </geometry>
     </collision>
@@ -183,6 +183,6 @@
     <parent link="ee_${suffix}"/>
     <child link="coxa_${suffix}"/>
-    <origin xyz="0 -${ee_length + motor_diameter} 0" rpy="0.785398 0 0" />
-    <axis xyz="1 0 0" />
+    <origin xyz="0 -${ee_length + motor_diameter/2} 0" rpy="0 0 0" />
+    <axis xyz="0 0 1" />
     <limit effort="2.8" velocity="5.6548668" lower="-2.6179939" upper="2.6179939" />
   </joint>
@@ -190,5 +190,5 @@
     <parent link="coxa_${suffix}"/>
     <child link="thigh_${suffix}"/>
-    <origin xyz="0 -${coxa_length + motor_diameter} 0" rpy="0 0 0" />
+    <origin xyz="0 -${coxa_length + motor_diameter} 0" rpy="0.785 0 0" />
     <axis xyz="1 0 0" />
     <limit effort="2.8" velocity="5.6548668" lower="-2.6179939" upper="2.6179939" />
@@ -197,5 +197,5 @@
     <parent link="thigh_${suffix}"/>
     <child link="shin_${suffix}"/>
-    <origin xyz="0 -${thigh_length + motor_diameter} 0" rpy="0.785398 0 0" />
+    <origin xyz="0 -${thigh_length + motor_diameter} 0" rpy="0.785 0 0" />
     <axis xyz="1 0 0" />
     <limit effort="2.8" velocity="5.6548668" lower="-2.6179939" upper="2.6179939" />
