Commit message: added variables for component masses

File: catkin_ws/src/worms_description/urdf/worms.urdf (robot description, URDF)
Before this commit: robot worms, 32 links, 31 joints
Links:
- link MP_BODY: mass 0.01 -> 7
- link coxa_lf: mass 0.024357719 -> 1.35
- link coxa_lm: mass 0.024357719 -> 1.35
- link coxa_lr: mass 0.024357719 -> 1.35
- link coxa_rf: mass 0.024357719 -> 1.35
- link coxa_rm: mass 0.024357719 -> 1.35
- link coxa_rr: mass 0.024357719 -> 1.35
- link ee_lf: mass 0.024357719 -> 1.85
- link ee_lm: mass 0.024357719 -> 1.85
- link ee_lr: mass 0.024357719 -> 1.85
- link ee_rf: mass 0.024357719 -> 1.85
- link ee_rm: mass 0.024357719 -> 1.85
- link ee_rr: mass 0.024357719 -> 1.85
- link shin_lf: mass 0.024357719 -> 6.85
- link shin_lm: mass 0.024357719 -> 6.85
- link shin_lr: mass 0.024357719 -> 6.85
- link shin_rf: mass 0.024357719 -> 6.85
- link shin_rm: mass 0.024357719 -> 6.85
- link shin_rr: mass 0.024357719 -> 6.85
- link thigh_lf: mass 0.024357719 -> 2.85
- link thigh_lm: mass 0.024357719 -> 2.85
- link thigh_lr: mass 0.024357719 -> 2.85
- link thigh_rf: mass 0.024357719 -> 2.85
- link thigh_rm: mass 0.024357719 -> 2.85
- link thigh_rr: mass 0.024357719 -> 2.85
- link uib_lf: mass 0.024357719 -> 1
- link uib_lm: mass 0.024357719 -> 1
- link uib_lr: mass 0.024357719 -> 1
- link uib_rf: mass 0.024357719 -> 1
- link uib_rm: mass 0.024357719 -> 1
- link uib_rr: mass 0.024357719 -> 1
Joints:
- joint j_coxa_lf: limit lower=-2.6179939 upper=2.6179939 effort=2.8 velocity=5.6548668 -> lower=-2.6179939 upper=2.6179939 effort=48 velocity=5.6548668
- joint j_coxa_lm: limit lower=-2.6179939 upper=2.6179939 effort=2.8 velocity=5.6548668 -> lower=-2.6179939 upper=2.6179939 effort=48 velocity=5.6548668
- joint j_coxa_lr: limit lower=-2.6179939 upper=2.6179939 effort=2.8 velocity=5.6548668 -> lower=-2.6179939 upper=2.6179939 effort=48 velocity=5.6548668
- joint j_coxa_rf: limit lower=-2.6179939 upper=2.6179939 effort=2.8 velocity=5.6548668 -> lower=-2.6179939 upper=2.6179939 effort=48 velocity=5.6548668
- joint j_coxa_rm: limit lower=-2.6179939 upper=2.6179939 effort=2.8 velocity=5.6548668 -> lower=-2.6179939 upper=2.6179939 effort=48 velocity=5.6548668
- joint j_coxa_rr: limit lower=-2.6179939 upper=2.6179939 effort=2.8 velocity=5.6548668 -> lower=-2.6179939 upper=2.6179939 effort=48 velocity=5.6548668
- joint j_shin_lf: limit lower=-2.6179939 upper=2.6179939 effort=2.8 velocity=5.6548668 -> lower=-2.6179939 upper=2.6179939 effort=48 velocity=5.6548668
- joint j_shin_lm: limit lower=-2.6179939 upper=2.6179939 effort=2.8 velocity=5.6548668 -> lower=-2.6179939 upper=2.6179939 effort=48 velocity=5.6548668
- joint j_shin_lr: limit lower=-2.6179939 upper=2.6179939 effort=2.8 velocity=5.6548668 -> lower=-2.6179939 upper=2.6179939 effort=48 velocity=5.6548668
- joint j_shin_rf: limit lower=-2.6179939 upper=2.6179939 effort=2.8 velocity=5.6548668 -> lower=-2.6179939 upper=2.6179939 effort=48 velocity=5.6548668
- joint j_shin_rm: limit lower=-2.6179939 upper=2.6179939 effort=2.8 velocity=5.6548668 -> lower=-2.6179939 upper=2.6179939 effort=48 velocity=5.6548668
- joint j_shin_rr: limit lower=-2.6179939 upper=2.6179939 effort=2.8 velocity=5.6548668 -> lower=-2.6179939 upper=2.6179939 effort=48 velocity=5.6548668
- joint j_thigh_lf: limit lower=-2.6179939 upper=2.6179939 effort=2.8 velocity=5.6548668 -> lower=-2.6179939 upper=2.6179939 effort=48 velocity=5.6548668
- joint j_thigh_lm: limit lower=-2.6179939 upper=2.6179939 effort=2.8 velocity=5.6548668 -> lower=-2.6179939 upper=2.6179939 effort=48 velocity=5.6548668
- joint j_thigh_lr: limit lower=-2.6179939 upper=2.6179939 effort=2.8 velocity=5.6548668 -> lower=-2.6179939 upper=2.6179939 effort=48 velocity=5.6548668
- joint j_thigh_rf: limit lower=-2.6179939 upper=2.6179939 effort=2.8 velocity=5.6548668 -> lower=-2.6179939 upper=2.6179939 effort=48 velocity=5.6548668
- joint j_thigh_rm: limit lower=-2.6179939 upper=2.6179939 effort=2.8 velocity=5.6548668 -> lower=-2.6179939 upper=2.6179939 effort=48 velocity=5.6548668
- joint j_thigh_rr: limit lower=-2.6179939 upper=2.6179939 effort=2.8 velocity=5.6548668 -> lower=-2.6179939 upper=2.6179939 effort=48 velocity=5.6548668

File: catkin_ws/src/worms_description/urdf/worms_urdf.xacro (robot description, xacro)
@@ -1,5 +1,5 @@
 <?xml version="1.0" ?>
 <robot xmlns:xacro="http://www.ros.org/wiki/xacro">
-<!-- Basic dimensions of WORMS-1 components -->
+<!-- Basic dimensions of WORMS-1 components (in m) -->
 <xacro:property name="uib_length" value="0.08" />
 <xacro:property name="ee_length" value="0.055" />
@@ -8,4 +8,15 @@
 <xacro:property name="thigh_length" value="0.35" />
 <xacro:property name="shin_length" value="0.475" />
+<!--  Masses of WORMS-1 components (in kg)-->
+<!--  Source: https://docs.google.com/spreadsheets/d/1z4cjFRy08wv40s6Jl9g9mymmIja3-cVj/edit#gid=1875184855-->
+<xacro:property name="m_payload" value="15" />
+<xacro:property name="m_pallet" value="7" />
+<xacro:property name="m_motor" value="0.85" />
+<xacro:property name="m_coxa" value="0.5" />
+<xacro:property name="m_thigh" value="2" />
+<xacro:property name="m_shin" value="6" />
+<xacro:property name="m_uib" value="1" />
+<xacro:property name="m_ee" value="1" />
+<xacro:property name="m_shoe" value="1.52" />
 <!-- <xacro:property name="thigh_offset_y" value="-0.0645" />
 <xacro:property name="thigh_offset_z" value="-0.0145" /> -->
@@ -21,8 +32,6 @@
         <inertial>
           <origin xyz="0 0 0" rpy="0 0 1.57" />
-          <!-- <mass value="0.97559947"/> -->
-          <!--mass value="0.01"/> -->
-	  <mass value="6.0" />
-          <inertia ixx="3.1081800"  ixy="-0.25460189"  ixz="2.0318174" iyy="6.3787776" iyz="0.16417863" izz="5.3316425" />
+	        <mass value="${m_pallet}" />
+          <inertia ixx="0.003016"  ixy="0.0"  ixz="0.0" iyy="0.003016" iyz="0.0" izz="0.006014" />
         </inertial>
         <visual>
@@ -60,91 +69,87 @@
     <inertial>
       <origin xyz="0 -${uib_length/2} 0" rpy="0 0 0"  />
-      <!--mass value="0.024357719"/> -->
-      <mass value="0.5"/>
+      <mass value="${m_uib}"/>
+      <inertia ixx="0.0051411124"  ixy="-0.00057530255"  ixz="-0.000024729049" iyy="0.0081915737" iyz="-0.000019223094" izz="0.0011379812" />
+    </inertial>
+    <visual>
+      <origin xyz="0 -${uib_length/2} 0" rpy="0 0 0"  />
+      <geometry>
+        <mesh filename="package://worms_description/meshes/UIB.STL"  scale="1 1 1"/>
+      </geometry>
+      <material name="Grey">
+        <color rgba="0.20 0.20 0.20 1.0"/>
+      </material>
+    </visual>
+    <collision>
+      <origin xyz="0 -${uib_length/2} 0" rpy="0 0 0"  />
+      <geometry>
+        <mesh filename="package://worms_description/meshes/UIB.STL"  scale="1 1 1"/>
+      </geometry>
+    </collision>
+  </link>
+  <link name="ee_${suffix}">
+    <inertial>
+      <origin xyz="0 -${ee_length/2} 0" rpy="0 0 0"  />
+      <mass value = "${m_ee + m_motor}"/>
+      <inertia ixx="0.0051411124"  ixy="-0.00057530255"  ixz="-0.000024729049" iyy="0.0081915737" iyz="-0.000019223094" izz="0.0011379812" />
+    </inertial>
+    <visual>
+      <origin xyz="0 -${ee_length/2} 0" rpy="0 0 0"  />
+      <geometry>
+        <mesh filename="package://worms_description/meshes/end_effector.STL"  scale="1 1 1"/>
+      </geometry>
+      <material name="Grey">
+        <color rgba="0.20 0.20 0.20 1.0"/>
+      </material>
+    </visual>
+    <collision>
+      <origin xyz="0 -${ee_length/2} 0" rpy="0 0 0"  />
+      <geometry>
+        <mesh filename="package://worms_description/meshes/end_effector.STL"  scale="1 1 1"/>
+      </geometry>
+    </collision>
+  </link>
+  <link name="coxa_${suffix}">
+    <inertial>
+      <origin xyz="0 -${coxa_length/2 + motor_diameter/2} 0" rpy="0 0 0"  />
+      <mass value="${m_coxa + m_motor}"/>
      <inertia ixx="0.0051411124"  ixy="-0.00057530255"  ixz="-0.000024729049" iyy="0.0081915737" iyz="-0.000019223094" izz="0.0011379812" />
     </inertial>
     <visual>
-      <origin xyz="0 -${uib_length/2} 0" rpy="0 0 0"  />
-      <geometry>
-        <mesh filename="package://worms_description/meshes/UIB.STL"  scale="1 1 1"/>
-      </geometry>
-      <material name="Grey">
-        <color rgba="0.20 0.20 0.20 1.0"/>
-      </material>
-    </visual>
-    <collision>
-      <origin xyz="0 -${uib_length/2} 0" rpy="0 0 0"  />
-      <geometry>
-        <mesh filename="package://worms_description/meshes/UIB.STL"  scale="1 1 1"/>
-      </geometry>
-    </collision>
-  </link>
-  <link name="ee_${suffix}">
-    <inertial>
-      <origin xyz="0 -${ee_length/2} 0" rpy="0 0 0"  />
-      <!--mass value="0.024357719"/> -->
-      <mass value = "0.5"/>
+      <origin xyz="0 -${coxa_length/2 + motor_diameter/2} 0" rpy="0 0 0"  />
+      <geometry>
+        <mesh filename="package://worms_description/meshes/motor_coxa.stl"  scale="1 1 1"/>
+      </geometry>
+      <material name="Grey">
+        <color rgba="0.20 0.20 0.20 1.0"/>
+      </material>
+    </visual>
+    <collision>
+      <origin xyz="0 -${coxa_length/2 + motor_diameter/2} 0" rpy="0 0 0"  />
+      <geometry>
+        <mesh filename="package://worms_description/meshes/motor_coxa.stl"  scale="1 1 1"/>
+      </geometry>
+    </collision>
+  </link>
+  <link name="thigh_${suffix}">
+    <inertial>
+      <origin xyz="0 -${thigh_length/2 + motor_diameter/2} 0" rpy="0 0 0"  />
+      <mass value="${m_thigh + m_motor}"/>
      <inertia ixx="0.0051411124"  ixy="-0.00057530255"  ixz="-0.000024729049" iyy="0.0081915737" iyz="-0.000019223094" izz="0.0011379812" />
     </inertial>
     <visual>
-      <origin xyz="0 -${ee_length/2} 0" rpy="0 0 0"  />
-      <geometry>
-        <mesh filename="package://worms_description/meshes/end_effector.STL"  scale="1 1 1"/>
-      </geometry>
-      <material name="Grey">
-        <color rgba="0.20 0.20 0.20 1.0"/>
-      </material>
-    </visual>
-    <collision>
-      <origin xyz="0 -${ee_length/2} 0" rpy="0 0 0"  />
-      <geometry>
-        <mesh filename="package://worms_description/meshes/end_effector.STL"  scale="1 1 1"/>
-      </geometry>
-    </collision>
-  </link>
-  <link name="coxa_${suffix}">
-    <inertial>
-      <origin xyz="0 -${coxa_length/2 + motor_diameter/2} 0" rpy="0 0 0"  />
-      <!--mass value="0.024357719"/> -->
-      <mass value="3.67"/>
-     <inertia ixx="0.0051411124"  ixy="-0.00057530255"  ixz="-0.000024729049" iyy="0.0081915737" iyz="-0.000019223094" izz="0.0011379812" />
-    </inertial>
-    <visual>
-      <origin xyz="0 -${coxa_length/2 + motor_diameter/2} 0" rpy="0 0 0"  />
-      <geometry>
-        <mesh filename="package://worms_description/meshes/motor_coxa.stl"  scale="1 1 1"/>
-      </geometry>
-      <material name="Grey">
-        <color rgba="0.20 0.20 0.20 1.0"/>
-      </material>
-    </visual>
-    <collision>
-      <origin xyz="0 -${coxa_length/2 + motor_diameter/2} 0" rpy="0 0 0"  />
-      <geometry>
-        <mesh filename="package://worms_description/meshes/motor_coxa.stl"  scale="1 1 1"/>
-      </geometry>
-    </collision>
-  </link>
-  <link name="thigh_${suffix}">
-    <inertial>
       <origin xyz="0 -${thigh_length/2 + motor_diameter/2} 0" rpy="0 0 0"  />
-      <!--mass value="0.024357719"/> -->
-      <mass value="3.67"/>
-     <inertia ixx="0.0051411124"  ixy="-0.00057530255"  ixz="-0.000024729049" iyy="0.0081915737" iyz="-0.000019223094" izz="0.0011379812" />
-    </inertial>
-    <visual>
+      <geometry>
+        <mesh filename="package://worms_description/meshes/motor_thigh.stl"  scale="1 1 1"/>
+      </geometry>
+      <material name="Grey">
+        <color rgba="0.20 0.20 0.20 1.0"/>
+      </material>
+    </visual>
+    <collision>
       <origin xyz="0 -${thigh_length/2 + motor_diameter/2} 0" rpy="0 0 0"  />
       <geometry>
         <mesh filename="package://worms_description/meshes/motor_thigh.stl"  scale="1 1 1"/>
       </geometry>
-      <material name="Grey">
-        <color rgba="0.20 0.20 0.20 1.0"/>
-      </material>
-    </visual>
-    <collision>
-      <origin xyz="0 -${thigh_length/2 + motor_diameter/2} 0" rpy="0 0 0"  />
-      <geometry>
-        <mesh filename="package://worms_description/meshes/motor_thigh.stl"  scale="1 1 1"/>
-      </geometry>
     </collision>
   </link>
@@ -152,7 +157,6 @@
     <inertial>
       <origin xyz="0 -${shin_length/2 + motor_diameter/2} 0" rpy="0 0 0"  />
-      <!-- mass value="0.024357719"/> -->
-      <mass value="3.67"/>
-     <inertia ixx="0.0051411124"  ixy="-0.00057530255"  ixz="-0.000024729049" iyy="0.0081915737" iyz="-0.000019223094" izz="0.0011379812" />
+      <mass value="${m_shin + m_motor}"/>
+      <inertia ixx="0.0051411124"  ixy="-0.00057530255"  ixz="-0.000024729049" iyy="0.0081915737" iyz="-0.000019223094" izz="0.0011379812" />
     </inertial>
     <visual>
@@ -192,5 +196,7 @@
     <origin xyz="0 -${ee_length + motor_diameter/2} 0" rpy="0 0 0" />
     <axis xyz="0 0 1" />
-    <limit effort="2.8" velocity="5.6548668" lower="-2.6179939" upper="2.6179939" />
+    <!-- <dynamics damping="0.0" friction="100000.0"/> -->
+    <!-- <limit effort="100.0" velocity="5.6548668" lower="-2.6179939" upper="2.6179939" /> -->
+    <limit effort="48" velocity="5.6548668" lower="-2.6179939" upper="2.6179939" />
   </joint>
   <joint name="j_thigh_${suffix}" type="revolute">
@@ -199,5 +205,7 @@
     <origin xyz="0 -${coxa_length + motor_diameter} 0" rpy="0.785 0 0" />
     <axis xyz="1 0 0" />
-    <limit effort="2.8" velocity="5.6548668" lower="-2.6179939" upper="2.6179939" />
+    <!-- <dynamics damping="0.0" friction="100000.0"/> -->
+    <!-- <limit effort="100.0" velocity="5.6548668" lower="-2.6179939" upper="2.6179939" /> -->
+    <limit effort="48" velocity="5.6548668" lower="-2.6179939" upper="2.6179939" />
   </joint>
   <joint name="j_shin_${suffix}" type="revolute">
@@ -206,5 +214,7 @@
     <origin xyz="0 -${thigh_length + motor_diameter} 0" rpy="0.785 0 0" />
     <axis xyz="1 0 0" />
-    <limit effort="2.8" velocity="5.6548668" lower="-2.6179939" upper="2.6179939" />
+    <!-- <dynamics damping="0.0" friction="100000.0"/> -->
+    <!-- <limit effort="100.0" velocity="5.6548668" lower="-2.6179939" upper="2.6179939" /> -->
+    <limit effort="48" velocity="5.6548668" lower="-2.6179939" upper="2.6179939" />
   </joint>
   <!-- Joint transmission definitions -->
@@ -255,4 +265,6 @@
     <material>Gazebo/Grey</material>
   </gazebo>
+<!-- Gazebo gravity setting -->
+  <!-- <turnGravityOff>1</turnGravityOff> -->
 </xacro:macro>
 </robot>

Commit message: added updated part meshes and urdf scripts

File: catkin_ws/src/worms_description/urdf/worms.urdf (robot description, URDF)
Before this commit: robot worms, 32 links, 31 joints
Joints:
- joint j_uib_lf: origin xyz=0.4330 0.2500 0.0000 rpy=0 0 2.09 -> xyz=0.4330 0.2500 1.0 rpy=0 0 2.09
- joint j_uib_lm: origin xyz=0.0000 0.5000 0.0000 rpy=0 0 3.14 -> xyz=0.0000 0.5000 1.0 rpy=0 0 3.14
- joint j_uib_lr: origin xyz=-0.4330 0.2500 0.0000 rpy=0 0 4.180000000000001 -> xyz=-0.4330 0.2500 1.0 rpy=0 0 4.180000000000001
- joint j_uib_rf: origin xyz=0.4330 -0.2500 0.0000 rpy=0 0 1.05 -> xyz=0.4330 -0.2500 1.0 rpy=0 0 1.05
- joint j_uib_rm: origin xyz=0.0000 -0.5000 0.0000 rpy=0 0 0.0 -> xyz=0.0000 -0.5000 1.0 rpy=0 0 0.0
- joint j_uib_rr: origin xyz=-0.4330 -0.2500 0.0000 rpy=0 0 -1.0400000000000003 -> xyz=-0.4330 -0.2500 1.0 rpy=0 0 -1.0400000000000003

File: catkin_ws/src/worms_description/urdf/worms_urdf.xacro (robot description, xacro)
@@ -1,4 +1,6 @@
 <?xml version="1.0" ?>
 <robot xmlns:xacro="http://www.ros.org/wiki/xacro">
+<!-- World Init Settings -->
+<xacro:property name="initial_z_offset" value="1.0" />
 <!-- Basic dimensions of WORMS-1 components (in m) -->
 <xacro:property name="uib_length" value="0.08" />
@@ -31,10 +33,10 @@
       <link name="MP_BODY">
         <inertial>
-          <origin xyz="0 0 0" rpy="0 0 1.57" />
+          <origin xyz="0 0 ${initial_z_offset}" rpy="0 0 1.57" />
 	        <mass value="${m_pallet}" />
           <inertia ixx="0.003016"  ixy="0.0"  ixz="0.0" iyy="0.003016" iyz="0.0" izz="0.006014" />
         </inertial>
         <visual>
-          <origin xyz="0 0 0" rpy="0 0 1.57" />
+          <origin xyz="0 0 ${initial_z_offset}" rpy="0 0 1.57" />
           <geometry>
             <!--box size="0.102 0.109 0.106" /-->
@@ -46,5 +48,5 @@
         </visual>
         <collision>
-          <origin xyz="0 0 0" rpy="0 0 0" />
+          <origin xyz="0 0 ${initial_z_offset}" rpy="0 0 0" />
           <geometry>
             <mesh filename="package://worms_description/meshes/pallet_coll.STL"  scale="1 1 1"/>
@@ -57,10 +59,10 @@
 <!-- RPY are set to offset the UIB (first component in leg from the pallet) by 90 degrees then by the angle to match the hexagon -->
 <!-- TODO: Replace xyz with calculations based on hexagon diameter -->
-    <xacro:leg_l xyz="0.4330 -0.2500 0.0000"  rpy="0 0 ${-0.52 + 1.57}" suffix="rf"/>
-    <xacro:leg_l xyz="0.0000 -0.5000 0.0000"  rpy="0 0 ${-1.57 + 1.57}" suffix="rm"/>
-    <xacro:leg_l xyz="-0.4330 -0.2500 0.0000"  rpy="0 0 ${-1.57 -1.04 + 1.57}" suffix="rr"/>
-    <xacro:leg_l xyz="0.4330 0.2500 0.0000"  rpy="0 0 ${0.52 + 1.57}" suffix="lf"/>
-    <xacro:leg_l xyz="0.0000 0.5000 0.0000"  rpy="0 0 ${1.57 + 1.57}" suffix="lm"/>
-    <xacro:leg_l xyz="-0.4330 0.2500 0.0000"  rpy="0 0 ${1.57 + 1.04 + 1.57}" suffix="lr"/>
+    <xacro:leg_l xyz="0.4330 -0.2500 ${initial_z_offset}"  rpy="0 0 ${-0.52 + 1.57}" suffix="rf"/>
+    <xacro:leg_l xyz="0.0000 -0.5000 ${initial_z_offset}"  rpy="0 0 ${-1.57 + 1.57}" suffix="rm"/>
+    <xacro:leg_l xyz="-0.4330 -0.2500 ${initial_z_offset}"  rpy="0 0 ${-1.57 -1.04 + 1.57}" suffix="rr"/>
+    <xacro:leg_l xyz="0.4330 0.2500 ${initial_z_offset}"  rpy="0 0 ${0.52 + 1.57}" suffix="lf"/>
+    <xacro:leg_l xyz="0.0000 0.5000 ${initial_z_offset}"  rpy="0 0 ${1.57 + 1.57}" suffix="lm"/>
+    <xacro:leg_l xyz="-0.4330 0.2500 ${initial_z_offset}"  rpy="0 0 ${1.57 + 1.04 + 1.57}" suffix="lr"/>
 </xacro:macro>
 <!-- Leg generation sub-macro -->
