Commit message: new meshes

File: catkin_ws/src/worms_description/urdf/worms.urdf (robot description, URDF)
Before this commit: robot worms, 32 links, 31 joints
Links:
- link coxa_lf: geometry collision mesh filename=package://worms_description/meshes/updated_parts/motor_coxa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 scale=1 1 1; visual mesh filename=package://worms_description/meshes/updated_parts/motor_coxa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 scale=1 1 1
- link coxa_lm: geometry collision mesh filename=package://worms_description/meshes/updated_parts/motor_coxa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 scale=1 1 1; visual mesh filename=package://worms_description/meshes/updated_parts/motor_coxa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 scale=1 1 1
- link coxa_lr: geometry collision mesh filename=package://worms_description/meshes/updated_parts/motor_coxa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 scale=1 1 1; visual mesh filename=package://worms_description/meshes/updated_parts/motor_coxa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 scale=1 1 1
- link coxa_rf: geometry collision mesh filename=package://worms_description/meshes/updated_parts/motor_coxa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 scale=1 1 1; visual mesh filename=package://worms_description/meshes/updated_parts/motor_coxa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 scale=1 1 1
- link coxa_rm: geometry collision mesh filename=package://worms_description/meshes/updated_parts/motor_coxa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 scale=1 1 1; visual mesh filename=package://worms_description/meshes/updated_parts/motor_coxa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 scale=1 1 1
- link coxa_rr: geometry collision mesh filename=package://worms_description/meshes/updated_parts/motor_coxa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 scale=1 1 1; visual mesh filename=package://worms_description/meshes/updated_parts/motor_coxa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 scale=1 1 1
- link shin_lf: geometry collision mesh filename=package://worms_description/meshes/updated_parts/motor_shin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 scale=1 1 1; visual mesh filename=package://worms_description/meshes/updated_parts/motor_shin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 scale=1 1 1
- link shin_lm: geometry collision mesh filename=package://worms_description/meshes/updated_parts/motor_shin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 scale=1 1 1; visual mesh filename=package://worms_description/meshes/updated_parts/motor_shin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 scale=1 1 1
- link shin_lr: geometry collision mesh filename=package://worms_description/meshes/updated_parts/motor_shin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 scale=1 1 1; visual mesh filename=package://worms_description/meshes/updated_parts/motor_shin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 scale=1 1 1
- link shin_rf: geometry collision mesh filename=package://worms_description/meshes/updated_parts/motor_shin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 scale=1 1 1; visual mesh filename=package://worms_description/meshes/updated_parts/motor_shin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 scale=1 1 1
- link shin_rm: geometry collision mesh filename=package://worms_description/meshes/updated_parts/motor_shin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 scale=1 1 1; visual mesh filename=package://worms_description/meshes/updated_parts/motor_shin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 scale=1 1 1
- link shin_rr: geometry collision mesh filename=package://worms_description/meshes/updated_parts/motor_shin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 scale=1 1 1; visual mesh filename=package://worms_description/meshes/updated_parts/motor_shin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 scale=1 1 1
- link thigh_lf: geometry collision mesh filename=package://worms_description/meshes/updated_parts/motor_thig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 scale=1 1 1; visual mesh filename=package://worms_description/meshes/updated_parts/motor_thig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 scale=1 1 1
- link thigh_lm: geometry collision mesh filename=package://worms_description/meshes/updated_parts/motor_thig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 scale=1 1 1; visual mesh filename=package://worms_description/meshes/updated_parts/motor_thig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 scale=1 1 1
- link thigh_lr: geometry collision mesh filename=package://worms_description/meshes/updated_parts/motor_thig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 scale=1 1 1; visual mesh filename=package://worms_description/meshes/updated_parts/motor_thig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 scale=1 1 1
- link thigh_rf: geometry collision mesh filename=package://worms_description/meshes/updated_parts/motor_thig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 scale=1 1 1; visual mesh filename=package://worms_description/meshes/updated_parts/motor_thig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 scale=1 1 1
- link thigh_rm: geometry collision mesh filename=package://worms_description/meshes/updated_parts/motor_thig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 scale=1 1 1; visual mesh filename=package://worms_description/meshes/updated_parts/motor_thig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 scale=1 1 1
- link thigh_rr: geometry collision mesh filename=package://worms_description/meshes/updated_parts/motor_thig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 scale=1 1 1; visual mesh filename=package://worms_description/meshes/updated_parts/motor_thig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 scale=1 1 1
Joints:
- joint j_coxa_lf: origin xyz=0 -0.08 0 rpy=0 0 0 -> xyz=0 -0.10400000000000001 0 rpy=0 0 0
- joint j_coxa_lm: origin xyz=0 -0.08 0 rpy=0 0 0 -> xyz=0 -0.10400000000000001 0 rpy=0 0 0
- joint j_coxa_lr: origin xyz=0 -0.08 0 rpy=0 0 0 -> xyz=0 -0.10400000000000001 0 rpy=0 0 0
- joint j_coxa_rf: origin xyz=0 -0.08 0 rpy=0 0 0 -> xyz=0 -0.10400000000000001 0 rpy=0 0 0
- joint j_coxa_rm: origin xyz=0 -0.08 0 rpy=0 0 0 -> xyz=0 -0.10400000000000001 0 rpy=0 0 0
- joint j_coxa_rr: origin xyz=0 -0.08 0 rpy=0 0 0 -> xyz=0 -0.10400000000000001 0 rpy=0 0 0
- joint j_shin_lf: origin xyz=0 -0.39999999999999997 0 rpy=0.785 0 0 -> xyz=0 -0.368 0 rpy=0.785 0 0
- joint j_shin_lm: origin xyz=0 -0.39999999999999997 0 rpy=0.785 0 0 -> xyz=0 -0.368 0 rpy=0.785 0 0
- joint j_shin_lr: origin xyz=0 -0.39999999999999997 0 rpy=0.785 0 0 -> xyz=0 -0.368 0 rpy=0.785 0 0
- joint j_shin_rf: origin xyz=0 -0.39999999999999997 0 rpy=0.785 0 0 -> xyz=0 -0.368 0 rpy=0.785 0 0
- joint j_shin_rm: origin xyz=0 -0.39999999999999997 0 rpy=0.785 0 0 -> xyz=0 -0.368 0 rpy=0.785 0 0
- joint j_shin_rr: origin xyz=0 -0.39999999999999997 0 rpy=0.785 0 0 -> xyz=0 -0.368 0 rpy=0.785 0 0
- joint j_thigh_lf: origin xyz=0 -0.1 0 rpy=0.785 0 0 -> xyz=0 -0.248 0 rpy=0.785 0 0
- joint j_thigh_lm: origin xyz=0 -0.1 0 rpy=0.785 0 0 -> xyz=0 -0.248 0 rpy=0.785 0 0
- joint j_thigh_lr: origin xyz=0 -0.1 0 rpy=0.785 0 0 -> xyz=0 -0.248 0 rpy=0.785 0 0
- joint j_thigh_rf: origin xyz=0 -0.1 0 rpy=0.785 0 0 -> xyz=0 -0.248 0 rpy=0.785 0 0
- joint j_thigh_rm: origin xyz=0 -0.1 0 rpy=0.785 0 0 -> xyz=0 -0.248 0 rpy=0.785 0 0
- joint j_thigh_rr: origin xyz=0 -0.1 0 rpy=0.785 0 0 -> xyz=0 -0.248 0 rpy=0.785 0 0

File: catkin_ws/src/worms_description/urdf/worms_urdf.xacro (robot description, xacro)
@@ -4,6 +4,9 @@
 <xacro:property name="initial_z_offset" value="1.0" />
 <!-- Basic dimensions of WORMS-1 components (in m) -->
-<xacro:property name="uib_length" value="0.08" />
-<xacro:property name="ee_length" value="0.055" />
+<!-- Note: Lengths are reported as distances between consecutive joints (motor axes) -->
+<xacro:property name="uib_length" value="0.062373" />
+<xacro:property name="ee_length" value="0.062373" />
+<xacro:property name="uib_ee_gap_length" value="0.0127" />
+<xacro:property name="hip_structure_length" value="0.1397" />
 <xacro:property name="coxa_length" value="0.15" />
 <xacro:property name="motor_diameter" value="0.098" />
@@ -26,4 +29,5 @@
 <!-- TODO: Add second ee, uib, and shoe -->
 <!-- TODO: Check link length specs -->
+<!-- TODO: Add simplified collision meshes -->
 <xacro:macro name="worms" params="parent *origin">
       <joint name="j_worms_attachment" type="fixed">
@@ -42,5 +46,5 @@
           <geometry>
             <!--box size="0.102 0.109 0.106" /-->
-            <mesh filename="package://worms_description/meshes/pallet.STL"  scale="1 1 1"/>
+            <mesh filename="package://worms_description/meshes/pallet.stl"  scale="1 1 1"/>
           </geometry>
           <material name="Red">
@@ -51,5 +55,5 @@
           <origin xyz="0 0 ${initial_z_offset}" rpy="0 0 1.57" />
           <geometry>
-            <mesh filename="package://worms_description/meshes/pallet_coll.STL"  scale="1 1 1"/>
+            <mesh filename="package://worms_description/meshes/pallet.stl"  scale="1 1 1"/>
           </geometry>
         </collision>
@@ -69,5 +73,5 @@
 <!-- Leg generation sub-macro -->
  <xacro:macro name="leg_l" params="xyz rpy suffix">
-  <link name="uib_${suffix}">
+  <link name="hip_structure_${suffix}">
     <inertial>
       <origin xyz="0 -${uib_length/2} 0" rpy="0 0 0"  />
@@ -78,36 +82,14 @@
       <origin xyz="0 -${uib_length/2} 0" rpy="0 0 0"  />
       <geometry>
+        <mesh filename="package://worms_description/meshes/ee_hip_structure.STL"  scale="1 1 1"/>
+      </geometry>
+      <material name="Grey">
+        <color rgba="0.20 0.20 0.20 1.0"/>
+      </material>
+    </visual>
+    <collision>
+      <origin xyz="0 -${uib_length/2} 0" rpy="0 0 0"  />
+      <geometry>
         <mesh filename="package://worms_description/meshes/UIB.STL"  scale="1 1 1"/>
-      </geometry>
-      <material name="Grey">
-        <color rgba="0.20 0.20 0.20 1.0"/>
-      </material>
-    </visual>
-    <collision>
-      <origin xyz="0 -${uib_length/2} 0" rpy="0 0 0"  />
-      <geometry>
-        <mesh filename="package://worms_description/meshes/UIB.STL"  scale="1 1 1"/>
-      </geometry>
-    </collision>
-  </link>
-  <link name="ee_${suffix}">
-    <inertial>
-      <origin xyz="0 -${ee_length/2} 0" rpy="0 0 0"  />
-      <mass value = "${m_ee + m_motor}"/>
-      <inertia ixx="0.0004167"  ixy="0.0"  ixz="0.0" iyy="0.0007417" iyz="0.0" izz="0.0007417" />
-    </inertial>
-    <visual>
-      <origin xyz="0 -${ee_length/2} 0" rpy="0 0 0"  />
-      <geometry>
-        <mesh filename="package://worms_description/meshes/end_effector.STL"  scale="1 1 1"/>
-      </geometry>
-      <material name="Grey">
-        <color rgba="0.20 0.20 0.20 1.0"/>
-      </material>
-    </visual>
-    <collision>
-      <origin xyz="0 -${ee_length/2} 0" rpy="0 0 0"  />
-      <geometry>
-        <mesh filename="package://worms_description/meshes/end_effector.STL"  scale="1 1 1"/>
       </geometry>
     </collision>
@@ -179,23 +161,38 @@
     </collision>
   </link>
+  <link name="shoe_${suffix}">
+    <inertial>
+      <origin xyz="0 -${shin_length/2 + motor_diameter/2} 0" rpy="0 0 0"  />
+      <mass value="${m_shin + m_motor}"/>
+      <inertia ixx="0.0004167"  ixy="0.0"  ixz="0.0" iyy="0.0007417" iyz="0.0" izz="0.0007417" />
+    </inertial>
+    <visual>
+      <origin xyz="0 -${shin_length/2 + motor_diameter/2} 0" rpy="0 0 0"  />
+      <geometry>
+        <mesh filename="package://worms_description/meshes/updated_parts/motor_shin.stl"  scale="1 1 1"/>
+      </geometry>
+      <material name="Grey">
+        <color rgba="0.20 0.20 0.20 1.0"/>
+      </material>
+    </visual>
+    <collision>
+      <origin xyz="0 -${shin_length/2 + motor_diameter/2} 0" rpy="0 0 0"  />
+      <geometry>
+        <mesh filename="package://worms_description/meshes/updated_parts/motor_shin.stl"  scale="1 1 1"/>
+      </geometry>
+    </collision>
+  </link>
   <!-- Joint definitions -->
-  <joint name="j_uib_${suffix}" type="fixed">
+  <joint name="j_hip_structure_${suffix}" type="fixed">
     <parent link="MP_BODY"/>
-    <child link="uib_${suffix}"/>
+    <child link="hip_structure_${suffix}"/>
     <origin xyz="${xyz}" rpy="${rpy}" />
     <axis xyz="1 0 0" />
     <limit effort="2.8" velocity="5.6548668" lower="-2.6179939" upper="2.6179939" />
   </joint>
-  <joint name="j_ee_${suffix}" type="fixed">
-    <parent link="uib_${suffix}"/>
-    <child link="ee_${suffix}"/>
-    <origin xyz="0 -${uib_length} 0" rpy="0 0 0" />
-    <axis xyz="1 0 0" />
-    <limit effort="2.8" velocity="5.6548668" lower="-2.6179939" upper="2.6179939" />
-  </joint>
   <joint name="j_coxa_${suffix}" type="revolute">
-    <parent link="ee_${suffix}"/>
+    <parent link="hip_structure_${suffix}"/>
     <child link="coxa_${suffix}"/>
-    <origin xyz="0 -${ee_length + motor_diameter/2} 0" rpy="0 0 0" />
+    <origin xyz="0 -${hip_structure_length} 0" rpy="0 0 0" />
     <axis xyz="0 0 1" />
     <!-- <dynamics damping="0.0" friction="100000.0"/> -->
@@ -206,5 +203,5 @@
     <parent link="coxa_${suffix}"/>
     <child link="thigh_${suffix}"/>
-    <origin xyz="0 -${coxa_length + motor_diameter} 0" rpy="0.785 0 0" />
+    <origin xyz="0 -${coxa_length} 0" rpy="0.785 0 0" />
     <axis xyz="1 0 0" />
     <!-- <dynamics damping="0.0" friction="100000.0"/> -->
@@ -215,5 +212,14 @@
     <parent link="thigh_${suffix}"/>
     <child link="shin_${suffix}"/>
-    <origin xyz="0 -${thigh_length + motor_diameter} 0" rpy="0.785 0 0" />
+    <origin xyz="0 -${thigh_length} 0" rpy="0.785 0 0" />
+    <axis xyz="1 0 0" />
+    <!-- <dynamics damping="0.0" friction="100000.0"/> -->
+    <!-- <limit effort="100.0" velocity="5.6548668" lower="-2.6179939" upper="2.6179939" /> -->
+    <limit effort="48" velocity="5.6548668" lower="-2.6179939" upper="2.6179939" />
+  </joint>
+  <joint name="j_shoe_${suffix}" type="fixed">
+    <parent link="shin_${suffix}"/>
+    <child link="shoe_${suffix}"/>
+    <origin xyz="0 -${shin_length} 0" rpy="0 0 0" />
     <axis xyz="1 0 0" />
     <!-- <dynamics damping="0.0" friction="100000.0"/> -->
@@ -253,10 +259,4 @@
   </transmission>
 <!-- Gazebo material definitions -->
-  <gazebo reference="uib_${suffix}">
-    <material>Gazebo/Grey</material>
-  </gazebo>
-  <gazebo reference="ee_${suffix}">
-    <material>Gazebo/Grey</material>
-  </gazebo>
   <gazebo reference="coxa_${suffix}">
     <material>Gazebo/Grey</material>
