Commit message: updated worm_urdf.xacro for latest part meshes (WIP)

File: catkin_ws/src/worms_description/urdf/worms.urdf (robot description, URDF)
Before this commit: robot worms, 32 links, 31 joints
Links:
- removed link ee_lf
- removed link ee_lm
- removed link ee_lr
- removed link ee_rf
- removed link ee_rm
- removed link ee_rr
- removed link uib_lf
- removed link uib_lm
- removed link uib_lr
- removed link uib_rf
- removed link uib_rm
- removed link uib_rr
- added link hip_structure_lf, mass 1; collision mesh filename=package://worms_description/meshes/ee_hip_structure.stl scale=1 1 1; visual mesh filename=package://worms_description/meshes/ee_hip_structure.stl scale=1 1 1
- added link hip_structure_lm, mass 1; collision mesh filename=package://worms_description/meshes/ee_hip_structure.stl scale=1 1 1; visual mesh filename=package://worms_description/meshes/ee_hip_structure.stl scale=1 1 1
- added link hip_structure_lr, mass 1; collision mesh filename=package://worms_description/meshes/ee_hip_structure.stl scale=1 1 1; visual mesh filename=package://worms_description/meshes/ee_hip_structure.stl scale=1 1 1
- added link hip_structure_rf, mass 1; collision mesh filename=package://worms_description/meshes/ee_hip_structure.stl scale=1 1 1; visual mesh filename=package://worms_description/meshes/ee_hip_structure.stl scale=1 1 1
- added link hip_structure_rm, mass 1; collision mesh filename=package://worms_description/meshes/ee_hip_structure.stl scale=1 1 1; visual mesh filename=package://worms_description/meshes/ee_hip_structure.stl scale=1 1 1
- added link hip_structure_rr, mass 1; collision mesh filename=package://worms_description/meshes/ee_hip_structure.stl scale=1 1 1; visual mesh filename=package://worms_description/meshes/ee_hip_structure.stl scale=1 1 1
- added link shoe_lf, mass 6.85; collision mesh filename=package://worms_description/meshes/ee_shoe.stl scale=1 1 1; visual mesh filename=package://worms_description/meshes/ee_shoe.stl scale=1 1 1
- added link shoe_lm, mass 6.85; collision mesh filename=package://worms_description/meshes/ee_shoe.stl scale=1 1 1; visual mesh filename=package://worms_description/meshes/ee_shoe.stl scale=1 1 1
- added link shoe_lr, mass 6.85; collision mesh filename=package://worms_description/meshes/ee_shoe.stl scale=1 1 1; visual mesh filename=package://worms_description/meshes/ee_shoe.stl scale=1 1 1
- added link shoe_rf, mass 6.85; collision mesh filename=package://worms_description/meshes/ee_shoe.stl scale=1 1 1; visual mesh filename=package://worms_description/meshes/ee_shoe.stl scale=1 1 1
- added link shoe_rm, mass 6.85; collision mesh filename=package://worms_description/meshes/ee_shoe.stl scale=1 1 1; visual mesh filename=package://worms_description/meshes/ee_shoe.stl scale=1 1 1
- added link shoe_rr, mass 6.85; collision mesh filename=package://worms_description/meshes/ee_shoe.stl scale=1 1 1; visual mesh filename=package://worms_description/meshes/ee_shoe.stl scale=1 1 1
- link MP_BODY: geometry collision mesh filename=package://worms_description/meshes/pallet_reduced.stl scale=1 1 1; visual mesh filename=package://worms_description/meshes/pallet_reduced.stl scale=1 1 1
- link coxa_lf: geometry collision mesh filename=package://worms_description/meshes/motor_coxa.stl scale=1 1 1; visual mesh filename=package://worms_description/meshes/motor_coxa.stl scale=1 1 1
- link coxa_lm: geometry collision mesh filename=package://worms_description/meshes/motor_coxa.stl scale=1 1 1; visual mesh filename=package://worms_description/meshes/motor_coxa.stl scale=1 1 1
- link coxa_lr: geometry collision mesh filename=package://worms_description/meshes/motor_coxa.stl scale=1 1 1; visual mesh filename=package://worms_description/meshes/motor_coxa.stl scale=1 1 1
- link coxa_rf: geometry collision mesh filename=package://worms_description/meshes/motor_coxa.stl scale=1 1 1; visual mesh filename=package://worms_description/meshes/motor_coxa.stl scale=1 1 1
- link coxa_rm: geometry collision mesh filename=package://worms_description/meshes/motor_coxa.stl scale=1 1 1; visual mesh filename=package://worms_description/meshes/motor_coxa.stl scale=1 1 1
- link coxa_rr: geometry collision mesh filename=package://worms_description/meshes/motor_coxa.stl scale=1 1 1; visual mesh filename=package://worms_description/meshes/motor_coxa.stl scale=1 1 1
- link shin_lf: geometry collision mesh filename=package://worms_description/meshes/motor_shin_ee.stl scale=1 1 1; visual mesh filename=package://worms_description/meshes/motor_shin_ee.stl scale=1 1 1
- link shin_lm: geometry collision mesh filename=package://worms_description/meshes/motor_shin_ee.stl scale=1 1 1; visual mesh filename=package://worms_description/meshes/motor_shin_ee.stl scale=1 1 1
- link shin_lr: geometry collision mesh filename=package://worms_description/meshes/motor_shin_ee.stl scale=1 1 1; visual mesh filename=package://worms_description/meshes/motor_shin_ee.stl scale=1 1 1
- link shin_rf: geometry collision mesh filename=package://worms_description/meshes/motor_shin_ee.stl scale=1 1 1; visual mesh filename=package://worms_description/meshes/motor_shin_ee.stl scale=1 1 1
- link shin_rm: geometry collision mesh filename=package://worms_description/meshes/motor_shin_ee.stl scale=1 1 1; visual mesh filename=package://worms_description/meshes/motor_shin_ee.stl scale=1 1 1
- link shin_rr: geometry collision mesh filename=package://worms_description/meshes/motor_shin_ee.stl scale=1 1 1; visual mesh filename=package://worms_description/meshes/motor_shin_ee.stl scale=1 1 1
- link thigh_lf: geometry collision mesh filename=package://worms_description/meshes/motor_thigh.stl scale=1 1 1; visual mesh filename=package://worms_description/meshes/motor_thigh.stl scale=1 1 1
- link thigh_lm: geometry collision mesh filename=package://worms_description/meshes/motor_thigh.stl scale=1 1 1; visual mesh filename=package://worms_description/meshes/motor_thigh.stl scale=1 1 1
- link thigh_lr: geometry collision mesh filename=package://worms_description/meshes/motor_thigh.stl scale=1 1 1; visual mesh filename=package://worms_description/meshes/motor_thigh.stl scale=1 1 1
- link thigh_rf: geometry collision mesh filename=package://worms_description/meshes/motor_thigh.stl scale=1 1 1; visual mesh filename=package://worms_description/meshes/motor_thigh.stl scale=1 1 1
- link thigh_rm: geometry collision mesh filename=package://worms_description/meshes/motor_thigh.stl scale=1 1 1; visual mesh filename=package://worms_description/meshes/motor_thigh.stl scale=1 1 1
- link thigh_rr: geometry collision mesh filename=package://worms_description/meshes/motor_thigh.stl scale=1 1 1; visual mesh filename=package://worms_description/meshes/motor_thigh.stl scale=1 1 1
Joints:
- removed joint j_ee_lf
- removed joint j_ee_lm
- removed joint j_ee_lr
- removed joint j_ee_rf
- removed joint j_ee_rm
- removed joint j_ee_rr
- removed joint j_uib_lf
- removed joint j_uib_lm
- removed joint j_uib_lr
- removed joint j_uib_rf
- removed joint j_uib_rm
- removed joint j_uib_rr
- added joint j_hip_structure_lf: type fixed, parent MP_BODY, child hip_structure_lf, origin xyz=0.476 0.2748 1.0 rpy=0 0 2.09, axis 1 0 0, limit lower=-2.6179939 upper=2.6179939 effort=2.8 velocity=5.6548668
- added joint j_hip_structure_lm: type fixed, parent MP_BODY, child hip_structure_lm, origin xyz=0.0000 0.5497 1.0 rpy=0 0 3.14, axis 1 0 0, limit lower=-2.6179939 upper=2.6179939 effort=2.8 velocity=5.6548668
- added joint j_hip_structure_lr: type fixed, parent MP_BODY, child hip_structure_lr, origin xyz=-0.476 0.2748 1.0 rpy=0 0 4.180000000000001, axis 1 0 0, limit lower=-2.6179939 upper=2.6179939 effort=2.8 velocity=5.6548668
- added joint j_hip_structure_rf: type fixed, parent MP_BODY, child hip_structure_rf, origin xyz=0.476 -0.2748 1.0 rpy=0 0 1.05, axis 1 0 0, limit lower=-2.6179939 upper=2.6179939 effort=2.8 velocity=5.6548668
- added joint j_hip_structure_rm: type fixed, parent MP_BODY, child hip_structure_rm, origin xyz=0.0000 -0.5497 1.0 rpy=0 0 0.0, axis 1 0 0, limit lower=-2.6179939 upper=2.6179939 effort=2.8 velocity=5.6548668
- added joint j_hip_structure_rr: type fixed, parent MP_BODY, child hip_structure_rr, origin xyz=-0.476 -0.2748 1.0 rpy=0 0 -1.0400000000000003, axis 1 0 0, limit lower=-2.6179939 upper=2.6179939 effort=2.8 velocity=5.6548668
- added joint j_shoe_lf: type fixed, parent shin_lf, child shoe_lf, origin xyz=0 -0.45 0 rpy=0 0 0, axis 1 0 0, limit lower=-2.6179939 upper=2.6179939 effort=48 velocity=5.6548668
- added joint j_shoe_lm: type fixed, parent shin_lm, child shoe_lm, origin xyz=0 -0.45 0 rpy=0 0 0, axis 1 0 0, limit lower=-2.6179939 upper=2.6179939 effort=48 velocity=5.6548668
- added joint j_shoe_lr: type fixed, parent shin_lr, child shoe_lr, origin xyz=0 -0.45 0 rpy=0 0 0, axis 1 0 0, limit lower=-2.6179939 upper=2.6179939 effort=48 velocity=5.6548668
- added joint j_shoe_rf: type fixed, parent shin_rf, child shoe_rf, origin xyz=0 -0.45 0 rpy=0 0 0, axis 1 0 0, limit lower=-2.6179939 upper=2.6179939 effort=48 velocity=5.6548668
- added joint j_shoe_rm: type fixed, parent shin_rm, child shoe_rm, origin xyz=0 -0.45 0 rpy=0 0 0, axis 1 0 0, limit lower=-2.6179939 upper=2.6179939 effort=48 velocity=5.6548668
- added joint j_shoe_rr: type fixed, parent shin_rr, child shoe_rr, origin xyz=0 -0.45 0 rpy=0 0 0, axis 1 0 0, limit lower=-2.6179939 upper=2.6179939 effort=48 velocity=5.6548668
- joint j_coxa_lf: origin xyz=0 -0.10400000000000001 0 rpy=0 0 0 -> xyz=0 -0.1397 0 rpy=0 0 0; parent ee_lf -> hip_structure_lf
- joint j_coxa_lm: origin xyz=0 -0.10400000000000001 0 rpy=0 0 0 -> xyz=0 -0.1397 0 rpy=0 0 0; parent ee_lm -> hip_structure_lm
- joint j_coxa_lr: origin xyz=0 -0.10400000000000001 0 rpy=0 0 0 -> xyz=0 -0.1397 0 rpy=0 0 0; parent ee_lr -> hip_structure_lr
- joint j_coxa_rf: origin xyz=0 -0.10400000000000001 0 rpy=0 0 0 -> xyz=0 -0.1397 0 rpy=0 0 0; parent ee_rf -> hip_structure_rf
- joint j_coxa_rm: origin xyz=0 -0.10400000000000001 0 rpy=0 0 0 -> xyz=0 -0.1397 0 rpy=0 0 0; parent ee_rm -> hip_structure_rm
- joint j_coxa_rr: origin xyz=0 -0.10400000000000001 0 rpy=0 0 0 -> xyz=0 -0.1397 0 rpy=0 0 0; parent ee_rr -> hip_structure_rr
- joint j_shin_lf: origin xyz=0 -0.368 0 rpy=0.785 0 0 -> xyz=0 -0.27 0 rpy=0.785 0 0
- joint j_shin_lm: origin xyz=0 -0.368 0 rpy=0.785 0 0 -> xyz=0 -0.27 0 rpy=0.785 0 0
- joint j_shin_lr: origin xyz=0 -0.368 0 rpy=0.785 0 0 -> xyz=0 -0.27 0 rpy=0.785 0 0
- joint j_shin_rf: origin xyz=0 -0.368 0 rpy=0.785 0 0 -> xyz=0 -0.27 0 rpy=0.785 0 0
- joint j_shin_rm: origin xyz=0 -0.368 0 rpy=0.785 0 0 -> xyz=0 -0.27 0 rpy=0.785 0 0
- joint j_shin_rr: origin xyz=0 -0.368 0 rpy=0.785 0 0 -> xyz=0 -0.27 0 rpy=0.785 0 0
- joint j_thigh_lf: origin xyz=0 -0.248 0 rpy=0.785 0 0 -> xyz=0 -0.15 0 rpy=0.785 0 0
- joint j_thigh_lm: origin xyz=0 -0.248 0 rpy=0.785 0 0 -> xyz=0 -0.15 0 rpy=0.785 0 0
- joint j_thigh_lr: origin xyz=0 -0.248 0 rpy=0.785 0 0 -> xyz=0 -0.15 0 rpy=0.785 0 0
- joint j_thigh_rf: origin xyz=0 -0.248 0 rpy=0.785 0 0 -> xyz=0 -0.15 0 rpy=0.785 0 0
- joint j_thigh_rm: origin xyz=0 -0.248 0 rpy=0.785 0 0 -> xyz=0 -0.15 0 rpy=0.785 0 0
- joint j_thigh_rr: origin xyz=0 -0.248 0 rpy=0.785 0 0 -> xyz=0 -0.15 0 rpy=0.785 0 0

File: catkin_ws/src/worms_description/urdf/worms_urdf.xacro (robot description, xacro)
@@ -46,5 +46,5 @@
           <geometry>
             <!--box size="0.102 0.109 0.106" /-->
-            <mesh filename="package://worms_description/meshes/pallet.stl"  scale="1 1 1"/>
+            <mesh filename="package://worms_description/meshes/pallet_reduced.stl"  scale="1 1 1"/>
           </geometry>
           <material name="Red">
@@ -55,5 +55,5 @@
           <origin xyz="0 0 ${initial_z_offset}" rpy="0 0 1.57" />
           <geometry>
-            <mesh filename="package://worms_description/meshes/pallet.stl"  scale="1 1 1"/>
+            <mesh filename="package://worms_description/older_parts/pallet.stl"  scale="1 1 1"/>
           </geometry>
         </collision>
@@ -64,10 +64,10 @@
 <!-- RPY are set to offset the UIB (first component in leg from the pallet) by 90 degrees then by the angle to match the hexagon -->
 <!-- TODO: Replace xyz with calculations based on hexagon diameter -->
-    <xacro:leg_l xyz="0.4330 -0.2500 ${initial_z_offset}"  rpy="0 0 ${-0.52 + 1.57}" suffix="rf"/>
-    <xacro:leg_l xyz="0.0000 -0.5000 ${initial_z_offset}"  rpy="0 0 ${-1.57 + 1.57}" suffix="rm"/>
-    <xacro:leg_l xyz="-0.4330 -0.2500 ${initial_z_offset}"  rpy="0 0 ${-1.57 -1.04 + 1.57}" suffix="rr"/>
-    <xacro:leg_l xyz="0.4330 0.2500 ${initial_z_offset}"  rpy="0 0 ${0.52 + 1.57}" suffix="lf"/>
-    <xacro:leg_l xyz="0.0000 0.5000 ${initial_z_offset}"  rpy="0 0 ${1.57 + 1.57}" suffix="lm"/>
-    <xacro:leg_l xyz="-0.4330 0.2500 ${initial_z_offset}"  rpy="0 0 ${1.57 + 1.04 + 1.57}" suffix="lr"/>
+    <xacro:leg_l xyz="0.476 -0.2748 ${initial_z_offset}"  rpy="0 0 ${-0.52 + 1.57}" suffix="rf"/>
+    <xacro:leg_l xyz="0.0000 -0.5497 ${initial_z_offset}"  rpy="0 0 ${-1.57 + 1.57}" suffix="rm"/>
+    <xacro:leg_l xyz="-0.476 -0.2748 ${initial_z_offset}"  rpy="0 0 ${-1.57 -1.04 + 1.57}" suffix="rr"/>
+    <xacro:leg_l xyz="0.476 0.2748 ${initial_z_offset}"  rpy="0 0 ${0.52 + 1.57}" suffix="lf"/>
+    <xacro:leg_l xyz="0.0000 0.5497 ${initial_z_offset}"  rpy="0 0 ${1.57 + 1.57}" suffix="lm"/>
+    <xacro:leg_l xyz="-0.476 0.2748 ${initial_z_offset}"  rpy="0 0 ${1.57 + 1.04 + 1.57}" suffix="lr"/>
 </xacro:macro>
 <!-- Leg generation sub-macro -->
@@ -75,21 +75,21 @@
   <link name="hip_structure_${suffix}">
     <inertial>
-      <origin xyz="0 -${uib_length/2} 0" rpy="0 0 0"  />
+      <origin xyz="0 -${hip_structure_length + uib_ee_gap_length/2} 0" rpy="0 0 0"  />
       <mass value="${m_uib}"/>
       <inertia ixx="0.0004167"  ixy="0.0"  ixz="0.0" iyy="0.0007417" iyz="0.0" izz="0.0007417" />
     </inertial>
     <visual>
-      <origin xyz="0 -${uib_length/2} 0" rpy="0 0 0"  />
-      <geometry>
-        <mesh filename="package://worms_description/meshes/ee_hip_structure.STL"  scale="1 1 1"/>
-      </geometry>
-      <material name="Grey">
-        <color rgba="0.20 0.20 0.20 1.0"/>
-      </material>
-    </visual>
-    <collision>
-      <origin xyz="0 -${uib_length/2} 0" rpy="0 0 0"  />
-      <geometry>
-        <mesh filename="package://worms_description/meshes/UIB.STL"  scale="1 1 1"/>
+      <origin xyz="0 -${hip_structure_length + uib_ee_gap_length} 0" rpy="0 0 0"  />
+      <geometry>
+        <mesh filename="package://worms_description/meshes/ee_hip_structure.stl"  scale="1 1 1"/>
+      </geometry>
+      <material name="Grey">
+        <color rgba="0.20 0.20 0.20 1.0"/>
+      </material>
+    </visual>
+    <collision>
+      <origin xyz="0 -${hip_structure_length + uib_ee_gap_length/2} 0" rpy="0 0 0"  />
+      <geometry>
+        <mesh filename="package://worms_description/meshes/ee_hip_structure.stl"  scale="1 1 1"/>
       </geometry>
     </collision>
@@ -97,21 +97,21 @@
   <link name="coxa_${suffix}">
     <inertial>
-      <origin xyz="0 -${coxa_length/2 + motor_diameter/2} 0" rpy="0 0 0"  />
+      <origin xyz="0 0 0" rpy="0 0 0"  />
       <mass value="${m_coxa + m_motor}"/>
       <inertia ixx="0.0004167"  ixy="0.0"  ixz="0.0" iyy="0.0007417" iyz="0.0" izz="0.0007417" />
     </inertial>
     <visual>
-      <origin xyz="0 -${coxa_length/2 + motor_diameter/2} 0" rpy="0 0 0"  />
-      <geometry>
-        <mesh filename="package://worms_description/meshes/updated_parts/motor_coxa.stl"  scale="1 1 1"/>
-      </geometry>
-      <material name="Grey">
-        <color rgba="0.20 0.20 0.20 1.0"/>
-      </material>
-    </visual>
-    <collision>
-      <origin xyz="0 -${coxa_length/2 + motor_diameter/2} 0" rpy="0 0 0"  />
-      <geometry>
-        <mesh filename="package://worms_description/meshes/updated_parts/motor_coxa.stl"  scale="1 1 1"/>
+      <origin xyz="0 0 0" rpy="0 0 0"  />
+      <geometry>
+        <mesh filename="package://worms_description/meshes/motor_coxa.stl"  scale="1 1 1"/>
+      </geometry>
+      <material name="Grey">
+        <color rgba="0.20 0.20 0.20 1.0"/>
+      </material>
+    </visual>
+    <collision>
+      <origin xyz="0 0 0" rpy="0 0 0"  />
+      <geometry>
+        <mesh filename="package://worms_description/meshes/motor_coxa.stl"  scale="1 1 1"/>
       </geometry>
     </collision>
@@ -119,21 +119,21 @@
   <link name="thigh_${suffix}">
     <inertial>
-      <origin xyz="0 -${thigh_length/2 + motor_diameter/2} 0" rpy="0 0 0"  />
+      <origin xyz="0 0 0" rpy="0 0 0"  />
       <mass value="${m_thigh + m_motor}"/>
       <inertia ixx="0.0004167"  ixy="0.0"  ixz="0.0" iyy="0.0007417" iyz="0.0" izz="0.0007417" />
     </inertial>
     <visual>
-      <origin xyz="0 -${thigh_length/2 + motor_diameter/2} 0" rpy="0 0 0"  />
-      <geometry>
-        <mesh filename="package://worms_description/meshes/updated_parts/motor_thigh.stl"  scale="1 1 1"/>
-      </geometry>
-      <material name="Grey">
-        <color rgba="0.20 0.20 0.20 1.0"/>
-      </material>
-    </visual>
-    <collision>
-      <origin xyz="0 -${thigh_length/2 + motor_diameter/2} 0" rpy="0 0 0"  />
-      <geometry>
-        <mesh filename="package://worms_description/meshes/updated_parts/motor_thigh.stl"  scale="1 1 1"/>
+      <origin xyz="0 0 0" rpy="0 0 0"  />
+      <geometry>
+        <mesh filename="package://worms_description/meshes/motor_thigh.stl"  scale="1 1 1"/>
+      </geometry>
+      <material name="Grey">
+        <color rgba="0.20 0.20 0.20 1.0"/>
+      </material>
+    </visual>
+    <collision>
+      <origin xyz="0 0 0" rpy="0 0 0"  />
+      <geometry>
+        <mesh filename="package://worms_description/meshes/motor_thigh.stl"  scale="1 1 1"/>
       </geometry>
     </collision>
@@ -141,21 +141,21 @@
   <link name="shin_${suffix}">
     <inertial>
-      <origin xyz="0 -${shin_length/2 + motor_diameter/2} 0" rpy="0 0 0"  />
+      <origin xyz="0 0 0" rpy="0 0 0"  />
       <mass value="${m_shin + m_motor}"/>
       <inertia ixx="0.0004167"  ixy="0.0"  ixz="0.0" iyy="0.0007417" iyz="0.0" izz="0.0007417" />
     </inertial>
     <visual>
-      <origin xyz="0 -${shin_length/2 + motor_diameter/2} 0" rpy="0 0 0"  />
-      <geometry>
-        <mesh filename="package://worms_description/meshes/updated_parts/motor_shin.stl"  scale="1 1 1"/>
-      </geometry>
-      <material name="Grey">
-        <color rgba="0.20 0.20 0.20 1.0"/>
-      </material>
-    </visual>
-    <collision>
-      <origin xyz="0 -${shin_length/2 + motor_diameter/2} 0" rpy="0 0 0"  />
-      <geometry>
-        <mesh filename="package://worms_description/meshes/updated_parts/motor_shin.stl"  scale="1 1 1"/>
+      <origin xyz="0 0 0" rpy="0 0 0"  />
+      <geometry>
+        <mesh filename="package://worms_description/meshes/motor_shin_ee.stl"  scale="1 1 1"/>
+      </geometry>
+      <material name="Grey">
+        <color rgba="0.20 0.20 0.20 1.0"/>
+      </material>
+    </visual>
+    <collision>
+      <origin xyz="0 0 0" rpy="0 0 0"  />
+      <geometry>
+        <mesh filename="package://worms_description/meshes/motor_shin_ee.stl"  scale="1 1 1"/>
       </geometry>
     </collision>
@@ -163,21 +163,21 @@
   <link name="shoe_${suffix}">
     <inertial>
-      <origin xyz="0 -${shin_length/2 + motor_diameter/2} 0" rpy="0 0 0"  />
+      <origin xyz="0 0 0" rpy="0 0 0"  />
       <mass value="${m_shin + m_motor}"/>
       <inertia ixx="0.0004167"  ixy="0.0"  ixz="0.0" iyy="0.0007417" iyz="0.0" izz="0.0007417" />
     </inertial>
     <visual>
-      <origin xyz="0 -${shin_length/2 + motor_diameter/2} 0" rpy="0 0 0"  />
-      <geometry>
-        <mesh filename="package://worms_description/meshes/updated_parts/motor_shin.stl"  scale="1 1 1"/>
-      </geometry>
-      <material name="Grey">
-        <color rgba="0.20 0.20 0.20 1.0"/>
-      </material>
-    </visual>
-    <collision>
-      <origin xyz="0 -${shin_length/2 + motor_diameter/2} 0" rpy="0 0 0"  />
-      <geometry>
-        <mesh filename="package://worms_description/meshes/updated_parts/motor_shin.stl"  scale="1 1 1"/>
+      <origin xyz="0 0 0" rpy="0 0 0"  />
+      <geometry>
+        <mesh filename="package://worms_description/meshes/ee_shoe.stl"  scale="1 1 1"/>
+      </geometry>
+      <material name="Grey">
+        <color rgba="0.20 0.20 0.20 1.0"/>
+      </material>
+    </visual>
+    <collision>
+      <origin xyz="0 0 0" rpy="0 0 0"  />
+      <geometry>
+        <mesh filename="package://worms_description/meshes/ee_shoe.stl"  scale="1 1 1"/>
       </geometry>
     </collision>
@@ -196,6 +196,4 @@
     <origin xyz="0 -${hip_structure_length} 0" rpy="0 0 0" />
     <axis xyz="0 0 1" />
-    <!-- <dynamics damping="0.0" friction="100000.0"/> -->
-    <!-- <limit effort="100.0" velocity="5.6548668" lower="-2.6179939" upper="2.6179939" /> -->
     <limit effort="48" velocity="5.6548668" lower="-2.6179939" upper="2.6179939" />
   </joint>
@@ -205,6 +203,4 @@
     <origin xyz="0 -${coxa_length} 0" rpy="0.785 0 0" />
     <axis xyz="1 0 0" />
-    <!-- <dynamics damping="0.0" friction="100000.0"/> -->
-    <!-- <limit effort="100.0" velocity="5.6548668" lower="-2.6179939" upper="2.6179939" /> -->
     <limit effort="48" velocity="5.6548668" lower="-2.6179939" upper="2.6179939" />
   </joint>
@@ -214,6 +210,4 @@
     <origin xyz="0 -${thigh_length} 0" rpy="0.785 0 0" />
     <axis xyz="1 0 0" />
-    <!-- <dynamics damping="0.0" friction="100000.0"/> -->
-    <!-- <limit effort="100.0" velocity="5.6548668" lower="-2.6179939" upper="2.6179939" /> -->
     <limit effort="48" velocity="5.6548668" lower="-2.6179939" upper="2.6179939" />
   </joint>
@@ -223,6 +217,4 @@
     <origin xyz="0 -${shin_length} 0" rpy="0 0 0" />
     <axis xyz="1 0 0" />
-    <!-- <dynamics damping="0.0" friction="100000.0"/> -->
-    <!-- <limit effort="100.0" velocity="5.6548668" lower="-2.6179939" upper="2.6179939" /> -->
     <limit effort="48" velocity="5.6548668" lower="-2.6179939" upper="2.6179939" />
   </joint>
