Commit message: updated worms urdf and xacro

File: catkin_ws/src/worms_description/urdf/worms.urdf (robot description, URDF)
Before this commit: robot worms, 32 links, 31 joints
Links:
- link MP_BODY: geometry collision mesh filename=package://worms_description/older_parts/pallet.stl scale=1 1 1; visual mesh filename=package://worms_description/meshes/pallet_reduced.stl scale=1 1 1
Joints:
- joint j_coxa_lf: origin xyz=0 -0.1397 0 rpy=0 0 0 -> xyz=0 -0.15239999999999998 0 rpy=0 0 0
- joint j_coxa_lm: origin xyz=0 -0.1397 0 rpy=0 0 0 -> xyz=0 -0.15239999999999998 0 rpy=0 0 0
- joint j_coxa_lr: origin xyz=0 -0.1397 0 rpy=0 0 0 -> xyz=0 -0.15239999999999998 0 rpy=0 0 0
- joint j_coxa_rf: origin xyz=0 -0.1397 0 rpy=0 0 0 -> xyz=0 -0.15239999999999998 0 rpy=0 0 0
- joint j_coxa_rm: origin xyz=0 -0.1397 0 rpy=0 0 0 -> xyz=0 -0.15239999999999998 0 rpy=0 0 0
- joint j_coxa_rr: origin xyz=0 -0.1397 0 rpy=0 0 0 -> xyz=0 -0.15239999999999998 0 rpy=0 0 0
- joint j_shoe_lf: origin xyz=0 -0.45 0 rpy=0 0 0 -> xyz=0 -0.5680000000000001 0 rpy=0 0 0
- joint j_shoe_lm: origin xyz=0 -0.45 0 rpy=0 0 0 -> xyz=0 -0.5680000000000001 0 rpy=0 0 0
- joint j_shoe_lr: origin xyz=0 -0.45 0 rpy=0 0 0 -> xyz=0 -0.5680000000000001 0 rpy=0 0 0
- joint j_shoe_rf: origin xyz=0 -0.45 0 rpy=0 0 0 -> xyz=0 -0.5680000000000001 0 rpy=0 0 0
- joint j_shoe_rm: origin xyz=0 -0.45 0 rpy=0 0 0 -> xyz=0 -0.5680000000000001 0 rpy=0 0 0
- joint j_shoe_rr: origin xyz=0 -0.45 0 rpy=0 0 0 -> xyz=0 -0.5680000000000001 0 rpy=0 0 0

File: catkin_ws/src/worms_description/urdf/worms_urdf.xacro (robot description, xacro)
@@ -75,5 +75,5 @@
   <link name="hip_structure_${suffix}">
     <inertial>
-      <origin xyz="0 -${hip_structure_length + uib_ee_gap_length/2} 0" rpy="0 0 0"  />
+      <origin xyz="0 -${hip_structure_length + uib_ee_gap_length} 0" rpy="0 0 0"  />
       <mass value="${m_uib}"/>
       <inertia ixx="0.0004167"  ixy="0.0"  ixz="0.0" iyy="0.0007417" iyz="0.0" izz="0.0007417" />
@@ -89,5 +89,5 @@
     </visual>
     <collision>
-      <origin xyz="0 -${hip_structure_length + uib_ee_gap_length/2} 0" rpy="0 0 0"  />
+      <origin xyz="0 -${hip_structure_length + uib_ee_gap_length} 0" rpy="0 0 0"  />
       <geometry>
         <mesh filename="package://worms_description/meshes/ee_hip_structure.stl"  scale="1 1 1"/>
@@ -194,5 +194,5 @@
     <parent link="hip_structure_${suffix}"/>
     <child link="coxa_${suffix}"/>
-    <origin xyz="0 -${hip_structure_length} 0" rpy="0 0 0" />
+    <origin xyz="0 -${hip_structure_length + uib_ee_gap_length} 0" rpy="0 0 0" />
     <axis xyz="0 0 1" />
     <limit effort="48" velocity="5.6548668" lower="-2.6179939" upper="2.6179939" />
@@ -215,5 +215,5 @@
     <parent link="shin_${suffix}"/>
     <child link="shoe_${suffix}"/>
-    <origin xyz="0 -${shin_length} 0" rpy="0 0 0" />
+    <origin xyz="0 -${shin_length + 0.118} 0" rpy="0 0 0" />
     <axis xyz="1 0 0" />
     <limit effort="48" velocity="5.6548668" lower="-2.6179939" upper="2.6179939" />

Commit message: added reduced meshes (reduced EE) and updated urdfs and xacro

File: catkin_ws/src/worms_description/urdf/worms.urdf (robot description, URDF)
Before this commit: robot worms, 32 links, 31 joints
Links:
- link MP_BODY: geometry collision mesh filename=package://worms_description/older_parts/pallet.stl scale=1 1 1; visual mesh filename=package://worms_description/meshes/pallet_reduced_new.stl scale=1 1 1
- link hip_structure_lf: geometry collision mesh filename=package://worms_description/meshes/hip_structure_reduced.stl scale=1 1 1; visual mesh filename=package://worms_description/meshes/hip_structure_reduced.stl scale=1 1 1
- link hip_structure_lm: geometry collision mesh filename=package://worms_description/meshes/hip_structure_reduced.stl scale=1 1 1; visual mesh filename=package://worms_description/meshes/hip_structure_reduced.stl scale=1 1 1
- link hip_structure_lr: geometry collision mesh filename=package://worms_description/meshes/hip_structure_reduced.stl scale=1 1 1; visual mesh filename=package://worms_description/meshes/hip_structure_reduced.stl scale=1 1 1
- link hip_structure_rf: geometry collision mesh filename=package://worms_description/meshes/hip_structure_reduced.stl scale=1 1 1; visual mesh filename=package://worms_description/meshes/hip_structure_reduced.stl scale=1 1 1
- link hip_structure_rm: geometry collision mesh filename=package://worms_description/meshes/hip_structure_reduced.stl scale=1 1 1; visual mesh filename=package://worms_description/meshes/hip_structure_reduced.stl scale=1 1 1
- link hip_structure_rr: geometry collision mesh filename=package://worms_description/meshes/hip_structure_reduced.stl scale=1 1 1; visual mesh filename=package://worms_description/meshes/hip_structure_reduced.stl scale=1 1 1
- link shin_lf: geometry collision mesh filename=package://worms_description/meshes/motor_shin_ee_reduced.stl scale=1 1 1; visual mesh filename=package://worms_description/meshes/motor_shin_ee_reduced.stl scale=1 1 1
- link shin_lm: geometry collision mesh filename=package://worms_description/meshes/motor_shin_ee_reduced.stl scale=1 1 1; visual mesh filename=package://worms_description/meshes/motor_shin_ee_reduced.stl scale=1 1 1
- link shin_lr: geometry collision mesh filename=package://worms_description/meshes/motor_shin_ee_reduced.stl scale=1 1 1; visual mesh filename=package://worms_description/meshes/motor_shin_ee_reduced.stl scale=1 1 1
- link shin_rf: geometry collision mesh filename=package://worms_description/meshes/motor_shin_ee_reduced.stl scale=1 1 1; visual mesh filename=package://worms_description/meshes/motor_shin_ee_reduced.stl scale=1 1 1
- link shin_rm: geometry collision mesh filename=package://worms_description/meshes/motor_shin_ee_reduced.stl scale=1 1 1; visual mesh filename=package://worms_description/meshes/motor_shin_ee_reduced.stl scale=1 1 1
- link shin_rr: geometry collision mesh filename=package://worms_description/meshes/motor_shin_ee_reduced.stl scale=1 1 1; visual mesh filename=package://worms_description/meshes/motor_shin_ee_reduced.stl scale=1 1 1
- link shoe_lf: geometry collision mesh filename=package://worms_description/meshes/ee_shoe_reduced.stl scale=1 1 1; visual mesh filename=package://worms_description/meshes/ee_shoe_reduced.stl scale=1 1 1
- link shoe_lm: geometry collision mesh filename=package://worms_description/meshes/ee_shoe_reduced.stl scale=1 1 1; visual mesh filename=package://worms_description/meshes/ee_shoe_reduced.stl scale=1 1 1
- link shoe_lr: geometry collision mesh filename=package://worms_description/meshes/ee_shoe_reduced.stl scale=1 1 1; visual mesh filename=package://worms_description/meshes/ee_shoe_reduced.stl scale=1 1 1
- link shoe_rf: geometry collision mesh filename=package://worms_description/meshes/ee_shoe_reduced.stl scale=1 1 1; visual mesh filename=package://worms_description/meshes/ee_shoe_reduced.stl scale=1 1 1
- link shoe_rm: geometry collision mesh filename=package://worms_description/meshes/ee_shoe_reduced.stl scale=1 1 1; visual mesh filename=package://worms_description/meshes/ee_shoe_reduced.stl scale=1 1 1
- link shoe_rr: geometry collision mesh filename=package://worms_description/meshes/ee_shoe_reduced.stl scale=1 1 1; visual mesh filename=package://worms_description/meshes/ee_shoe_reduced.stl scale=1 1 1

File: catkin_ws/src/worms_description/urdf/worms_urdf.xacro (robot description, xacro)
@@ -13,4 +13,5 @@
 <xacro:property name="thigh_length" value="0.27" />
 <xacro:property name="shin_length" value="0.45" />
+<xacro:property name="shin_shoe_length" value="0.118" />
 <!--  Masses of WORMS-1 components (in kg)-->
 <!--  Source: https://docs.google.com/spreadsheets/d/1z4cjFRy08wv40s6Jl9g9mymmIja3-cVj/edit#gid=1875184855-->
@@ -46,5 +47,5 @@
           <geometry>
             <!--box size="0.102 0.109 0.106" /-->
-            <mesh filename="package://worms_description/meshes/pallet_reduced.stl"  scale="1 1 1"/>
+            <mesh filename="package://worms_description/meshes/pallet_reduced_new.stl"  scale="1 1 1"/>
           </geometry>
           <material name="Red">
@@ -82,5 +83,5 @@
       <origin xyz="0 -${hip_structure_length + uib_ee_gap_length} 0" rpy="0 0 0"  />
       <geometry>
-        <mesh filename="package://worms_description/meshes/ee_hip_structure.stl"  scale="1 1 1"/>
+        <mesh filename="package://worms_description/meshes/hip_structure_reduced.stl"  scale="1 1 1"/>
       </geometry>
       <material name="Grey">
@@ -91,5 +92,5 @@
       <origin xyz="0 -${hip_structure_length + uib_ee_gap_length} 0" rpy="0 0 0"  />
       <geometry>
-        <mesh filename="package://worms_description/meshes/ee_hip_structure.stl"  scale="1 1 1"/>
+        <mesh filename="package://worms_description/meshes/hip_structure_reduced.stl"  scale="1 1 1"/>
       </geometry>
     </collision>
@@ -148,14 +149,14 @@
       <origin xyz="0 0 0" rpy="0 0 0"  />
       <geometry>
-        <mesh filename="package://worms_description/meshes/motor_shin_ee.stl"  scale="1 1 1"/>
-      </geometry>
-      <material name="Grey">
-        <color rgba="0.20 0.20 0.20 1.0"/>
-      </material>
-    </visual>
-    <collision>
-      <origin xyz="0 0 0" rpy="0 0 0"  />
-      <geometry>
-        <mesh filename="package://worms_description/meshes/motor_shin_ee.stl"  scale="1 1 1"/>
+        <mesh filename="package://worms_description/meshes/motor_shin_ee_reduced.stl"  scale="1 1 1"/>
+      </geometry>
+      <material name="Grey">
+        <color rgba="0.20 0.20 0.20 1.0"/>
+      </material>
+    </visual>
+    <collision>
+      <origin xyz="0 0 0" rpy="0 0 0"  />
+      <geometry>
+        <mesh filename="package://worms_description/meshes/motor_shin_ee_reduced.stl"  scale="1 1 1"/>
       </geometry>
     </collision>
@@ -170,14 +171,14 @@
       <origin xyz="0 0 0" rpy="0 0 0"  />
       <geometry>
-        <mesh filename="package://worms_description/meshes/ee_shoe.stl"  scale="1 1 1"/>
-      </geometry>
-      <material name="Grey">
-        <color rgba="0.20 0.20 0.20 1.0"/>
-      </material>
-    </visual>
-    <collision>
-      <origin xyz="0 0 0" rpy="0 0 0"  />
-      <geometry>
-        <mesh filename="package://worms_description/meshes/ee_shoe.stl"  scale="1 1 1"/>
+        <mesh filename="package://worms_description/meshes/ee_shoe_reduced.stl"  scale="1 1 1"/>
+      </geometry>
+      <material name="Grey">
+        <color rgba="0.20 0.20 0.20 1.0"/>
+      </material>
+    </visual>
+    <collision>
+      <origin xyz="0 0 0" rpy="0 0 0"  />
+      <geometry>
+        <mesh filename="package://worms_description/meshes/ee_shoe_reduced.stl"  scale="1 1 1"/>
       </geometry>
     </collision>
@@ -215,5 +216,5 @@
     <parent link="shin_${suffix}"/>
     <child link="shoe_${suffix}"/>
-    <origin xyz="0 -${shin_length + 0.118} 0" rpy="0 0 0" />
+    <origin xyz="0 -${shin_length + shin_shoe_length} 0" rpy="0 0 0" />
     <axis xyz="1 0 0" />
     <limit effort="48" velocity="5.6548668" lower="-2.6179939" upper="2.6179939" />
@@ -251,4 +252,7 @@
   </transmission>
 <!-- Gazebo material definitions -->
+  <gazebo reference="hip_structure_${suffix}">
+    <material>Gazebo/Grey</material>
+  </gazebo>
   <gazebo reference="coxa_${suffix}">
     <material>Gazebo/Grey</material>
@@ -258,4 +262,7 @@
   </gazebo>
   <gazebo reference="shin_${suffix}">
+    <material>Gazebo/Grey</material>
+  </gazebo>
+  <gazebo reference="shoe_${suffix}">
     <material>Gazebo/Grey</material>
   </gazebo>

Commit message: added simplified ee_shoe collision mesh, updated urdfs

File: catkin_ws/src/worms_description/urdf/worms.urdf (robot description, URDF)
Before this commit: robot worms, 32 links, 31 joints
Links:
- link MP_BODY: geometry visual mesh filename=package://worms_description/meshes/pallet_reduced_new.stl scale=1 1 1
- link coxa_lf: geometry visual mesh filename=package://worms_description/meshes/motor_coxa.stl scale=1 1 1
- link coxa_lm: geometry visual mesh filename=package://worms_description/meshes/motor_coxa.stl scale=1 1 1
- link coxa_lr: geometry visual mesh filename=package://worms_description/meshes/motor_coxa.stl scale=1 1 1
- link coxa_rf: geometry visual mesh filename=package://worms_description/meshes/motor_coxa.stl scale=1 1 1
- link coxa_rm: geometry visual mesh filename=package://worms_description/meshes/motor_coxa.stl scale=1 1 1
- link coxa_rr: geometry visual mesh filename=package://worms_description/meshes/motor_coxa.stl scale=1 1 1
- link hip_structure_lf: geometry visual mesh filename=package://worms_description/meshes/hip_structure_reduced.stl scale=1 1 1
- link hip_structure_lm: geometry visual mesh filename=package://worms_description/meshes/hip_structure_reduced.stl scale=1 1 1
- link hip_structure_lr: geometry visual mesh filename=package://worms_description/meshes/hip_structure_reduced.stl scale=1 1 1
- link hip_structure_rf: geometry visual mesh filename=package://worms_description/meshes/hip_structure_reduced.stl scale=1 1 1
- link hip_structure_rm: geometry visual mesh filename=package://worms_description/meshes/hip_structure_reduced.stl scale=1 1 1
- link hip_structure_rr: geometry visual mesh filename=package://worms_description/meshes/hip_structure_reduced.stl scale=1 1 1
- link shin_lf: geometry visual mesh filename=package://worms_description/meshes/motor_shin_ee_reduced.stl scale=1 1 1
- link shin_lm: geometry visual mesh filename=package://worms_description/meshes/motor_shin_ee_reduced.stl scale=1 1 1
- link shin_lr: geometry visual mesh filename=package://worms_description/meshes/motor_shin_ee_reduced.stl scale=1 1 1
- link shin_rf: geometry visual mesh filename=package://worms_description/meshes/motor_shin_ee_reduced.stl scale=1 1 1
- link shin_rm: geometry visual mesh filename=package://worms_description/meshes/motor_shin_ee_reduced.stl scale=1 1 1
- link shin_rr: geometry visual mesh filename=package://worms_description/meshes/motor_shin_ee_reduced.stl scale=1 1 1
- link shoe_lf: geometry collision mesh filename=package://worms_description/meshes/ee_shoe_coll.stl scale=1 1 1; visual mesh filename=package://worms_description/meshes/ee_shoe_reduced.stl scale=1 1 1
- link shoe_lm: geometry collision mesh filename=package://worms_description/meshes/ee_shoe_coll.stl scale=1 1 1; visual mesh filename=package://worms_description/meshes/ee_shoe_reduced.stl scale=1 1 1
- link shoe_lr: geometry collision mesh filename=package://worms_description/meshes/ee_shoe_coll.stl scale=1 1 1; visual mesh filename=package://worms_description/meshes/ee_shoe_reduced.stl scale=1 1 1
- link shoe_rf: geometry collision mesh filename=package://worms_description/meshes/ee_shoe_coll.stl scale=1 1 1; visual mesh filename=package://worms_description/meshes/ee_shoe_reduced.stl scale=1 1 1
- link shoe_rm: geometry collision mesh filename=package://worms_description/meshes/ee_shoe_coll.stl scale=1 1 1; visual mesh filename=package://worms_description/meshes/ee_shoe_reduced.stl scale=1 1 1
- link shoe_rr: geometry collision mesh filename=package://worms_description/meshes/ee_shoe_coll.stl scale=1 1 1; visual mesh filename=package://worms_description/meshes/ee_shoe_reduced.stl scale=1 1 1
- link thigh_lf: geometry visual mesh filename=package://worms_description/meshes/motor_thigh.stl scale=1 1 1
- link thigh_lm: geometry visual mesh filename=package://worms_description/meshes/motor_thigh.stl scale=1 1 1
- link thigh_lr: geometry visual mesh filename=package://worms_description/meshes/motor_thigh.stl scale=1 1 1
- link thigh_rf: geometry visual mesh filename=package://worms_description/meshes/motor_thigh.stl scale=1 1 1
- link thigh_rm: geometry visual mesh filename=package://worms_description/meshes/motor_thigh.stl scale=1 1 1
- link thigh_rr: geometry visual mesh filename=package://worms_description/meshes/motor_thigh.stl scale=1 1 1

File: catkin_ws/src/worms_description/urdf/worms_urdf.xacro (robot description, xacro)
@@ -53,10 +53,10 @@
           </material>
         </visual>
-        <collision>
+        <!-- <collision>
           <origin xyz="0 0 ${initial_z_offset}" rpy="0 0 1.57" />
           <geometry>
             <mesh filename="package://worms_description/older_parts/pallet.stl"  scale="1 1 1"/>
           </geometry>
-        </collision>
+        </collision> -->
       </link>
       <gazebo reference="MP_BODY">
@@ -89,96 +89,96 @@
       </material>
     </visual>
+    <!-- <collision>
+      <origin xyz="0 -${hip_structure_length + uib_ee_gap_length} 0" rpy="0 0 0"  />
+      <geometry>
+        <mesh filename="package://worms_description/meshes/hip_structure_reduced.stl"  scale="1 1 1"/>
+      </geometry>
+    </collision> -->
+  </link>
+  <link name="coxa_${suffix}">
+    <inertial>
+      <origin xyz="0 0 0" rpy="0 0 0"  />
+      <mass value="${m_coxa + m_motor}"/>
+      <inertia ixx="0.0004167"  ixy="0.0"  ixz="0.0" iyy="0.0007417" iyz="0.0" izz="0.0007417" />
+    </inertial>
+    <visual>
+      <origin xyz="0 0 0" rpy="0 0 0"  />
+      <geometry>
+        <mesh filename="package://worms_description/meshes/motor_coxa.stl"  scale="1 1 1"/>
+      </geometry>
+      <material name="Grey">
+        <color rgba="0.20 0.20 0.20 1.0"/>
+      </material>
+    </visual>
+    <!-- <collision>
+      <origin xyz="0 0 0" rpy="0 0 0"  />
+      <geometry>
+        <mesh filename="package://worms_description/meshes/motor_coxa.stl"  scale="1 1 1"/>
+      </geometry>
+    </collision> -->
+  </link>
+  <link name="thigh_${suffix}">
+    <inertial>
+      <origin xyz="0 0 0" rpy="0 0 0"  />
+      <mass value="${m_thigh + m_motor}"/>
+      <inertia ixx="0.0004167"  ixy="0.0"  ixz="0.0" iyy="0.0007417" iyz="0.0" izz="0.0007417" />
+    </inertial>
+    <visual>
+      <origin xyz="0 0 0" rpy="0 0 0"  />
+      <geometry>
+        <mesh filename="package://worms_description/meshes/motor_thigh.stl"  scale="1 1 1"/>
+      </geometry>
+      <material name="Grey">
+        <color rgba="0.20 0.20 0.20 1.0"/>
+      </material>
+    </visual>
+    <!-- <collision>
+      <origin xyz="0 0 0" rpy="0 0 0"  />
+      <geometry>
+        <mesh filename="package://worms_description/meshes/motor_thigh.stl"  scale="1 1 1"/>
+      </geometry>
+    </collision> -->
+  </link>
+  <link name="shin_${suffix}">
+    <inertial>
+      <origin xyz="0 0 0" rpy="0 0 0"  />
+      <mass value="${m_shin + m_motor}"/>
+      <inertia ixx="0.0004167"  ixy="0.0"  ixz="0.0" iyy="0.0007417" iyz="0.0" izz="0.0007417" />
+    </inertial>
+    <visual>
+      <origin xyz="0 0 0" rpy="0 0 0"  />
+      <geometry>
+        <mesh filename="package://worms_description/meshes/motor_shin_ee_reduced.stl"  scale="1 1 1"/>
+      </geometry>
+      <material name="Grey">
+        <color rgba="0.20 0.20 0.20 1.0"/>
+      </material>
+    </visual>
+    <!-- <collision>
+      <origin xyz="0 0 0" rpy="0 0 0"  />
+      <geometry>
+        <mesh filename="package://worms_description/meshes/motor_shin_ee_reduced.stl"  scale="1 1 1"/>
+      </geometry>
+    </collision> -->
+  </link>
+  <link name="shoe_${suffix}">
+    <inertial>
+      <origin xyz="0 0 0" rpy="0 0 0"  />
+      <mass value="${m_shin + m_motor}"/>
+      <inertia ixx="0.0004167"  ixy="0.0"  ixz="0.0" iyy="0.0007417" iyz="0.0" izz="0.29" />
+    </inertial>
+    <visual>
+      <origin xyz="0 0 0" rpy="0 0 0"  />
+      <geometry>
+        <mesh filename="package://worms_description/meshes/ee_shoe_reduced.stl"  scale="1 1 1"/>
+      </geometry>
+      <material name="Grey">
+        <color rgba="0.20 0.20 0.20 1.0"/>
+      </material>
+    </visual>
     <collision>
-      <origin xyz="0 -${hip_structure_length + uib_ee_gap_length} 0" rpy="0 0 0"  />
-      <geometry>
-        <mesh filename="package://worms_description/meshes/hip_structure_reduced.stl"  scale="1 1 1"/>
-      </geometry>
-    </collision>
-  </link>
-  <link name="coxa_${suffix}">
-    <inertial>
-      <origin xyz="0 0 0" rpy="0 0 0"  />
-      <mass value="${m_coxa + m_motor}"/>
-      <inertia ixx="0.0004167"  ixy="0.0"  ixz="0.0" iyy="0.0007417" iyz="0.0" izz="0.0007417" />
-    </inertial>
-    <visual>
-      <origin xyz="0 0 0" rpy="0 0 0"  />
-      <geometry>
-        <mesh filename="package://worms_description/meshes/motor_coxa.stl"  scale="1 1 1"/>
-      </geometry>
-      <material name="Grey">
-        <color rgba="0.20 0.20 0.20 1.0"/>
-      </material>
-    </visual>
-    <collision>
-      <origin xyz="0 0 0" rpy="0 0 0"  />
-      <geometry>
-        <mesh filename="package://worms_description/meshes/motor_coxa.stl"  scale="1 1 1"/>
-      </geometry>
-    </collision>
-  </link>
-  <link name="thigh_${suffix}">
-    <inertial>
-      <origin xyz="0 0 0" rpy="0 0 0"  />
-      <mass value="${m_thigh + m_motor}"/>
-      <inertia ixx="0.0004167"  ixy="0.0"  ixz="0.0" iyy="0.0007417" iyz="0.0" izz="0.0007417" />
-    </inertial>
-    <visual>
-      <origin xyz="0 0 0" rpy="0 0 0"  />
-      <geometry>
-        <mesh filename="package://worms_description/meshes/motor_thigh.stl"  scale="1 1 1"/>
-      </geometry>
-      <material name="Grey">
-        <color rgba="0.20 0.20 0.20 1.0"/>
-      </material>
-    </visual>
-    <collision>
-      <origin xyz="0 0 0" rpy="0 0 0"  />
-      <geometry>
-        <mesh filename="package://worms_description/meshes/motor_thigh.stl"  scale="1 1 1"/>
-      </geometry>
-    </collision>
-  </link>
-  <link name="shin_${suffix}">
-    <inertial>
-      <origin xyz="0 0 0" rpy="0 0 0"  />
-      <mass value="${m_shin + m_motor}"/>
-      <inertia ixx="0.0004167"  ixy="0.0"  ixz="0.0" iyy="0.0007417" iyz="0.0" izz="0.0007417" />
-    </inertial>
-    <visual>
-      <origin xyz="0 0 0" rpy="0 0 0"  />
-      <geometry>
-        <mesh filename="package://worms_description/meshes/motor_shin_ee_reduced.stl"  scale="1 1 1"/>
-      </geometry>
-      <material name="Grey">
-        <color rgba="0.20 0.20 0.20 1.0"/>
-      </material>
-    </visual>
-    <collision>
-      <origin xyz="0 0 0" rpy="0 0 0"  />
-      <geometry>
-        <mesh filename="package://worms_description/meshes/motor_shin_ee_reduced.stl"  scale="1 1 1"/>
-      </geometry>
-    </collision>
-  </link>
-  <link name="shoe_${suffix}">
-    <inertial>
-      <origin xyz="0 0 0" rpy="0 0 0"  />
-      <mass value="${m_shin + m_motor}"/>
-      <inertia ixx="0.0004167"  ixy="0.0"  ixz="0.0" iyy="0.0007417" iyz="0.0" izz="0.0007417" />
-    </inertial>
-    <visual>
-      <origin xyz="0 0 0" rpy="0 0 0"  />
-      <geometry>
-        <mesh filename="package://worms_description/meshes/ee_shoe_reduced.stl"  scale="1 1 1"/>
-      </geometry>
-      <material name="Grey">
-        <color rgba="0.20 0.20 0.20 1.0"/>
-      </material>
-    </visual>
-    <collision>
-      <origin xyz="0 0 0" rpy="0 0 0"  />
-      <geometry>
-        <mesh filename="package://worms_description/meshes/ee_shoe_reduced.stl"  scale="1 1 1"/>
+      <origin xyz="0 0 0" rpy="0 0 0"  />
+      <geometry>
+        <mesh filename="package://worms_description/meshes/ee_shoe_coll.stl"  scale="1 1 1"/>
       </geometry>
     </collision>
