Commit message: finished adding lidar/GNC arm with fixed joints

File: catkin_ws/src/worms_description/urdf/worms.urdf (robot description, URDF)
Before this commit: robot worms, 36 links, 35 joints
Links:
- added link arm_lidar_gnc, mass 1; visual mesh filename=package://worms_description/meshes/lidar.STL scale=1 1 1
Joints:
- added joint j_arm_lidar_gnc: type fixed, parent arm_hip_structure_gnc, child arm_lidar_gnc, origin xyz=0 0.1397 0 rpy=0 0 0, axis 1 0 0, limit lower=-2.6179939 upper=2.6179939 effort=2.8 velocity=5.6548668
- joint j_arm_coxa_gnc: origin xyz=0 0.27 0 rpy=0 0 0 -> xyz=0 0.27 0 rpy=-0.785 0 0; type revolute -> fixed
- joint j_arm_hip_structure_gnc: origin xyz=0 0.15 0 rpy=0 0 0 -> xyz=0 0.15 0 rpy=0 0 0 
- joint j_arm_thigh_gnc: origin xyz=0 0 0.5224000000000001 rpy=0 0 0 -> xyz=0 0 0.5224000000000001 rpy=0.785 0 0; type revolute -> fixed

File: catkin_ws/src/worms_description/urdf/worms_urdf.xacro (robot description, xacro)
@@ -15,4 +15,5 @@
 <xacro:property name="shin_shoe_length" value="0.118" />
 <xacro:property name="shin_ee_length" value="0.5097" />
+<xacro:property name="hip_structure_lidar_length" value="0.1397" />
 <!--  Masses of WORMS-1 components (in kg)-->
 <!--  Source: https://docs.google.com/spreadsheets/d/1z4cjFRy08wv40s6Jl9g9mymmIja3-cVj/edit#gid=1875184855-->
@@ -126,5 +127,5 @@
   <link name="arm_hip_structure_${suffix}">
     <inertial>
-      <origin xyz="0 -${hip_structure_length + uib_ee_gap_length} 0" rpy="0 0 0"  />
+      <origin xyz="0 0 0" rpy="0 0 0"  />
       <mass value="${m_uib}"/>
       <inertia ixx="0.0004167"  ixy="0.0"  ixz="0.0" iyy="0.0007417" iyz="0.0" izz="0.0007417" />
@@ -134,4 +135,20 @@
       <geometry>
         <mesh filename="package://worms_description/meshes/hip_structure_reduced.stl"  scale="1 1 1"/>
+      </geometry>
+      <material name="Grey">
+        <color rgba="0.20 0.20 0.20 1.0"/>
+      </material>
+    </visual>
+  </link>
+  <link name="arm_lidar_${suffix}">
+    <inertial>
+      <origin xyz="0 0 0" rpy="0 0 0"  />
+      <mass value="${m_uib}"/>
+      <inertia ixx="0.0004167"  ixy="0.0"  ixz="0.0" iyy="0.0007417" iyz="0.0" izz="0.0007417" />
+    </inertial>
+    <visual>
+      <origin xyz="0 0 0" rpy="0 0 0"  />
+      <geometry>
+        <mesh filename="package://worms_description/meshes/lidar.STL"  scale="1 1 1"/>
       </geometry>
       <material name="Grey">
@@ -148,15 +165,15 @@
     <limit effort="2.8" velocity="5.6548668" lower="-2.6179939" upper="2.6179939" />
   </joint>
-  <joint name="j_arm_thigh_${suffix}" type="revolute">
+  <joint name="j_arm_thigh_${suffix}" type="fixed">
     <parent link="arm_shin_${suffix}"/>
     <child link="arm_thigh_${suffix}"/>
-    <origin xyz="0 0 ${uib_ee_gap_length + shin_ee_length}" rpy="0 0 0" />
-    <axis xyz="1 0 0" />
-    <limit effort="48" velocity="5.6548668" lower="-2.6179939" upper="2.6179939" />
-  </joint>
-  <joint name="j_arm_coxa_${suffix}" type="revolute">
+    <origin xyz="0 0 ${uib_ee_gap_length + shin_ee_length}" rpy="0.785 0 0" />
+    <axis xyz="1 0 0" />
+    <limit effort="48" velocity="5.6548668" lower="-2.6179939" upper="2.6179939" />
+  </joint>
+  <joint name="j_arm_coxa_${suffix}" type="fixed">
     <parent link="arm_thigh_${suffix}"/>
     <child link="arm_coxa_${suffix}"/>
-    <origin xyz="0 ${thigh_length} 0" rpy="0 0 0" />
+    <origin xyz="0 ${thigh_length} 0" rpy="-0.785 0 0" />
     <axis xyz="0 0 1" />
     <limit effort="48" velocity="5.6548668" lower="-2.6179939" upper="2.6179939" />
@@ -165,10 +182,205 @@
     <parent link="arm_coxa_${suffix}"/>
     <child link="arm_hip_structure_${suffix}"/>
-    <origin xyz="0 ${coxa_length} 0" rpy="${rpy}" />
+    <origin xyz="0 ${coxa_length} 0" rpy="0 0 0 " />
     <axis xyz="1 0 0" />
     <limit effort="2.8" velocity="5.6548668" lower="-2.6179939" upper="2.6179939" />
   </joint>
+  <joint name="j_arm_lidar_${suffix}" type="fixed">
+    <parent link="arm_hip_structure_${suffix}"/>
+    <child link="arm_lidar_${suffix}"/>
+    <origin xyz="0 ${hip_structure_lidar_length} 0" rpy="0 0 0" />
+    <axis xyz="1 0 0" />
+    <limit effort="2.8" velocity="5.6548668" lower="-2.6179939" upper="2.6179939" />
+  </joint>
   <!-- Joint transmission definitions -->
-   <!-- <transmission name="t_coxa_${suffix}">
+   <!-- <transmission name="t_arm_coxa_${suffix}">
+    <type>transmission_interface/SimpleTransmission</type>
+    <joint name="j_arm_coxa_${suffix}">
+      <hardwareInterface>EffortJointInterface</hardwareInterface>
+    </joint>
+    <actuator name="m_arm_coxa_${suffix}">
+      <hardwareInterface>EffortJointInterface</hardwareInterface>
+      <mechanicalReduction>1</mechanicalReduction>
+    </actuator>
+  </transmission>
+   <transmission name="t_arm_thigh_${suffix}">
+    <type>transmission_interface/SimpleTransmission</type>
+    <joint name="j_arm_thigh_${suffix}">
+      <hardwareInterface>EffortJointInterface</hardwareInterface>
+    </joint>
+    <actuator name="m_arm_thigh_${suffix}">
+      <hardwareInterface>EffortJointInterface</hardwareInterface>
+      <mechanicalReduction>1</mechanicalReduction>
+    </actuator>
+  </transmission> -->
+<!-- Gazebo material definitions -->
+  <gazebo reference="arm_shin_${suffix}">
+    <material>Gazebo/Grey</material>
+  </gazebo>
+  <gazebo reference="arm_thigh_${suffix}">
+    <material>Gazebo/Grey</material>
+  </gazebo>
+  <gazebo reference="arm_coxa_${suffix}">
+    <material>Gazebo/Grey</material>
+  </gazebo>
+  <gazebo reference="arm_hip_structure_${suffix}">
+    <material>Gazebo/Grey</material>
+  </gazebo>
+  <gazebo reference="arm_lidar_${suffix}">
+    <material>Gazebo/Grey</material>
+  </gazebo>
+<!-- Gazebo gravity setting -->
+  <!-- <turnGravityOff>1</turnGravityOff> -->
+</xacro:macro>
+<!-- Leg generation sub-macro -->
+ <xacro:macro name="leg_l" params="xyz rpy suffix">
+  <link name="hip_structure_${suffix}">
+    <inertial>
+      <origin xyz="0 -${hip_structure_length + uib_ee_gap_length} 0" rpy="0 0 0"  />
+      <mass value="${m_uib}"/>
+      <inertia ixx="0.0004167"  ixy="0.0"  ixz="0.0" iyy="0.0007417" iyz="0.0" izz="0.0007417" />
+    </inertial>
+    <visual>
+      <origin xyz="0 -${hip_structure_length + uib_ee_gap_length} 0" rpy="0 0 0"  />
+      <geometry>
+        <mesh filename="package://worms_description/meshes/hip_structure_reduced.stl"  scale="1 1 1"/>
+      </geometry>
+      <material name="Grey">
+        <color rgba="0.20 0.20 0.20 1.0"/>
+      </material>
+    </visual>
+    <!-- <collision>
+      <origin xyz="0 -${hip_structure_length + uib_ee_gap_length} 0" rpy="0 0 0"  />
+      <geometry>
+        <mesh filename="package://worms_description/meshes/hip_structure_reduced.stl"  scale="1 1 1"/>
+      </geometry>
+    </collision> -->
+  </link>
+  <link name="coxa_${suffix}">
+    <inertial>
+      <origin xyz="0 0 0" rpy="0 0 0"  />
+      <mass value="${m_coxa + m_motor}"/>
+      <inertia ixx="0.0004167"  ixy="0.0"  ixz="0.0" iyy="0.0007417" iyz="0.0" izz="0.0007417" />
+    </inertial>
+    <visual>
+      <origin xyz="0 0 0" rpy="0 0 0"  />
+      <geometry>
+        <mesh filename="package://worms_description/meshes/motor_coxa.stl"  scale="1 1 1"/>
+      </geometry>
+      <material name="Grey">
+        <color rgba="0.20 0.20 0.20 1.0"/>
+      </material>
+    </visual>
+    <!-- <collision>
+      <origin xyz="0 0 0" rpy="0 0 0"  />
+      <geometry>
+        <mesh filename="package://worms_description/meshes/motor_coxa.stl"  scale="1 1 1"/>
+      </geometry>
+    </collision> -->
+  </link>
+  <link name="thigh_${suffix}">
+    <inertial>
+      <origin xyz="0 0 0" rpy="0 0 0"  />
+      <mass value="${m_thigh + m_motor}"/>
+      <inertia ixx="0.0004167"  ixy="0.0"  ixz="0.0" iyy="0.0007417" iyz="0.0" izz="0.0007417" />
+    </inertial>
+    <visual>
+      <origin xyz="0 0 0" rpy="0 0 0"  />
+      <geometry>
+        <mesh filename="package://worms_description/meshes/motor_thigh.stl"  scale="1 1 1"/>
+      </geometry>
+      <material name="Grey">
+        <color rgba="0.20 0.20 0.20 1.0"/>
+      </material>
+    </visual>
+    <!-- <collision>
+      <origin xyz="0 0 0" rpy="0 0 0"  />
+      <geometry>
+        <mesh filename="package://worms_description/meshes/motor_thigh.stl"  scale="1 1 1"/>
+      </geometry>
+    </collision> -->
+  </link>
+  <link name="shin_${suffix}">
+    <inertial>
+      <origin xyz="0 0 0" rpy="0 0 0"  />
+      <mass value="${m_shin + m_motor}"/>
+      <inertia ixx="0.0004167"  ixy="0.0"  ixz="0.0" iyy="0.0007417" iyz="0.0" izz="0.0007417" />
+    </inertial>
+    <visual>
+      <origin xyz="0 0 0" rpy="0 0 0"  />
+      <geometry>
+        <mesh filename="package://worms_description/meshes/motor_shin_ee_reduced.stl"  scale="1 1 1"/>
+      </geometry>
+      <material name="Grey">
+        <color rgba="0.20 0.20 0.20 1.0"/>
+      </material>
+    </visual>
+    <!-- <collision>
+      <origin xyz="0 0 0" rpy="0 0 0"  />
+      <geometry>
+        <mesh filename="package://worms_description/meshes/motor_shin_ee_reduced.stl"  scale="1 1 1"/>
+      </geometry>
+    </collision> -->
+  </link>
+  <link name="shoe_${suffix}">
+    <inertial>
+      <origin xyz="0 0 0" rpy="0 0 0"  />
+      <mass value="${m_shin + m_motor}"/>
+      <inertia ixx="0.0004167"  ixy="0.0"  ixz="0.0" iyy="0.0007417" iyz="0.0" izz="0.29" />
+    </inertial>
+    <visual>
+      <origin xyz="0 0 0" rpy="0 0 0"  />
+      <geometry>
+        <mesh filename="package://worms_description/meshes/ee_shoe_reduced.stl"  scale="1 1 1"/>
+      </geometry>
+      <material name="Grey">
+        <color rgba="0.20 0.20 0.20 1.0"/>
+      </material>
+    </visual>
+    <collision>
+      <origin xyz="0 0 0" rpy="0 0 0"  />
+      <geometry>
+        <mesh filename="package://worms_description/meshes/ee_shoe_coll.stl"  scale="1 1 1"/>
+      </geometry>
+    </collision>
+  </link>
+  <!-- Joint definitions -->
+  <joint name="j_hip_structure_${suffix}" type="fixed">
+    <parent link="MP_BODY"/>
+    <child link="hip_structure_${suffix}"/>
+    <origin xyz="${xyz}" rpy="${rpy}" />
+    <axis xyz="1 0 0" />
+    <limit effort="2.8" velocity="5.6548668" lower="-2.6179939" upper="2.6179939" />
+  </joint>
+  <joint name="j_coxa_${suffix}" type="revolute">
+    <parent link="hip_structure_${suffix}"/>
+    <child link="coxa_${suffix}"/>
+    <origin xyz="0 -${hip_structure_length + uib_ee_gap_length} 0" rpy="0 0 0" />
+    <axis xyz="0 0 1" />
+    <limit effort="48" velocity="5.6548668" lower="-2.6179939" upper="2.6179939" />
+  </joint>
+  <joint name="j_thigh_${suffix}" type="revolute">
+    <parent link="coxa_${suffix}"/>
+    <child link="thigh_${suffix}"/>
+    <origin xyz="0 -${coxa_length} 0" rpy="0.785 0 0" />
+    <axis xyz="1 0 0" />
+    <limit effort="48" velocity="5.6548668" lower="-2.6179939" upper="2.6179939" />
+  </joint>
+  <joint name="j_shin_${suffix}" type="revolute">
+    <parent link="thigh_${suffix}"/>
+    <child link="shin_${suffix}"/>
+    <origin xyz="0 -${thigh_length} 0" rpy="0.785 0 0" />
+    <axis xyz="1 0 0" />
+    <limit effort="48" velocity="5.6548668" lower="-2.6179939" upper="2.6179939" />
+  </joint>
+  <joint name="j_shoe_${suffix}" type="fixed">
+    <parent link="shin_${suffix}"/>
+    <child link="shoe_${suffix}"/>
+    <origin xyz="0 -${shin_length + shin_shoe_length} 0" rpy="0 0 0" />
+    <axis xyz="1 0 0" />
+    <limit effort="48" velocity="5.6548668" lower="-2.6179939" upper="2.6179939" />
+  </joint>
+  <!-- Joint transmission definitions -->
+   <transmission name="t_coxa_${suffix}">
     <type>transmission_interface/SimpleTransmission</type>
     <joint name="j_coxa_${suffix}">
@@ -199,199 +411,4 @@
       <mechanicalReduction>1</mechanicalReduction>
     </actuator>
-  </transmission> -->
-<!-- Gazebo material definitions -->
-  <!-- <gazebo reference="hip_structure_${suffix}">
-    <material>Gazebo/Grey</material>
-  </gazebo>
-  <gazebo reference="coxa_${suffix}">
-    <material>Gazebo/Grey</material>
-  </gazebo>
-  <gazebo reference="thigh_${suffix}">
-    <material>Gazebo/Grey</material>
-  </gazebo>
-  <gazebo reference="shin_${suffix}">
-    <material>Gazebo/Grey</material>
-  </gazebo> -->
-<!-- Gazebo gravity setting -->
-  <!-- <turnGravityOff>1</turnGravityOff> -->
-</xacro:macro>
-<!-- Leg generation sub-macro -->
- <xacro:macro name="leg_l" params="xyz rpy suffix">
-  <link name="hip_structure_${suffix}">
-    <inertial>
-      <origin xyz="0 -${hip_structure_length + uib_ee_gap_length} 0" rpy="0 0 0"  />
-      <mass value="${m_uib}"/>
-      <inertia ixx="0.0004167"  ixy="0.0"  ixz="0.0" iyy="0.0007417" iyz="0.0" izz="0.0007417" />
-    </inertial>
-    <visual>
-      <origin xyz="0 -${hip_structure_length + uib_ee_gap_length} 0" rpy="0 0 0"  />
-      <geometry>
-        <mesh filename="package://worms_description/meshes/hip_structure_reduced.stl"  scale="1 1 1"/>
-      </geometry>
-      <material name="Grey">
-        <color rgba="0.20 0.20 0.20 1.0"/>
-      </material>
-    </visual>
-    <!-- <collision>
-      <origin xyz="0 -${hip_structure_length + uib_ee_gap_length} 0" rpy="0 0 0"  />
-      <geometry>
-        <mesh filename="package://worms_description/meshes/hip_structure_reduced.stl"  scale="1 1 1"/>
-      </geometry>
-    </collision> -->
-  </link>
-  <link name="coxa_${suffix}">
-    <inertial>
-      <origin xyz="0 0 0" rpy="0 0 0"  />
-      <mass value="${m_coxa + m_motor}"/>
-      <inertia ixx="0.0004167"  ixy="0.0"  ixz="0.0" iyy="0.0007417" iyz="0.0" izz="0.0007417" />
-    </inertial>
-    <visual>
-      <origin xyz="0 0 0" rpy="0 0 0"  />
-      <geometry>
-        <mesh filename="package://worms_description/meshes/motor_coxa.stl"  scale="1 1 1"/>
-      </geometry>
-      <material name="Grey">
-        <color rgba="0.20 0.20 0.20 1.0"/>
-      </material>
-    </visual>
-    <!-- <collision>
-      <origin xyz="0 0 0" rpy="0 0 0"  />
-      <geometry>
-        <mesh filename="package://worms_description/meshes/motor_coxa.stl"  scale="1 1 1"/>
-      </geometry>
-    </collision> -->
-  </link>
-  <link name="thigh_${suffix}">
-    <inertial>
-      <origin xyz="0 0 0" rpy="0 0 0"  />
-      <mass value="${m_thigh + m_motor}"/>
-      <inertia ixx="0.0004167"  ixy="0.0"  ixz="0.0" iyy="0.0007417" iyz="0.0" izz="0.0007417" />
-    </inertial>
-    <visual>
-      <origin xyz="0 0 0" rpy="0 0 0"  />
-      <geometry>
-        <mesh filename="package://worms_description/meshes/motor_thigh.stl"  scale="1 1 1"/>
-      </geometry>
-      <material name="Grey">
-        <color rgba="0.20 0.20 0.20 1.0"/>
-      </material>
-    </visual>
-    <!-- <collision>
-      <origin xyz="0 0 0" rpy="0 0 0"  />
-      <geometry>
-        <mesh filename="package://worms_description/meshes/motor_thigh.stl"  scale="1 1 1"/>
-      </geometry>
-    </collision> -->
-  </link>
-  <link name="shin_${suffix}">
-    <inertial>
-      <origin xyz="0 0 0" rpy="0 0 0"  />
-      <mass value="${m_shin + m_motor}"/>
-      <inertia ixx="0.0004167"  ixy="0.0"  ixz="0.0" iyy="0.0007417" iyz="0.0" izz="0.0007417" />
-    </inertial>
-    <visual>
-      <origin xyz="0 0 0" rpy="0 0 0"  />
-      <geometry>
-        <mesh filename="package://worms_description/meshes/motor_shin_ee_reduced.stl"  scale="1 1 1"/>
-      </geometry>
-      <material name="Grey">
-        <color rgba="0.20 0.20 0.20 1.0"/>
-      </material>
-    </visual>
-    <!-- <collision>
-      <origin xyz="0 0 0" rpy="0 0 0"  />
-      <geometry>
-        <mesh filename="package://worms_description/meshes/motor_shin_ee_reduced.stl"  scale="1 1 1"/>
-      </geometry>
-    </collision> -->
-  </link>
-  <link name="shoe_${suffix}">
-    <inertial>
-      <origin xyz="0 0 0" rpy="0 0 0"  />
-      <mass value="${m_shin + m_motor}"/>
-      <inertia ixx="0.0004167"  ixy="0.0"  ixz="0.0" iyy="0.0007417" iyz="0.0" izz="0.29" />
-    </inertial>
-    <visual>
-      <origin xyz="0 0 0" rpy="0 0 0"  />
-      <geometry>
-        <mesh filename="package://worms_description/meshes/ee_shoe_reduced.stl"  scale="1 1 1"/>
-      </geometry>
-      <material name="Grey">
-        <color rgba="0.20 0.20 0.20 1.0"/>
-      </material>
-    </visual>
-    <collision>
-      <origin xyz="0 0 0" rpy="0 0 0"  />
-      <geometry>
-        <mesh filename="package://worms_description/meshes/ee_shoe_coll.stl"  scale="1 1 1"/>
-      </geometry>
-    </collision>
-  </link>
-  <!-- Joint definitions -->
-  <joint name="j_hip_structure_${suffix}" type="fixed">
-    <parent link="MP_BODY"/>
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
Commit message: changed inertias of all arm components to near-zero, fixed arm hip actuator torque limit

File: catkin_ws/src/worms_description/urdf/worms.urdf (robot description, URDF)
Before this commit: robot worms, 37 links, 36 joints
Joints:
- joint j_arm_hip_structure_gnc: limit lower=-2.6179939 upper=2.6179939 effort=2.8 velocity=5.6548668 -> lower=-2.6179939 upper=2.6179939 effort=48 velocity=5.6548668

File: catkin_ws/src/worms_description/urdf/worms_urdf.xacro (robot description, xacro)
@@ -81,5 +81,5 @@
       <origin xyz="0 0 0" rpy="0 0 0"  />
       <mass value="${m_shin + m_motor}"/>
-      <inertia ixx="0.0004167"  ixy="0.0"  ixz="0.0" iyy="0.0007417" iyz="0.0" izz="0.0007417" />
+      <inertia ixx="1e-9"  ixy="0.0"  ixz="0.0" iyy="1e-9" iyz="0.0" izz="1e-9" />
     </inertial>
     <visual>
@@ -97,5 +97,5 @@
       <origin xyz="0 0 0" rpy="0 0 0"  />
       <mass value="${m_thigh + m_motor}"/>
-      <inertia ixx="0.0004167"  ixy="0.0"  ixz="0.0" iyy="0.0007417" iyz="0.0" izz="0.0007417" />
+      <inertia ixx="1e-9"  ixy="0.0"  ixz="0.0" iyy="1e-9" iyz="0.0" izz="1e-9" />
     </inertial>
     <visual>
@@ -113,5 +113,5 @@
       <origin xyz="0 0 0" rpy="0 0 0"  />
       <mass value="${m_coxa + m_motor}"/>
-      <inertia ixx="0.0004167"  ixy="0.0"  ixz="0.0" iyy="0.0007417" iyz="0.0" izz="0.0007417" />
+      <inertia ixx="1e-9"  ixy="0.0"  ixz="0.0" iyy="1e-9" iyz="0.0" izz="1e-9" />
     </inertial>
     <visual>
@@ -129,5 +129,5 @@
       <origin xyz="0 0 0" rpy="0 0 0"  />
       <mass value="${m_uib}"/>
-      <inertia ixx="0.0004167"  ixy="0.0"  ixz="0.0" iyy="0.0007417" iyz="0.0" izz="0.0007417" />
+      <inertia ixx="1e-9"  ixy="0.0"  ixz="0.0" iyy="1e-9" iyz="0.0" izz="1e-9" />
     </inertial>
     <visual>
@@ -145,5 +145,5 @@
       <origin xyz="0 0 0" rpy="0 0 0"  />
       <mass value="${m_uib}"/>
-      <inertia ixx="0.0004167"  ixy="0.0"  ixz="0.0" iyy="0.0007417" iyz="0.0" izz="0.0007417" />
+      <inertia ixx="1e-9"  ixy="0.0"  ixz="0.0" iyy="1e-9" iyz="0.0" izz="1e-9" />
     </inertial>
     <visual>
@@ -184,5 +184,5 @@
     <origin xyz="0 ${coxa_length} 0" rpy="0 0 0 " />
     <axis xyz="1 0 0" />
-    <limit effort="2.8" velocity="5.6548668" lower="-2.6179939" upper="2.6179939" />
+    <limit effort="48" velocity="5.6548668" lower="-2.6179939" upper="2.6179939" />
   </joint>
   <joint name="j_arm_lidar_${suffix}" type="fixed">
