Commit message: updated inertias (needs checking)

File: catkin_ws/src/worms_description/urdf/worms.urdf (robot description, URDF)
Before this commit: robot worms, 37 links, 36 joints
Links:
- link arm_coxa_gnc: mass 1.35 -> 1e-9
- link arm_hip_structure_gnc: mass 1 -> 1e-9
- link arm_lidar_gnc: mass 1 -> 1e-9
- link arm_shin_gnc: mass 6.85 -> 13.049999999999999
- link arm_thigh_gnc: mass 2.85 -> 1e-9
- link shoe_lf: mass 6.85 -> 2.52
- link shoe_lm: mass 6.85 -> 2.52
- link shoe_lr: mass 6.85 -> 2.52
- link shoe_rf: mass 6.85 -> 2.52
- link shoe_rm: mass 6.85 -> 2.52
- link shoe_rr: mass 6.85 -> 2.52

File: catkin_ws/src/worms_description/urdf/worms_urdf.xacro (robot description, xacro)
@@ -30,7 +30,4 @@
 <xacro:property name="thigh_offset_z" value="-0.0145" /> -->
 <!-- TODO: Update component masses and inertias -->
-<!-- TODO: Add second ee, uib, and shoe -->
-<!-- TODO: Check link length specs -->
-<!-- TODO: Add simplified collision meshes -->
 <xacro:macro name="worms" params="parent *origin">
       <joint name="j_worms_attachment" type="fixed">
@@ -43,5 +40,5 @@
           <origin xyz="0 0 ${initial_z_offset}" rpy="0 0 1.57" />
 	        <mass value="${m_pallet}" />
-          <inertia ixx="0.003016"  ixy="0.0"  ixz="0.0" iyy="0.003016" iyz="0.0" izz="0.006014" />
+          <inertia ixx="4.501530"  ixy="0.000001"  ixz=" -0.000005" iyy="4.501530" iyz="-0.000001" izz="8.711449" />
         </inertial>
         <visual>
@@ -80,5 +77,6 @@
     <inertial>
       <origin xyz="0 0 0" rpy="0 0 0"  />
-      <mass value="${m_shin + m_motor}"/>
+      <mass value="${m_shin + m_motor + m_thigh + m_motor + m_coxa + m_motor + m_uib + m_uib}"/>
+      <!-- <mass value="${m_shin + m_motor}"/> -->
       <inertia ixx="1e-9"  ixy="0.0"  ixz="0.0" iyy="1e-9" iyz="0.0" izz="1e-9" />
     </inertial>
@@ -96,5 +94,6 @@
     <inertial>
       <origin xyz="0 0 0" rpy="0 0 0"  />
-      <mass value="${m_thigh + m_motor}"/>
+      <mass value="1e-9"/>
+      <!-- <mass value="${m_thigh + m_motor}"/> -->
       <inertia ixx="1e-9"  ixy="0.0"  ixz="0.0" iyy="1e-9" iyz="0.0" izz="1e-9" />
     </inertial>
@@ -112,5 +111,6 @@
     <inertial>
       <origin xyz="0 0 0" rpy="0 0 0"  />
-      <mass value="${m_coxa + m_motor}"/>
+      <mass value="1e-9"/>
+      <!-- <mass value="${m_coxa + m_motor}"/> -->
       <inertia ixx="1e-9"  ixy="0.0"  ixz="0.0" iyy="1e-9" iyz="0.0" izz="1e-9" />
     </inertial>
@@ -128,5 +128,6 @@
     <inertial>
       <origin xyz="0 0 0" rpy="0 0 0"  />
-      <mass value="${m_uib}"/>
+      <mass value="1e-9"/>
+      <!-- <mass value="${m_uib}"/> -->
       <inertia ixx="1e-9"  ixy="0.0"  ixz="0.0" iyy="1e-9" iyz="0.0" izz="1e-9" />
     </inertial>
@@ -144,5 +145,6 @@
     <inertial>
       <origin xyz="0 0 0" rpy="0 0 0"  />
-      <mass value="${m_uib}"/>
+      <mass value="1e-9"/>
+      <!-- <mass value="${m_uib}"/> -->
       <inertia ixx="1e-9"  ixy="0.0"  ixz="0.0" iyy="1e-9" iyz="0.0" izz="1e-9" />
     </inertial>
@@ -239,5 +241,5 @@
       <origin xyz="0 -${hip_structure_length + uib_ee_gap_length} 0" rpy="0 0 0"  />
       <mass value="${m_uib}"/>
-      <inertia ixx="0.0004167"  ixy="0.0"  ixz="0.0" iyy="0.0007417" iyz="0.0" izz="0.0007417" />
+      <inertia ixx="0.001999"  ixy="0.000001"  ixz="0.000001" iyy="0.001386" iyz="0.000035" izz="0.002027" />
     </inertial>
     <visual>
@@ -261,5 +263,5 @@
       <origin xyz="0 0 0" rpy="0 0 0"  />
       <mass value="${m_coxa + m_motor}"/>
-      <inertia ixx="0.0004167"  ixy="0.0"  ixz="0.0" iyy="0.0007417" iyz="0.0" izz="0.0007417" />
+      <inertia ixx="0.003441"  ixy="0.000110"  ixz="-0.000001" iyy="0.000974" iyz="-0.000027" izz="0.003627" />
     </inertial>
     <visual>
@@ -283,5 +285,5 @@
       <origin xyz="0 0 0" rpy="0 0 0"  />
       <mass value="${m_thigh + m_motor}"/>
-      <inertia ixx="0.0004167"  ixy="0.0"  ixz="0.0" iyy="0.0007417" iyz="0.0" izz="0.0007417" />
+      <inertia ixx="0.012495"  ixy="0.000134"  ixz="0.000071" iyy="0.003683" iyz="0.004692" izz="0.009695" />
     </inertial>
     <visual>
@@ -305,5 +307,5 @@
       <origin xyz="0 0 0" rpy="0 0 0"  />
       <mass value="${m_shin + m_motor}"/>
-      <inertia ixx="0.0004167"  ixy="0.0"  ixz="0.0" iyy="0.0007417" iyz="0.0" izz="0.0007417" />
+      <inertia ixx="0.097990"  ixy="0.0"  ixz="0.0" iyy="0.004706" iyz="0.0" izz="0.097765" />
     </inertial>
     <visual>
@@ -326,6 +328,6 @@
     <inertial>
       <origin xyz="0 0 0" rpy="0 0 0"  />
-      <mass value="${m_shin + m_motor}"/>
-      <inertia ixx="0.0004167"  ixy="0.0"  ixz="0.0" iyy="0.0007417" iyz="0.0" izz="0.29" />
+      <mass value="${m_shoe + m_ee}"/>
+      <inertia ixx="0.025955"  ixy="0.0"  ixz="0.0" iyy="0.014273" iyz="0.0" izz="0.014273" />
     </inertial>
     <visual>

Commit message: rotated lidar/gnc arm to match CAD assembly

File: catkin_ws/src/worms_description/urdf/worms.urdf (robot description, URDF)
Before this commit: robot worms, 37 links, 36 joints
Joints:
- joint j_arm_shin_gnc: origin xyz=0 0 1.131 rpy=0 0 0 -> xyz=0 0 1.131 rpy=0 0 -0.523599

File: catkin_ws/src/worms_description/urdf/worms_urdf.xacro (robot description, xacro)
@@ -62,5 +62,5 @@
         <material>Gazebo/Red</material>
       </gazebo>
-    <xacro:arm xyz="0 0 ${initial_z_offset + 0.131}"  rpy="0 0 0" suffix="gnc"/>
+    <xacro:arm xyz="0 0 ${initial_z_offset + 0.131}"  rpy="0 0 -0.523599" suffix="gnc"/>
 <!-- RPY are set to offset the UIB (first component in leg from the pallet) by 90 degrees then by the angle to match the hexagon -->
 <!-- TODO: Replace xyz with calculations based on hexagon diameter -->

Commit message: switched to 1-leg gait

File: catkin_ws/src/worms_description/urdf/worms.urdf (robot description, URDF)
Before this commit: robot worms, 37 links, 36 joints
Joints:
- joint j_thigh_lf: limit lower=-2.6179939 upper=2.6179939 effort=48 velocity=5.6548668 -> lower=-5 upper=5 effort=48 velocity=10
- joint j_thigh_lm: limit lower=-2.6179939 upper=2.6179939 effort=48 velocity=5.6548668 -> lower=-5 upper=5 effort=48 velocity=10
- joint j_thigh_lr: limit lower=-2.6179939 upper=2.6179939 effort=48 velocity=5.6548668 -> lower=-5 upper=5 effort=48 velocity=10
- joint j_thigh_rf: limit lower=-2.6179939 upper=2.6179939 effort=48 velocity=5.6548668 -> lower=-5 upper=5 effort=48 velocity=10
- joint j_thigh_rm: limit lower=-2.6179939 upper=2.6179939 effort=48 velocity=5.6548668 -> lower=-5 upper=5 effort=48 velocity=10
- joint j_thigh_rr: limit lower=-2.6179939 upper=2.6179939 effort=48 velocity=5.6548668 -> lower=-5 upper=5 effort=48 velocity=10

File: catkin_ws/src/worms_description/urdf/worms_urdf.xacro (robot description, xacro)
@@ -367,5 +367,6 @@
     <origin xyz="0 -${coxa_length} 0" rpy="0.785 0 0" />
     <axis xyz="1 0 0" />
-    <limit effort="48" velocity="5.6548668" lower="-2.6179939" upper="2.6179939" />
+    <limit effort="48" velocity="10" lower="-5" upper="5" />
+    <!-- <limit effort="48" velocity="5.6548668" lower="-2.6179939" upper="2.6179939" /> -->
   </joint>
   <joint name="j_shin_${suffix}" type="revolute">

Commit message: two legged gait but front and rear legs have trouble getting off the ground

File: catkin_ws/src/worms_description/urdf/worms.urdf (robot description, URDF)
Before this commit: robot worms, 37 links, 36 joints
Links:
- link MP_BODY: mass 7 -> 7.96891856

File: catkin_ws/src/worms_description/urdf/worms_urdf.xacro (robot description, xacro)
@@ -19,5 +19,5 @@
 <!--  Source: https://docs.google.com/spreadsheets/d/1z4cjFRy08wv40s6Jl9g9mymmIja3-cVj/edit#gid=1875184855-->
 <xacro:property name="m_payload" value="15" />
-<xacro:property name="m_pallet" value="7" />
+<xacro:property name="m_pallet" value="7.96891856" />
 <xacro:property name="m_motor" value="0.85" />
 <xacro:property name="m_hip_structure" value="0.41" />
@@ -41,5 +41,5 @@
           <origin xyz="0 0 ${initial_z_offset}" rpy="0 0 1.57" />
 	        <mass value="${m_pallet}" />
-          <inertia ixx="4.501530"  ixy="0.000001"  ixz=" -0.000005" iyy="4.501530" iyz="-0.000001" izz="8.711449" />
+          <inertia ixx="0.63670162"  ixy="0.000001"  ixz=" -0.000005" iyy="0.63670162" iyz="-0.000001" izz="1.23183903" />
         </inertial>
         <visual>

Commit message: legs are now parallel and the robot still walks straight

File: catkin_ws/src/worms_description/urdf/worms.urdf (robot description, URDF)
Before this commit: robot worms, 37 links, 36 joints
Joints:
- joint j_hip_structure_lf: origin xyz=0.476 0.2748 1.0 rpy=0 0 2.09 -> xyz=0.476 0.2748 1.0 rpy=0 0 3.1399999999999997
- joint j_hip_structure_lr: origin xyz=-0.476 0.2748 1.0 rpy=0 0 4.180000000000001 -> xyz=-0.476 0.2748 1.0 rpy=0 0 3.130000000000001
- joint j_hip_structure_rf: origin xyz=0.476 -0.2748 1.0 rpy=0 0 1.05 -> xyz=0.476 -0.2748 1.0 rpy=0 0 0.0
- joint j_hip_structure_rr: origin xyz=-0.476 -0.2748 1.0 rpy=0 0 -1.0400000000000003 -> xyz=-0.476 -0.2748 1.0 rpy=0 0 0.009999999999999787

File: catkin_ws/src/worms_description/urdf/worms_urdf.xacro (robot description, xacro)
@@ -66,10 +66,10 @@
 <!-- RPY are set to offset the UIB (first component in leg from the pallet) by 90 degrees then by the angle to match the hexagon -->
 <!-- TODO: Replace xyz with calculations based on hexagon diameter -->
-    <xacro:leg_l xyz="0.476 -0.2748 ${initial_z_offset}"  rpy="0 0 ${-0.52 + 1.57}" suffix="rf"/>
+    <xacro:leg_l xyz="0.476 -0.2748 ${initial_z_offset}"  rpy="0 0 ${-0.52 + 1.57 - 1.05}" suffix="rf"/>
     <xacro:leg_l xyz="0.0000 -0.5497 ${initial_z_offset}"  rpy="0 0 ${-1.57 + 1.57}" suffix="rm"/>
-    <xacro:leg_l xyz="-0.476 -0.2748 ${initial_z_offset}"  rpy="0 0 ${-1.57 -1.04 + 1.57}" suffix="rr"/>
-    <xacro:leg_l xyz="0.476 0.2748 ${initial_z_offset}"  rpy="0 0 ${0.52 + 1.57}" suffix="lf"/>
+    <xacro:leg_l xyz="-0.476 -0.2748 ${initial_z_offset}"  rpy="0 0 ${-1.57 -1.04 + 1.57 + 1.05}" suffix="rr"/>
+    <xacro:leg_l xyz="0.476 0.2748 ${initial_z_offset}"  rpy="0 0 ${0.52 + 1.57 + 1.05}" suffix="lf"/>
     <xacro:leg_l xyz="0.0000 0.5497 ${initial_z_offset}"  rpy="0 0 ${1.57 + 1.57}" suffix="lm"/>
-    <xacro:leg_l xyz="-0.476 0.2748 ${initial_z_offset}"  rpy="0 0 ${1.57 + 1.04 + 1.57}" suffix="lr"/>
+    <xacro:leg_l xyz="-0.476 0.2748 ${initial_z_offset}"  rpy="0 0 ${1.57 + 1.04 + 1.57 - 1.05}" suffix="lr"/>
 </xacro:macro>
 <!-- Arm generation sub-macro -->
